File: sw_low_side/main.sch (KiCad schematic (older format))
At the start: 9 parts, among them P1 CONN_XT60, P2 CONN_XT60, P3 CONN_01X02, Q1 IRFB7537PbF, U1 NSI45020AT1G, U2 LM3490IM5-12/NOPB

Commit message: test
Changed lines of the file:
@@
 LIBS:dev_mosfet
 LIBS:dev_switch
-LIBS:main-cache
 EELAYER 25 0
 EELAYER END
@@
 $EndComp
 $Comp
-L +BATT #PWR01
+L +BATT #PWR1
 U 1 1 581866AA
 P 1450 1300
-F 0 "#PWR01" H 1450 1150 50  0001 C CNN
+F 0 "#PWR1" H 1450 1150 50  0001 C CNN
 F 1 "+BATT" H 1450 1440 50  0000 C CNN
 F 2 "" H 1450 1300 50  0000 C CNN
@@
 $EndComp
 $Comp
-L GND #PWR02
+L GND #PWR2
 U 1 1 581868C3
 P 1450 4050
-F 0 "#PWR02" H 1450 3800 50  0001 C CNN
+F 0 "#PWR2" H 1450 3800 50  0001 C CNN
 F 1 "GND" H 1450 3900 50  0000 C CNN
 F 2 "" H 1450 4050 50  0000 C CNN
@@
 Connection ~ 2100 1300
 Wire Wire Line
-	1950 2700 2100 2700
-Wire Wire Line
-	2100 2700 2100 4050
+	1950 2650 2100 2650
+Wire Wire Line
+	2100 2650 2100 4050
 Connection ~ 2100 4050
 Wire Wire Line
-	6900 2700 6900 4050
+	6900 2650 6900 4050
 Connection ~ 6900 4050
-$Comp
-L CONN_XT60 P1
-U 1 1 5818BFBF
-P 1450 2850
-F 0 "P1" H 1650 2800 60  0000 C CNN
-F 1 "CONN_XT60" V 1500 2600 60  0000 C CNN
-F 2 "KiCad-Dev:XT60" H 1550 2750 60  0001 C CNN
-F 3 "" H 1550 2750 60  0001 C CNN
-	1    1450 2850
-	1    0    0    1
-$EndComp
-$Comp
-L CONN_XT60 P2
-U 1 1 5818C052
-P 7600 2850
-F 0 "P2" H 7800 2800 60  0000 C CNN
-F 1 "CONN_XT60" V 7650 2600 60  0000 C CNN
-F 2 "KiCad-Dev:XT60" H 7700 2750 60  0001 C CNN
-F 3 "" H 7700 2750 60  0001 C CNN
-	1    7600 2850
-	-1   0    0    1
-$EndComp
-Wire Wire Line
-	7100 2700 6900 2700
+Wire Wire Line
+	7100 2650 6900 2650
 Wire Wire Line
 	7100 2550 6900 2550
@@
 	3100 3850 3100 4050
 Connection ~ 3100 4050
+$Comp
+L CONN_XT60 P2
+U 1 1 581B5768
+P 7400 2600
+F 0 "P2" H 7400 2750 60  0000 C CNN
+F 1 "CONN_XT60" H 7400 2450 60  0000 C CNN
+F 2 "KiCad-Dev:XT60" H 7300 2750 60  0001 C CNN
+F 3 "" H 7300 2750 60  0001 C CNN
+	1    7400 2600
+	-1   0    0    1
+$EndComp
+$Comp
+L CONN_XT60 P1
+U 1 1 581B5929
+P 1650 2600
+F 0 "P1" H 1650 2750 60  0000 C CNN
+F 1 "CONN_XT60" H 1650 2450 60  0000 C CNN
+F 2 "KiCad-Dev:XT60" H 1550 2750 60  0001 C CNN
+F 3 "" H 1550 2750 60  0001 C CNN
+	1    1650 2600
+	1    0    0    1
+$EndComp
 $EndSCHEMATC
