File: sw_high_side/main.sch (KiCad schematic (older format))
At the start: 8 parts, among them P1 CONN_XT60, P2 CONN_01X02, P3 CONN_XT60, Q1 IRFB7537PbF, U1 NSI45020AT1G, U2 MIC5014

Commit message: test
Changed lines of the file:
@@
 EESchema Schematic File Version 2
+LIBS:main-rescue
 LIBS:power
 LIBS:device
@@
 	4650 3800 4650 4700
 Connection ~ 4650 4700
-$Comp
-L NSI45020AT1G U1
-U 1 1 5819D445
-P 5750 4150
-F 0 "U1" H 5750 4050 60  0000 C CNN
-F 1 "NSI45020AT1G" H 5750 4250 60  0000 C CNN
-F 2 "Diodes_SMD:SOD-123" H 5000 4300 60  0001 C CNN
-F 3 "" H 5000 4300 60  0001 C CNN
-	1    5750 4150
-	1    0    0    -1
-$EndComp
 Connection ~ 9650 4700
 $Comp
@@
 	5050 3800 5050 4150
 Wire Wire Line
-	5050 4150 5150 4150
+	5050 4150 5450 4150
 Wire Wire Line
 	8050 4350 8200 4350
@@
 Connection ~ 6600 4700
 Wire Wire Line
-	6350 4150 7150 4150
+	6050 4150 7150 4150
 Wire Wire Line
 	6600 4150 6600 4250
@@
 	0    -1   -1   0
 $EndComp
+$Comp
+L NSI45020AT1G U1
+U 1 1 5820831C
+P 5750 4150
+F 0 "U1" H 5750 4000 60  0000 C CNN
+F 1 "NSI45020AT1G" H 5750 4300 60  0000 C CNN
+F 2 "Diodes_SMD:SOD-123" H 5000 4300 60  0001 C CNN
+F 3 "" H 5000 4300 60  0001 C CNN
+	1    5750 4150
+	1    0    0    -1
+$EndComp
 $EndSCHEMATC
