File: sw_high_side3/main.sch (KiCad schematic (older format))
At the start: 10 parts, among them P1 CONN_01X02, Q1 IRFB7537PbF, U1 NSI45020AT1G, U2 MIC5014

Commit message: test
Parts:
- removed P?: CONN_01X02, symbol CONN_01X02
- removed U?: 74LVC1G08, symbol 74LVC1G08
- removed U?: LM3480-5.0, TO_SOT_Packages_SMD:SOT-23, symbol LM3480-5.0
- added P2: CONN_02X03, Pin_Headers:Pin_Header_Straight_2x03, symbol CONN_02X03
- added P4, P5: CONN_XT60, KiCad-Dev:XT60, symbol CONN_XT60
- added U3: 74LVC1G08, TO_SOT_Packages_SMD:SOT-353, symbol 74LVC1G08
- P3: renamed from P?; footprint (none) -> Pin_Headers:Pin_Header_Straight_1x02
Connections:
- net In+: now also P4.2 (+)
- net In-: now also P2.1 (P1), P4.1 (-), P5.1 (-), U3.3 (GND)
- net Out+: now also P5.2 (+)
- net at U2.2 (Input): now also U3.4 (Y)
- net at D1.2 (A), P3.1 (P1), R1.1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: now also U3.2 (B), U3.5 (VCC)
- net at P3.2 (P2): now also P2.2 (P2), U3.1 (A)
Other:
- moved on the sheet: P1
Changed lines of the file:
@@
 LIBS:dev_ic
 LIBS:dev_conn
+LIBS:main-cache
 EELAYER 25 0
 EELAYER END
@@
 L CONN_01X02 P1
 U 1 1 5821D69A
-P 5500 2800
-F 0 "P1" H 5500 2950 50  0000 C CNN
-F 1 "CONN_01X02" V 5600 2800 50  0000 C CNN
-F 2 "Pin_Headers:Pin_Header_Straight_1x02" H 5500 2800 50  0001 C CNN
-F 3 "" H 5500 2800 50  0000 C CNN
-	1    5500 2800
+P 5500 2400
+F 0 "P1" H 5500 2550 50  0000 C CNN
+F 1 "CONN_01X02" V 5600 2400 50  0000 C CNN
+F 2 "Pin_Headers:Pin_Header_Straight_1x02" H 5500 2400 50  0001 C CNN
+F 3 "" H 5500 2400 50  0000 C CNN
+	1    5500 2400
 	-1   0    0    1
 $EndComp
@@
 $EndComp
 $Comp
+L 74LVC1G08 U3
+U 1 1 5822357C
+P 7600 3550
+F 0 "U3" H 7700 3300 60  0000 C CNN
+F 1 "74LVC1G08" H 7900 3800 60  0000 C CNN
+F 2 "TO_SOT_Packages_SMD:SOT-353" H 7550 3600 60  0001 C CNN
+F 3 "http://www.nxp.com/documents/data_sheet/74LVC1G08.pdf?" H 8100 3100 60  0001 C CNN
+	1    7600 3550
+	1    0    0    -1
+$EndComp
+$Comp
 L NSI45020AT1G U1
-U 1 1 5821D786
+U 1 1 58223917
 P 5700 3200
 F 0 "U1" H 5700 3050 60  0000 C CNN
 F 1 "NSI45020AT1G" H 5700 3350 60  0000 C CNN
 F 2 "Diodes_SMD:SOD-123" H 4950 3350 60  0001 C CNN
-F 3 "" H 4950 3350 60  0001 C CNN
+F 3 "http://www.onsemi.com/pub_link/Collateral/NSI45020A-D.PDF" H 5800 2850 60  0001 C CNN
 	1    5700 3200
 	0    1    1    0
 $EndComp
 $Comp
-L 74LVC1G08 U?
-U 1 1 5821F12D
-P 7600 3550
-F 0 "U?" H 7700 3300 60  0000 C CNN
-F 1 "74LVC1G08" H 7900 3800 60  0000 C CNN
-F 2 "" H 7550 3600 60  0001 C CNN
-F 3 "" H 7550 3600 60  0001 C CNN
-	1    7600 3550
-	1    0    0    -1
-$EndComp
-$Comp
-L LM3480-5.0 U?
-U 1 1 5821F2E0
-P 7600 2450
-F 0 "U?" H 7300 2600 50  0000 L CNN
-F 1 "LM3480-5.0" H 7900 2600 50  0000 R CNN
-F 2 "TO_SOT_Packages_SMD:SOT-23" H 7600 2050 50  0001 C CIN
-F 3 "" H 7600 2450 50  0000 C CNN
-	1    7600 2450
-	0    1    1    0
-$EndComp
-Text HLabel 7200 2450 0    60   Input ~ 0
-In-
-$Comp
-L CONN_01X02 P?
+L CONN_XT60 P4
+U 1 1 5822400C
+P 4500 2850
+F 0 "P4" H 4500 3000 60  0000 C CNN
+F 1 "CONN_XT60" H 4500 2700 60  0000 C CNN
+F 2 "KiCad-Dev:XT60" H 4400 3000 60  0001 C CNN
+F 3 "" H 4400 3000 60  0001 C CNN
+	1    4500 2850
+	1    0    0    1
+$EndComp
+$Comp
+L CONN_XT60 P5
+U 1 1 582240B2
+P 10300 2800
+F 0 "P5" H 10300 2950 60  0000 C CNN
+F 1 "CONN_XT60" H 10300 2650 60  0000 C CNN
+F 2 "KiCad-Dev:XT60" H 10200 2950 60  0001 C CNN
+F 3 "" H 10200 2950 60  0001 C CNN
+	1    10300 2800
+	-1   0    0    1
+$EndComp
+Wire Wire Line
+	8300 3450 8350 3450
+Wire Wire Line
+	8300 1850 8300 3450
+Wire Wire Line
+	5000 1850 9150 1850
+Connection ~ 8300 1850
+Wire Wire Line
+	9400 2150 9400 3750
+Wire Wire Line
+	9400 3750 9250 3750
+Wire Wire Line
+	8350 3750 8200 3750
+Wire Wire Line
+	5000 4150 9850 4150
+Wire Wire Line
+	8350 3650 8300 3650
+Wire Wire Line
+	8300 3650 8300 3950
+Wire Wire Line
+	9650 1850 9650 3950
+Wire Wire Line
+	9550 1850 10050 1850
+Connection ~ 9650 1850
+Connection ~ 6100 4150
+Wire Wire Line
+	6100 4000 6100 4150
+Wire Wire Line
+	5700 4050 5700 4150
+Connection ~ 5700 4150
+Wire Wire Line
+	5700 3500 5700 3650
+Connection ~ 6100 3600
+Wire Wire Line
+	5700 2450 5700 2900
+Wire Wire Line
+	5700 1850 5700 2350
+Connection ~ 5700 1850
+Wire Wire Line
+	5700 3600 7250 3600
+Wire Wire Line
+	8050 3550 8350 3550
+Connection ~ 5700 3600
+Wire Wire Line
+	9650 3950 8300 3950
+Wire Wire Line
+	7600 4150 7600 3950
+Wire Wire Line
+	8200 3750 8200 4150
+Connection ~ 7600 4150
+Wire Wire Line
+	7000 3350 7000 3500
+Wire Wire Line
+	6450 3500 7250 3500
+Wire Wire Line
+	6900 3350 6900 3600
+Connection ~ 6900 3600
+Wire Wire Line
+	6350 3350 6350 4150
+Connection ~ 6350 4150
+Wire Wire Line
+	6450 3350 6450 3500
+Connection ~ 7000 3500
+Wire Wire Line
+	6100 2650 6100 3700
+Wire Wire Line
+	7600 3150 7600 2650
+Wire Wire Line
+	7600 2650 6100 2650
+Wire Wire Line
+	10000 2750 9850 2750
+Wire Wire Line
+	9850 2750 9850 1850
+Connection ~ 9850 1850
+Wire Wire Line
+	10000 2850 9850 2850
+Wire Wire Line
+	9850 2850 9850 4150
+Connection ~ 8200 4150
+Wire Wire Line
+	4800 2800 5200 2800
+Wire Wire Line
+	5200 2800 5200 1850
+Connection ~ 5200 1850
+Wire Wire Line
+	4800 2900 5200 2900
+Wire Wire Line
+	5200 2900 5200 4150
+Connection ~ 5200 4150
+$Comp
+L CONN_01X02 P3
 U 1 1 5821FA68
 P 6950 3150
-F 0 "P?" H 6950 3300 50  0000 C CNN
+F 0 "P3" H 6950 3300 50  0000 C CNN
 F 1 "CONN_01X02" V 7050 3150 50  0000 C CNN
-F 2 "" H 6950 3150 50  0000 C CNN
+F 2 "Pin_Headers:Pin_Header_Straight_1x02" H 6950 3150 50  0001 C CNN
 F 3 "" H 6950 3150 50  0000 C CNN
 	1    6950 3150
@@
 $EndComp
 $Comp
-L CONN_01X02 P?
-U 1 1 5821FB8D
-P 6400 3150
-F 0 "P?" H 6400 3300 50  0000 C CNN
-F 1 "CONN_01X02" V 6500 3150 50  0000 C CNN
-F 2 "" H 6400 3150 50  0000 C CNN
-F 3 "" H 6400 3150 50  0000 C CNN
-	1    6400 3150
-	0    -1   -1   0
-$EndComp
-Wire Wire Line
-	8300 3450 8350 3450
-Wire Wire Line
-	8300 1850 8300 3450
-Wire Wire Line
-	5000 1850 5700 1850
-Wire Wire Line
-	5700 1850 7600 1850
-Wire Wire Line
-	7600 1850 8300 1850
-Wire Wire Line
-	8300 1850 9150 1850
-Connection ~ 8300 1850
-Wire Wire Line
-	9400 2150 9400 3750
-Wire Wire Line
-	9400 3750 9250 3750
-Wire Wire Line
-	8350 3750 8200 3750
-Wire Wire Line
-	5000 4150 5700 4150
-Wire Wire Line
-	5700 4150 6100 4150
-Wire Wire Line
-	6100 4150 6350 4150
-Wire Wire Line
-	6350 4150 7600 4150
-Wire Wire Line
-	7600 4150 8200 4150
-Wire Wire Line
-	8350 3650 8300 3650
-Wire Wire Line
-	8300 3650 8300 3950
-Wire Wire Line
-	9650 1850 9650 3950
-Wire Wire Line
-	9550 1850 9650 1850
-Wire Wire Line
-	9650 1850 10050 1850
-Connection ~ 9650 1850
-Connection ~ 6100 4150
-Wire Wire Line
-	6100 4000 6100 4150
-Wire Wire Line
-	5700 4050 5700 4150
-Connection ~ 5700 4150
-Wire Wire Line
-	5700 3500 5700 3600
-Wire Wire Line
-	5700 3600 5700 3650
-Connection ~ 6100 3600
-Wire Wire Line
-	5700 2850 5700 2900
-Wire Wire Line
-	5700 1850 5700 2750
-Connection ~ 5700 1850
-Wire Wire Line
-	5700 3600 6100 3600
-Wire Wire Line
-	6100 3600 6900 3600
-Wire Wire Line
-	6900 3600 7250 3600
-Wire Wire Line
-	8050 3550 8350 3550
-Connection ~ 5700 3600
-Wire Wire Line
-	9650 3950 8300 3950
-Wire Wire Line
-	7600 2950 7600 3150
-Wire Wire Line
-	7600 1850 7600 1950
-Connection ~ 7600 1850
-Wire Wire Line
-	7600 4150 7600 3950
-Wire Wire Line
-	8200 4150 8200 3750
-Connection ~ 7600 4150
-Wire Wire Line
-	7200 2450 7300 2450
-Wire Wire Line
-	7000 3350 7000 3500
-Wire Wire Line
-	6450 3500 7000 3500
-Wire Wire Line
-	7000 3500 7250 3500
-Wire Wire Line
-	6900 3350 6900 3600
-Connection ~ 6900 3600
-Wire Wire Line
-	6350 3350 6350 4150
-Connection ~ 6350 4150
-Wire Wire Line
-	6450 3350 6450 3500
-Connection ~ 7000 3500
-Wire Wire Line
-	6100 3600 6100 3700
+L CONN_02X03 P2
+U 1 1 582244A7
+P 6500 2950
+F 0 "P2" H 6500 3150 50  0000 C CNN
+F 1 "CONN_02X03" H 6500 2750 50  0000 C CNN
+F 2 "Pin_Headers:Pin_Header_Straight_2x03" H 6500 1750 50  0001 C CNN
+F 3 "" H 6500 1750 50  0000 C CNN
+	1    6500 2950
+	1    0    0    -1
+$EndComp
+Wire Wire Line
+	6250 2850 6200 2850
+Wire Wire Line
+	6200 2850 6200 3350
+Wire Wire Line
+	6200 3350 6350 3350
+Wire Wire Line
+	6750 2850 6800 2850
+Wire Wire Line
+	6800 2850 6800 3350
+Wire Wire Line
+	6800 3350 6450 3350
 $EndSCHEMATC

Commit message: test
Parts:
- removed P2: CONN_02X03, Pin_Headers:Pin_Header_Straight_2x03, symbol CONN_02X03
- added P2: CONN_01X02, Pin_Headers:Pin_Header_Straight_1x02, symbol CONN_01X02
- added U4: LM3480-3.3, TO_SOT_Packages_SMD:SOT-23, symbol LM3480-3.3
Connections:
- net In+: now also U4.2 (VIN)
- net In-: now also P2.1 (P1), U4.3 (GND)
- net at D1.2 (A), P3.1 (P1), R1.1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: no longer U3.5 (VCC)
- net at P3.2 (P2), U3.1 (A): now also P2.2 (P2)
- new net: U3.5 (VCC), U4.1 (VOUT)
Changed lines of the file:
@@
 Wire Wire Line
 	5700 3500 5700 3650
-Connection ~ 6100 3600
 Wire Wire Line
 	5700 2450 5700 2900
@@
 Wire Wire Line
 	6350 3350 6350 4150
-Connection ~ 6350 4150
 Wire Wire Line
 	6450 3350 6450 3500
 Connection ~ 7000 3500
 Wire Wire Line
-	6100 2650 6100 3700
-Wire Wire Line
-	7600 3150 7600 2650
-Wire Wire Line
-	7600 2650 6100 2650
+	7600 2900 7600 3150
 Wire Wire Line
 	10000 2750 9850 2750
@@
 	0    -1   -1   0
 $EndComp
+Connection ~ 6350 4150
+Wire Wire Line
+	6100 3700 6100 3600
+Connection ~ 6100 3600
 $Comp
-L CONN_02X03 P2
-U 1 1 582244A7
-P 6500 2950
-F 0 "P2" H 6500 3150 50  0000 C CNN
-F 1 "CONN_02X03" H 6500 2750 50  0000 C CNN
-F 2 "Pin_Headers:Pin_Header_Straight_2x03" H 6500 1750 50  0001 C CNN
-F 3 "" H 6500 1750 50  0000 C CNN
-	1    6500 2950
-	1    0    0    -1
+L LM3480-3.3 U4
+U 1 1 5822E2E2
+P 7600 2400
+F 0 "U4" H 7300 2550 50  0000 L CNN
+F 1 "LM3480-3.3" H 7900 2550 50  0000 R CNN
+F 2 "TO_SOT_Packages_SMD:SOT-23" H 7600 2000 50  0001 C CIN
+F 3 "" H 7600 2400 50  0000 C CNN
+	1    7600 2400
+	0    1    1    0
 $EndComp
 Wire Wire Line
-	6250 2850 6200 2850
+	7600 1900 7600 1850
+Connection ~ 7600 1850
+Text HLabel 7150 2400 0    60   Input ~ 0
+In-
 Wire Wire Line
-	6200 2850 6200 3350
-Wire Wire Line
-	6200 3350 6350 3350
-Wire Wire Line
-	6750 2850 6800 2850
-Wire Wire Line
-	6800 2850 6800 3350
-Wire Wire Line
-	6800 3350 6450 3350
+	7150 2400 7300 2400
+$Comp
+L CONN_01X02 P2
+U 1 1 5822E658
+P 6400 3150
+F 0 "P2" H 6400 3300 50  0000 C CNN
+F 1 "CONN_01X02" V 6500 3150 50  0000 C CNN
+F 2 "Pin_Headers:Pin_Header_Straight_1x02" H 6400 3150 50  0001 C CNN
+F 3 "" H 6400 3150 50  0000 C CNN
+	1    6400 3150
+	0    -1   -1   0
+$EndComp
 $EndSCHEMATC
