File: pdb1/fuse.sch (KiCad schematic (older format))
At the start: 5 parts

Commit message: test
Parts:
- D6, D7: renamed from D?; footprint (none) -> LEDs:LED_0805
- F6: renamed from F?; footprint (none) -> KiCad-Dev:Fuseholder_test
- U2, U3: renamed from U?; footprint (none) -> Diodes_SMD:SOD-123
Changed lines of the file:
@@
 $Descr A4 11693 8268
 encoding utf-8
-Sheet 3 5
+Sheet 4 5
 Title ""
 Date ""
@@
 GND
 $Comp
-L FUSE F?
+L FUSE F6
 U 1 1 581F29E4
 P 4250 2400
-F 0 "F?" H 4350 2450 50  0000 C CNN
+F 0 "F6" H 4350 2450 50  0000 C CNN
 F 1 "FUSE" H 4150 2350 50  0000 C CNN
-F 2 "" H 4250 2400 50  0000 C CNN
+F 2 "KiCad-Dev:Fuseholder_test" H 4250 2400 50  0001 C CNN
 F 3 "" H 4250 2400 50  0000 C CNN
 	1    4250 2400
@@
 	3350 2400 4000 2400
 $Comp
-L LED D?
+L LED D6
 U 1 1 581F2A47
 P 3700 3750
-F 0 "D?" H 3700 3850 50  0000 C CNN
+F 0 "D6" H 3700 3850 50  0000 C CNN
 F 1 "LED" H 3700 3650 50  0000 C CNN
-F 2 "" H 3700 3750 50  0000 C CNN
+F 2 "LEDs:LED_0805" H 3700 3750 50  0001 C CNN
 F 3 "" H 3700 3750 50  0000 C CNN
 	1    3700 3750
@@
 $EndComp
 $Comp
-L LED D?
+L LED D7
 U 1 1 581F2A80
 P 4750 3750
-F 0 "D?" H 4750 3850 50  0000 C CNN
+F 0 "D7" H 4750 3850 50  0000 C CNN
 F 1 "LED" H 4750 3650 50  0000 C CNN
-F 2 "" H 4750 3750 50  0000 C CNN
+F 2 "LEDs:LED_0805" H 4750 3750 50  0001 C CNN
 F 3 "" H 4750 3750 50  0000 C CNN
 	1    4750 3750
@@
 Connection ~ 3700 4100
 $Comp
-L NSI45020AT1G U?
+L NSI45020AT1G U2
 U 1 1 581F329C
 P 3700 2850
-F 0 "U?" H 3700 2700 60  0000 C CNN
+F 0 "U2" H 3700 2700 60  0000 C CNN
 F 1 "NSI45020AT1G" H 3700 3000 60  0000 C CNN
-F 2 "" H 2950 3000 60  0001 C CNN
+F 2 "Diodes_SMD:SOD-123" H 2950 3000 60  0001 C CNN
 F 3 "" H 2950 3000 60  0001 C CNN
 	1    3700 2850
@@
 	3700 3150 3700 3550
 $Comp
-L NSI45020AT1G U?
+L NSI45020AT1G U3
 U 1 1 581F336B
 P 4750 2850
-F 0 "U?" H 4750 2700 60  0000 C CNN
+F 0 "U3" H 4750 2700 60  0000 C CNN
 F 1 "NSI45020AT1G" H 4750 3000 60  0000 C CNN
-F 2 "" H 4000 3000 60  0001 C CNN
+F 2 "Diodes_SMD:SOD-123" H 4000 3000 60  0001 C CNN
 F 3 "" H 4000 3000 60  0001 C CNN
 	1    4750 2850

Commit message: test
Changed lines of the file:
@@
 Wire Wire Line
 	4750 2400 4750 2550
-Connection ~ 4750 4100
 Text HLabel 5500 2400 2    60   Output ~ 0
 out+
