File: pdb1/current_sensor.sch (KiCad schematic (older format))
At the start: 5 parts

Commit message: test
Parts:
- C1, C2: renamed from C?; footprint (none) -> Capacitors_SMD:C_0805_HandSoldering
- R1: renamed from R?; footprint (none) -> KiCad-Dev:SMD_1052_Metric
- R2: renamed from R?; footprint (none) -> Resistors_SMD:R_0805_HandSoldering
- U1: renamed from U?; footprint SOT-23 -> TO_SOT_Packages_SMD:SOT-23-5
Changed lines of the file:
@@
 $Descr A4 11693 8268
 encoding utf-8
-Sheet 2 5
+Sheet 3 5
 Title ""
 Date ""
@@
 $EndDescr
 $Comp
-L INA169 U?
+L INA169 U1
 U 1 1 581F380C
 P 4900 3600
-F 0 "U?" H 5150 3650 60  0000 C CNN
+F 0 "U1" H 5150 3650 60  0000 C CNN
 F 1 "INA169" H 5150 3750 60  0000 C CNN
-F 2 "SOT-23" H 6950 3900 60  0001 C CNN
+F 2 "TO_SOT_Packages_SMD:SOT-23-5" H 6950 3900 60  0001 C CNN
 F 3 "http://www.ti.com/lit/ds/symlink/ina139.pdf" H 6750 3700 60  0001 C CNN
 	1    4900 3600
@@
 out+
 $Comp
-L R R?
+L R R1
 U 1 1 581F3902
 P 5200 3150
-F 0 "R?" V 5280 3150 50  0000 C CNN
+F 0 "R1" V 5280 3150 50  0000 C CNN
 F 1 "R" V 5200 3150 50  0000 C CNN
-F 2 "" V 5130 3150 50  0000 C CNN
+F 2 "KiCad-Dev:SMD_1052_Metric" V 5130 3150 50  0001 C CNN
 F 3 "" H 5200 3150 50  0000 C CNN
 	1    5200 3150
@@
 $EndComp
 $Comp
-L R R?
+L R R2
 U 1 1 581F39E8
 P 5900 4400
-F 0 "R?" V 5980 4400 50  0000 C CNN
+F 0 "R2" V 5980 4400 50  0000 C CNN
 F 1 "R" V 5900 4400 50  0000 C CNN
-F 2 "" V 5830 4400 50  0000 C CNN
+F 2 "Resistors_SMD:R_0805_HandSoldering" V 5830 4400 50  0001 C CNN
 F 3 "" H 5900 4400 50  0000 C CNN
 	1    5900 4400
@@
 Connection ~ 5900 4100
 $Comp
-L C C?
+L C C2
 U 1 1 581F3C78
 P 6150 4400
-F 0 "C?" H 6175 4500 50  0000 L CNN
+F 0 "C2" H 6175 4500 50  0000 L CNN
 F 1 "C" H 6175 4300 50  0000 L CNN
-F 2 "" H 6188 4250 50  0000 C CNN
+F 2 "Capacitors_SMD:C_0805_HandSoldering" H 6188 4250 50  0001 C CNN
 F 3 "" H 6150 4400 50  0000 C CNN
 	1    6150 4400
@@
 Connection ~ 6150 4100
 $Comp
-L C C?
+L C C1
 U 1 1 581F3D4F
 P 4500 4300
-F 0 "C?" H 4525 4400 50  0000 L CNN
+F 0 "C1" H 4525 4400 50  0000 L CNN
 F 1 "C" H 4525 4200 50  0000 L CNN
-F 2 "" H 4538 4150 50  0000 C CNN
+F 2 "Capacitors_SMD:C_0805_HandSoldering" H 4538 4150 50  0001 C CNN
 F 3 "" H 4500 4300 50  0000 C CNN
 	1    4500 4300

Commit message: test
Parts:
- added P5: CONN_01X02, Pin_Headers:Pin_Header_Straight_1x02, symbol CONN_01X02
- added P7, P8: CONN_01X01, Pin_Headers:Pin_Header_Straight_1x01, symbol CONN_01X01
Connections:
- net in+: now also P5.2 (P2), P7.1 (P1)
- net out+: now also P5.1 (P1), P8.1 (P1)
Changed lines of the file:
@@
 	4650 3400 4950 3400
 Wire Wire Line
-	4950 3400 4950 3150
+	4950 3400 4950 2850
 Wire Wire Line
 	5750 3700 5750 3400
@@
 	5750 3400 5450 3400
 Wire Wire Line
-	5450 3400 5450 3150
+	5450 3400 5450 2850
 Connection ~ 5450 3150
 Text HLabel 6700 4100 2    60   Output ~ 0
@@
 Wire Wire Line
 	6150 4550 6150 4750
-Connection ~ 6150 4750
 Wire Wire Line
 	6150 4250 6150 4100
@@
 Wire Wire Line
 	6150 4750 3700 4750
+$Comp
+L CONN_01X02 P5
+U 1 1 58247AF2
+P 5200 2650
+F 0 "P5" H 5200 2800 50  0000 C CNN
+F 1 "CONN_01X02" V 5300 2650 50  0000 C CNN
+F 2 "Pin_Headers:Pin_Header_Straight_1x02" H 5200 2650 50  0001 C CNN
+F 3 "" H 5200 2650 50  0000 C CNN
+	1    5200 2650
+	0    1    -1   0
+$EndComp
+Wire Wire Line
+	4550 2850 5150 2850
+Wire Wire Line
+	5250 2850 5800 2850
+$Comp
+L CONN_01X01 P7
+U 1 1 582496F0
+P 4550 2550
+F 0 "P7" H 4550 2650 50  0000 C CNN
+F 1 "CONN_01X01" V 4650 2550 50  0000 C CNN
+F 2 "Pin_Headers:Pin_Header_Straight_1x01" H 4550 2550 50  0001 C CNN
+F 3 "" H 4550 2550 50  0000 C CNN
+	1    4550 2550
+	0    -1   -1   0
+$EndComp
+Wire Wire Line
+	4550 2750 4550 2850
+Connection ~ 4950 2850
+$Comp
+L CONN_01X01 P8
+U 1 1 58249867
+P 5800 2550
+F 0 "P8" H 5800 2650 50  0000 C CNN
+F 1 "CONN_01X01" V 5900 2550 50  0000 C CNN
+F 2 "Pin_Headers:Pin_Header_Straight_1x01" H 5800 2550 50  0001 C CNN
+F 3 "" H 5800 2550 50  0000 C CNN
+	1    5800 2550
+	0    -1   -1   0
+$EndComp
+Wire Wire Line
+	5800 2850 5800 2750
+Connection ~ 5450 2850
 $EndSCHEMATC

Commit message: test
Parts:
- removed P5: CONN_01X02, Pin_Headers:Pin_Header_Straight_1x02, symbol CONN_01X02
- removed P7, P8: CONN_01X01, Pin_Headers:Pin_Header_Straight_1x01, symbol CONN_01X01
Changed lines of the file:
@@
 	4650 3400 4950 3400
-Wire Wire Line
-	4950 3400 4950 2850
 Wire Wire Line
 	5750 3700 5750 3400
 Wire Wire Line
 	5750 3400 5450 3400
-Wire Wire Line
-	5450 3400 5450 2850
 Connection ~ 5450 3150
 Text HLabel 6700 4100 2    60   Output ~ 0
@@
 Wire Wire Line
 	6150 4750 3700 4750
-$Comp
-L CONN_01X02 P5
-U 1 1 58247AF2
-P 5200 2650
-F 0 "P5" H 5200 2800 50  0000 C CNN
-F 1 "CONN_01X02" V 5300 2650 50  0000 C CNN
-F 2 "Pin_Headers:Pin_Header_Straight_1x02" H 5200 2650 50  0001 C CNN
-F 3 "" H 5200 2650 50  0000 C CNN
-	1    5200 2650
-	0    1    -1   0
-$EndComp
 Wire Wire Line
-	4550 2850 5150 2850
+	4950 3400 4950 3150
 Wire Wire Line
-	5250 2850 5800 2850
-$Comp
-L CONN_01X01 P7
-U 1 1 582496F0
-P 4550 2550
-F 0 "P7" H 4550 2650 50  0000 C CNN
-F 1 "CONN_01X01" V 4650 2550 50  0000 C CNN
-F 2 "Pin_Headers:Pin_Header_Straight_1x01" H 4550 2550 50  0001 C CNN
-F 3 "" H 4550 2550 50  0000 C CNN
-	1    4550 2550
-	0    -1   -1   0
-$EndComp
-Wire Wire Line
-	4550 2750 4550 2850
-Connection ~ 4950 2850
-$Comp
-L CONN_01X01 P8
-U 1 1 58249867
-P 5800 2550
-F 0 "P8" H 5800 2650 50  0000 C CNN
-F 1 "CONN_01X01" V 5900 2550 50  0000 C CNN
-F 2 "Pin_Headers:Pin_Header_Straight_1x01" H 5800 2550 50  0001 C CNN
-F 3 "" H 5800 2550 50  0000 C CNN
-	1    5800 2550
-	0    -1   -1   0
-$EndComp
-Wire Wire Line
-	5800 2850 5800 2750
-Connection ~ 5450 2850
+	5450 3400 5450 3150
 $EndSCHEMATC

Commit message: test
Parts:
- C1, C2: footprint Capacitors_SMD:C_0805_HandSoldering -> Capacitors_SMD:C_0603
- R2: footprint Resistors_SMD:R_0805_HandSoldering -> Resistors_SMD:R_0603
Changed lines of the file:
@@
 F 0 "R2" V 5980 4400 50  0000 C CNN
 F 1 "R" V 5900 4400 50  0000 C CNN
-F 2 "Resistors_SMD:R_0805_HandSoldering" V 5830 4400 50  0001 C CNN
+F 2 "Resistors_SMD:R_0603" V 5830 4400 50  0001 C CNN
 F 3 "" H 5900 4400 50  0000 C CNN
 	1    5900 4400
@@
 F 0 "C2" H 6175 4500 50  0000 L CNN
 F 1 "C" H 6175 4300 50  0000 L CNN
-F 2 "Capacitors_SMD:C_0805_HandSoldering" H 6188 4250 50  0001 C CNN
+F 2 "Capacitors_SMD:C_0603" H 6188 4250 50  0001 C CNN
 F 3 "" H 6150 4400 50  0000 C CNN
 	1    6150 4400
@@
 F 0 "C1" H 4525 4400 50  0000 L CNN
 F 1 "C" H 4525 4200 50  0000 L CNN
-F 2 "Capacitors_SMD:C_0805_HandSoldering" H 4538 4150 50  0001 C CNN
+F 2 "Capacitors_SMD:C_0603" H 4538 4150 50  0001 C CNN
 F 3 "" H 4500 4300 50  0000 C CNN
 	1    4500 4300
