File: pdb1/pdb1.kicad_pcb (KiCad board)
At the start: 2 copper layers, 33 parts, among them P1 CONN_XT60, P2 CONN_XT60, P3 CONN_02X03, P4 CONN_01X02, Q1 IRFB7537PbF, U1 INA169, U2 NSI45020AT1G, U3 NSI45020AT1G, U4 NSI45020AT1G, U5 LM3480-5.0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

Commit message: test
Routing:
- net /channel/in+: track 7.62 -> 13.7 mm
- net /channel/current_sensor/sense: track 0.00 -> 2.58 mm
- net /channel/GND: track 143.6 -> 146.2 mm
Changed lines of the file:
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@@
-(kicad_pcb (version 4) (host pcbnew 4.0.4-stable)
+(kicad_pcb (version 4) (host pcbnew 4.0.4+e1-6308~48~ubuntu16.04.1-stable)
   (general
     (links 64)
-    (no_connects 57)
+    (no_connects 39)
     (area 81.575 43.765 212.555001 67.945)
     (thickness 1.6)
     (drawings 0)
-    (tracks 94)
+    (tracks 103)
     (zones 0)
     (modules 33)
@@
     )
   )
-  (segment (start 96.52 53.34) (end 88.9 53.34) (width 2) (layer B.Cu) (net 1))
+  (segment (start 94.996 57.15) (end 96.52 57.15) (width 0.25) (layer B.Cu) (net 1))
+  (segment (start 96.52 57.15) (end 96.774 57.404) (width 0.25) (layer B.Cu) (net 1))
+  (segment (start 93.98 56.134) (end 94.996 57.15) (width 0.25) (layer B.Cu) (net 1))
+  (segment (start 93.98 53.34) (end 88.9 53.34) (width 2) (layer B.Cu) (net 1))
+  (segment (start 96.52 53.34) (end 93.98 53.34) (width 2) (layer B.Cu) (net 1))
+  (segment (start 93.98 53.34) (end 93.98 56.134) (width 0.25) (layer B.Cu) (net 1))
+  (segment (start 100.41 62.23) (end 100.41 64.67) (width 0.25) (layer F.Cu) (net 2))
+  (segment (start 100.41 64.67) (end 100.31 64.77) (width 0.25) (layer F.Cu) (net 2))
   (segment (start 208.28 60.84) (end 89.154619 60.84) (width 2) (layer B.Cu) (net 2))
   (segment (start 89.154619 60.84) (end 88.72216 60.407541) (width 2) (layer B.Cu) (net 2))
@@
   (segment (start 190.083017 59.846983) (end 190.083017 56.181254) (width 0.4) (layer F.Cu) (net 2))
   (segment (start 186.606763 52.705) (end 185.26 52.705) (width 0.4) (layer F.Cu) (net 2))
+  (segment (start 97.71 62.23) (end 97.71 64.67) (width 0.25) (layer F.Cu) (net 3))
+  (segment (start 97.71 64.67) (end 97.81 64.77) (width 0.25) (layer F.Cu) (net 3))
   (segment (start 149.86 53.34) (end 148.96 53.34) (width 0.25) (layer F.Cu) (net 4))
   (segment (start 148.96 53.34) (end 147.175117 51.555117) (width 0.25) (layer F.Cu) (net 4))

Commit message: test
Parts:
- removed Q1: IRFB7537PbF, KiCad-Dev:TO-220_Horizontal_LargePads_HeatsinkPad
- added P5: CONN_01X02, Pin_Headers:Pin_Header_Straight_1x02, F.Cu at (88.9, 41.9)
- added P6: CONN_01X03, Pin_Headers:Pin_Header_Straight_1x03, F.Cu at (130.8, 36.8)
- added P7: CONN_01X01, Pin_Headers:Pin_Header_Straight_1x01, F.Cu at (95.2, 41.9)
- added P8: CONN_01X01, Pin_Headers:Pin_Header_Straight_1x01, F.Cu at (105.4, 44.5)
- added Q2: BUK9Y4R8-60E, TO_SOT_Packages_SMD:SOT-669_LFPAK, B.Cu at (131.4, 54.6)
- C3: footprint Capacitors_ThroughHole:C_Radial_D5_L6_P2.5 -> Capacitors_SMD:C_0805_HandSoldering
- D1, D2, D3, D4, D5: footprint Discret:D3 -> Diodes_SMD:SOD-123
- F6: moved to B.Cu
- moved P1 58.4 mm to (149.9, 59.7)
- moved F6 48.3 mm to (116.8, 54.6)
- moved C1 33.0 mm to (102.9, 27.9)
- moved C3 33.0 mm to (188.0, 27.9)
- moved U1 33.0 mm to (100.0, 25.4)
- moved C2 33.0 mm to (99.1, 31.8)
- moved R2 33.0 mm to (99.1, 29.2)
- moved U5 33.0 mm to (179.1, 26.7)
- moved U6 33.0 mm to (182.9, 26.7)
- moved U7 33.0 mm to (188.0, 17.8)
- moved P4 31.9 mm to (152.4, 24.1)
- moved F5 29.9 mm to (99.1, 67.3)
- moved D8 29.9 mm to (111.8, 67.3)
- moved U4 29.9 mm to (106.7, 67.3), turned to 0 degrees
- moved F3 29.6 mm to (99.1, 63.5)
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Routing:
- net /channel/GND: track 146.2 -> 26.4 mm
- net /channel/fuse/in+: track 84.4 -> 0.00 mm
- net /channel/out+: track 85.4 -> 25.5 mm
- net /channel/kill_sw/enable: track 58.7 -> 3.03 mm
- net /channel/kill_sw/in+: track 66.7 -> 16.0 mm
- net /channel/kill_sw/enabled1_3.3v: track 46.1 -> 3.62 mm
- net Net-(P4-Pad1): track 18.6 -> 0.00 mm
- net /channel/in+: track 13.7 -> 0.00 mm
- net Net-(D4-Pad1): track 0.00 -> 11.6 mm
- net Net-(D5-Pad1): track 0.00 -> 11.4 mm
- net Net-(D2-Pad1): track 0.00 -> 11.4 mm
- net Net-(D3-Pad1): track 0.00 -> 11.4 mm
- net Net-(D1-Pad1): track 0.00 -> 11.4 mm
- net /channel/fuse/enabled2_3.3v: track 8.48 -> 0.00 mm
- net /channel/kill_sw/enabled2_3.3v: track 8.05 -> 0.00 mm
- added copper zone on B.Cu, net /channel/GND
- added copper zone on B.Cu, net /channel/fuse/in+
- added copper zone on B.Cu, net /channel/in+
- added copper zone on B.Cu, net /channel/kill_sw/in+
- added copper zone on B.Cu, net /channel/out+

Commit message: test
Parts:
- removed D1: 15v, Diodes_SMD:SOD-123
- removed D2, D3, D4, D5: 3.3v, Diodes_SMD:SOD-123
- removed D8: LED, LEDs:LED_0805
- removed F1, F2, F3, F4, F5: FUSE, Fuse_Holders_and_Fuses:Fuse_SMD1206_HandSoldering
- removed P5: CONN_01X02, Pin_Headers:Pin_Header_Straight_1x02
- removed P6: CONN_01X03, Pin_Headers:Pin_Header_Straight_1x03
- removed P7, P8: CONN_01X01, Pin_Headers:Pin_Header_Straight_1x01
- removed U4: NSI45020AT1G, Diodes_SMD:SOD-123
- removed U5: LM3480-5.0, TO_SOT_Packages_SMD:SOT-23
- removed U6: 74LVC1G08, TO_SOT_Packages_SMD:SOT-353
- C3: value C -> CP; footprint Capacitors_SMD:C_0805_HandSoldering -> Capacitors_ThroughHole:C_Radial_D5_L6_P2.5
- P4: value CONN_01X02 -> CONN_02X03; footprint Pin_Headers:Pin_Header_Straight_1x02 -> Pin_Headers:Pin_Header_Straight_2x03
- moved C3 51.8 mm to (144.8, 56.5), turned to 270 degrees
- moved U7 51.2 mm to (152.4, 54.6)
- moved P3 36.9 mm to (88.9, 61.0), turned to 90 degrees
- moved P4 36.6 mm to (139.7, 58.4), turned to 270 degrees
- moved C1 36.0 mm to (85.1, 59.3)
- moved R2 35.5 mm to (80.2, 59.3), turned to 270 degrees
- moved U1 33.4 mm to (83.8, 54.6)
- moved C2 32.1 mm to (82.5, 59.3), turned to 270 degrees
- moved Q2 21.1 mm to (152.6, 54.6)
- moved R1 15.2 mm to (83.8, 54.6)
- moved P1 15.2 mm to (165.1, 59.7)
- moved D7 13.1 mm to (100.3, 62.2), turned to 90 degrees
- moved D9 12.0 mm to (105.4, 62.2), turned to 90 degrees
- moved P2 11.4 mm to (72.4, 59.7)
- moved D6 9.25 mm to (102.9, 62.2), turned to 90 degrees
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Connections:
- C3 pad 1: /channel/GND -> /channel/kill_sw/in+
- C3 pad 2: /channel/kill_sw/in+ -> /channel/GND
- P3 pad 2: Net-(D5-Pad1) -> /channel/current_sensor/sense
- P3 pad 3: Net-(D1-Pad1) -> (no net)
- P3 pad 4: Net-(D4-Pad1) -> /channel/kill_sw/enabled2_3.3v
- P3 pad 5: Net-(D2-Pad1) -> /channel/fuse/enabled2_3.3v
- P3 pad 6: Net-(D3-Pad1) -> (no net)
- P4 pad 1: Net-(P4-Pad1) -> /channel/GND
- P4 pad 2: /channel/kill_sw/in+ -> Net-(P4-Pad2)
- U7 pad 2: Net-(U6-Pad4) -> Net-(P4-Pad2)
Routing:
- net /channel/in+: track 0.00 -> 27.7 mm, vias 0 -> 1
- net /channel/current_sensor/sense: track 2.58 -> 17.9 mm, vias 0 -> 1
- net Net-(P4-Pad2): track 0.00 -> 15.3 mm
- net /channel/out+: track 25.5 -> 13.1 mm, vias 0 -> 1
- net /channel/kill_sw/in+: track 16.0 -> 4.28 mm, vias 0 -> 1
- net Net-(D4-Pad1): track 11.6 -> 0.00 mm
- net Net-(D5-Pad1): track 11.4 -> 0.00 mm
- net Net-(D2-Pad1): track 11.4 -> 0.00 mm
- net Net-(D3-Pad1): track 11.4 -> 0.00 mm
- net Net-(D1-Pad1): track 11.4 -> 0.00 mm
- net Net-(U6-Pad4): track 9.82 -> 0.00 mm
- net /channel/GND: track 26.4 -> 33.6 mm, vias 0 -> 1
- net /channel/fuse/in+: track 0.00 -> 5.91 mm, vias 0 -> 1
- net Net-(U5-Pad1): track 4.36 -> 0.00 mm
- net /channel/kill_sw/enabled1_3.3v: track 3.62 -> 0.00 mm
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Other:
- board outline added: 116.8 x 45.7 mm

Commit message: test
Parts:
- added P5: CONN_01X03, Pin_Headers:Pin_Header_Straight_1x03, F.Cu at (149.9, 59.7)
- added P6: CONN_XT60, KiCad-Dev:XT60, F.Cu at (175.3, 59.7)
- added P7: CONN_XT60, KiCad-Dev:XT60, F.Cu at (185.4, 59.7)
- added P8: CONN_XT60, KiCad-Dev:XT60, F.Cu at (195.6, 59.7)
- added R3: R, Resistors_SMD:R_0603, F.Cu at (141.6, 64.8)
- added R4: R, Resistors_SMD:R_0603, F.Cu at (139.7, 64.8)
- added U4: 74LVC1G08, TO_SOT_Packages_SMD:SOT-353, F.Cu at (141.0, 61.0)
- C1, C2: footprint Capacitors_SMD:C_0805_HandSoldering -> Capacitors_SMD:C_0603
- R2: footprint Resistors_SMD:R_0805_HandSoldering -> Resistors_SMD:R_0603
- moved P4 8.03 mm to (132.1, 61.0), turned to 90 degrees
- moved F6 2.54 mm to (119.4, 54.6)
- moved D9 1.80 mm to (106.7, 63.5)
- moved D7 1.80 mm to (99.1, 63.5)
- moved U8 1.27 mm to (106.7, 55.9)
- moved D6 1.27 mm to (102.9, 63.5)
- moved U3 1.27 mm to (99.1, 55.9)
Connections:
- P3 pad 3: (no net) -> /channel/kill_sw/enabled2_3.3v
- P3 pad 4: /channel/kill_sw/enabled2_3.3v -> /channel/fuse/enabled1_3.3v
- P3 pad 5: /channel/fuse/enabled2_3.3v -> /channel/kill_sw/enable
- P3 pad 6: (no net) -> /channel/fuse/enabled2_3.3v
- P4 pad 2: Net-(P4-Pad2) -> (no net)
- P4 pad 5: (no net) -> Net-(P4-Pad5)
- P4 pad 6: (no net) -> Net-(P4-Pad6)
- U7 pad 2: Net-(P4-Pad2) -> Net-(P5-Pad2)
Routing:
- net /channel/out+: track 13.1 -> 76.7 mm
- net /channel/kill_sw/enable: track 0.00 -> 49.3 mm, vias 0 -> 1
- net /channel/kill_sw/in+: track 4.28 -> 51.0 mm, vias 1 -> 2
- net /channel/kill_sw/enabled2_3.3v: track 0.00 -> 35.9 mm
- net /channel/fuse/enabled1_3.3v: track 0.00 -> 25.3 mm
- net /channel/GND: track 33.6 -> 57.0 mm, vias 1 -> 2
- net /channel/fuse/enabled2_3.3v: track 0.00 -> 16.5 mm
- net Net-(P4-Pad2): track 15.3 -> 0.00 mm
- net Net-(P5-Pad1): track 0.00 -> 10.9 mm, vias 0 -> 1
- net Net-(P5-Pad2): track 0.00 -> 7.64 mm
- net Net-(P4-Pad5): track 0.00 -> 7.13 mm
- net Net-(P4-Pad6): track 0.00 -> 4.13 mm
- net /channel/fuse/in+: track 5.91 -> 7.54 mm, vias 1 -> 2
- net /channel/in+: track 27.7 -> 28.8 mm
Other:
- board outline removed

Commit message: test
Parts:
- removed R3, R4: R, Resistors_SMD:R_0603
- removed U4: 74LVC1G08, TO_SOT_Packages_SMD:SOT-353
- moved P5 21.6 mm to (128.3, 59.7), turned to 270 degrees
- moved C3 1.95 mm to (144.8, 58.5)
- moved P4 1.27 mm to (133.3, 61.0)
Connections:
- P4 pad 2: (no net) -> Net-(P4-Pad2)
- P4 pad 4: (no net) -> /channel/kill_sw/enable
- P4 pad 5: Net-(P4-Pad5) -> (no net)
- P4 pad 6: Net-(P4-Pad6) -> (no net)
- P5 pad 1: Net-(P5-Pad1) -> Net-(P4-Pad2)
Routing:
- net Net-(P5-Pad2): track 7.64 -> 26.6 mm
- net /channel/GND: track 57.0 -> 39.6 mm
- net Net-(P5-Pad1): track 10.9 -> 0.00 mm, vias 1 -> 0
- net /channel/kill_sw/in+: track 51.0 -> 42.5 mm
- net Net-(P4-Pad5): track 7.13 -> 0.00 mm
- net /channel/out+: track 76.7 -> 69.8 mm
- net /channel/kill_sw/enable: track 49.3 -> 43.2 mm, vias 1 -> 0
- net Net-(P4-Pad2): track 0.00 -> 5.61 mm
- net Net-(P4-Pad6): track 4.13 -> 0.00 mm
- net /channel/fuse/in+: track 7.54 -> 9.56 mm
Other:
- board outline added: 142.2 x 17.8 mm
- board text added: "Controll A"
- board text added: "Controll B"
- board text added: "FET Driver"
- board text added: "Sensor"
- board text added: "Status"
