File: pdb1/pdb1.kicad_pcb (KiCad board)
At the start: 2 copper layers, 142.2 x 17.8 mm, 23 parts, among them P1 CONN_XT60, P2 CONN_XT60, P3 CONN_02X03, P4 CONN_02X03, P5 CONN_01X03, P6 CONN_XT60, P7 CONN_XT60, P8 CONN_XT60, Q2 BUK9Y4R8-60E, U1 INA169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

Commit message: test
Parts:
- moved D6 3.81 mm to (99.1, 63.5)
- moved D7 3.81 mm to (102.9, 63.5)
- moved U2 3.81 mm to (99.1, 55.9)
- moved U3 3.81 mm to (102.9, 55.9)
Connections:
- P3 pad 4: /channel/fuse/enabled1_3.3v -> /channel/fuse/enabled2_3.3v
- P3 pad 6: /channel/fuse/enabled2_3.3v -> /channel/fuse/enabled1_3.3v
Routing:
- net /channel/fuse/enabled1_3.3v: track 25.3 -> 14.1 mm
- net /channel/fuse/enabled2_3.3v: track 16.5 -> 24.9 mm
- net /channel/fuse/in+: track 9.56 -> 11.4 mm
- net /channel/kill_sw/in+: track 42.5 -> 44.2 mm, vias 2 -> 1
- net /channel/in+: track 28.8 -> 27.7 mm
- net /channel/out+: track 69.8 -> 69.0 mm
Other:
- board text added: "Battery Input"
- board text added: "Battery Output"
- board text added: "Curr sens"
- board text added: "Current Sense"
- board text added: "Enb"
- board text added: "GND"
- board text added: "NC"
- board text added: "P3 Enb"
- board text added: "P4 Enb"
- board text added: "P5 Enb"
- board text added: "PWR 1"
- board text added: "PWR 2"
- board text added: "PWR 3"
- board text added: "Sig"
- board text added: "VCC0"
- board text added: "VCC1"
- board text added: "VCC1 PWR"
- board text added: "VCC2"
- board text added: "VCC2 PWR"
- board text added: "VCC3"
- board text added: "VCC3 PWR"
- board text removed: "Sensor"
- board text removed: "Status"

Commit message: test
Routing:
- net /channel/in+: track 27.7 -> 31.3 mm
- net Net-(Q2-Pad4): track 4.48 -> 5.67 mm
- net /channel/fuse/in+: track 11.4 -> 12.3 mm
Other:
- net class Default: via_dia 0.6 -> 1; via_drill 0.4 -> 0.8
Changed lines of the file:
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@@
-(kicad_pcb (version 4) (host pcbnew 4.0.4-stable)
+(kicad_pcb (version 4) (host pcbnew 4.0.4+e1-6308~48~ubuntu16.04.1-stable)
   (general
     (links 51)
@@
     (thickness 1.6)
     (drawings 58)
-    (tracks 119)
+    (tracks 122)
     (zones 0)
     (modules 23)
@@
     (segment_width 0.2)
     (edge_width 0.7)
-    (via_size 0.6)
-    (via_drill 0.4)
+    (via_size 1)
+    (via_drill 0.8)
     (via_min_size 0.4)
     (via_min_drill 0.3)
@@
     (clearance 0.2)
     (trace_width 0.25)
-    (via_dia 0.6)
-    (via_drill 0.4)
+    (via_dia 1)
+    (via_drill 0.8)
     (uvia_dia 0.3)
     (uvia_drill 0.1)
@@
   (gr_line (start 205.74 50.8) (end 205.74 68.58) (layer Edge.Cuts) (width 0.7))
   (segment (start 102.861339 55.888661) (end 102.867466 55.894788) (width 0.5) (layer B.Cu) (net 0))
-  (segment (start 84.77 56.769) (end 90.09998 56.769) (width 0.5) (layer F.Cu) (net 1))
-  (segment (start 90.398599 52.248087) (end 82.8675 52.248087) (width 0.5) (layer F.Cu) (net 1))
-  (segment (start 91.184452 53.03394) (end 90.398599 52.248087) (width 0.5) (layer F.Cu) (net 1))
-  (segment (start 91.184452 55.684528) (end 91.184452 53.03394) (width 0.5) (layer F.Cu) (net 1))
-  (segment (start 90.09998 56.769) (end 91.184452 55.684528) (width 0.5) (layer F.Cu) (net 1))
+  (segment (start 84.77 56.769) (end 91.520335 56.769) (width 0.5) (layer F.Cu) (net 1))
+  (segment (start 91.520335 56.769) (end 92.267073 56.022262) (width 0.5) (layer F.Cu) (net 1))
+  (segment (start 92.267073 52.831438) (end 91.683722 52.248087) (width 0.5) (layer F.Cu) (net 1))
+  (segment (start 92.267073 56.022262) (end 92.267073 52.831438) (width 0.5) (layer F.Cu) (net 1))
+  (segment (start 91.683722 52.248087) (end 82.8675 52.248087) (width 0.5) (layer F.Cu) (net 1))
+  (segment (start 77.939278 54.101997) (end 77.439279 54.601996) (width 0.5) (layer F.Cu) (net 1))
+  (segment (start 79.793188 52.248087) (end 77.939278 54.101997) (width 0.5) (layer F.Cu) (net 1))
+  (segment (start 82.8675 52.248087) (end 79.793188 52.248087) (width 0.5) (layer F.Cu) (net 1))
+  (via (at 77.439279 54.601996) (size 1) (drill 0.8) (layers F.Cu B.Cu) (net 1))
   (segment (start 84.77 56.769) (end 84.77 57.2135) (width 0.5) (layer F.Cu) (net 1))
   (segment (start 84.77 55.71) (end 84.77 56.769) (width 0.5) (layer F.Cu) (net 1))
-  (segment (start 78.044102 52.350562) (end 77.744103 52.650561) (width 0.5) (layer F.Cu) (net 1))
-  (segment (start 78.146577 52.248087) (end 78.044102 52.350562) (width 0.5) (layer F.Cu) (net 1))
-  (segment (start 82.8675 52.248087) (end 78.146577 52.248087) (width 0.5) (layer F.Cu) (net 1))
-  (via (at 77.744103 52.650561) (size 0.6) (drill 0.4) (layers F.Cu B.Cu) (net 1))
   (segment (start 82.87 53.51) (end 82.87 52.48) (width 0.5) (layer F.Cu) (net 1))
   (segment (start 82.8675 52.4775) (end 82.8675 52.248087) (width 0.5) (layer F.Cu) (net 1))
@@
   (segment (start 84.215 60.001086) (end 84.208586 60.0075) (width 0.5) (layer F.Cu) (net 2))
   (segment (start 84.208586 60.0075) (end 83.82 60.0075) (width 0.5) (layer F.Cu) (net 2))
-  (via (at 83.82 63.754) (size 0.6) (drill 0.4) (layers F.Cu B.Cu) (net 2))
+  (via (at 83.82 63.754) (size 1) (drill 0.8) (layers F.Cu B.Cu) (net 2))
   (segment (start 96.575773 64.54902) (end 96.574716 64.547963) (width 0.6) (layer F.Cu) (net 2))
   (segment (start 99.06 64.54902) (end 96.575773 64.54902) (width 0.6) (layer F.Cu) (net 2))
-  (via (at 96.574716 64.547963) (size 0.6) (drill 0.4) (layers F.Cu B.Cu) (net 2))
+  (via (at 96.574716 64.547963) (size 1) (drill 0.8) (layers F.Cu B.Cu) (net 2))
   (segment (start 102.87 64.54902) (end 99.06 64.54902) (width 0.6) (layer F.Cu) (net 2))
   (segment (start 106.68 64.54902) (end 102.87 64.54902) (width 0.6) (layer F.Cu) (net 2))
@@
   (segment (start 78.105 58.42) (end 88.330002 58.42) (width 0.4) (layer B.Cu) (net 3))
   (segment (start 88.330002 58.42) (end 88.9 58.42) (width 0.4) (layer B.Cu) (net 3))
-  (via (at 78.105 58.42) (size 0.6) (drill 0.4) (layers F.Cu B.Cu) (net 3))
+  (via (at 78.105 58.42) (size 1) (drill 0.8) (layers F.Cu B.Cu) (net 3))
   (segment (start 102.87 57.515) (end 102.87 56.179998) (width 0.5) (layer F.Cu) (net 4))
   (segment (start 102.87 56.179998) (end 106.284563 52.765435) (width 0.5) (layer F.Cu) (net 4))
@@
   (segment (start 152.1 54.61) (end 149.9 54.61) (width 0.4) (layer B.Cu) (net 4))
   (segment (start 149.7 52.705) (end 145.415 52.705) (width 0.6) (layer F.Cu) (net 4))
-  (via (at 145.415 52.705) (size 0.6) (drill 0.4) (layers F.Cu B.Cu) (net 4))
+  (via (at 145.415 52.705) (size 1) (drill 0.8) (layers F.Cu B.Cu) (net 4))
   (segment (start 97.044609 60.435589) (end 97.044609 58.42) (width 0.5) (layer F.Cu) (net 5))
   (segment (start 97.044609 58.42) (end 97.044609 56.260391) (width 0.5) (layer F.Cu) (net 5))
@@
   (segment (start 92.911879 66.241879) (end 91.44 64.77) (width 0.5) (layer F.Cu) (net 7))
   (segment (start 91.44 64.77) (end 91.44 60.96) (width 0.5) (layer F.Cu) (net 7))
+  (segment (start 90.131328 54.160988) (end 90.631327 54.660987) (width 0.5) (layer F.Cu) (net 8))
+  (segment (start 89.48034 53.51) (end 90.131328 54.160988) (width 0.5) (layer F.Cu) (net 8))
+  (segment (start 84.77 53.51) (end 89.48034 53.51) (width 0.5) (layer F.Cu) (net 8))
+  (via (at 90.631327 54.660987) (size 1) (drill 0.8) (layers F.Cu B.Cu) (net 8))
   (segment (start 99.06 59.69) (end 99.06 55.88) (width 0.5) (layer B.Cu) (net 8))
   (segment (start 99.06 57.515) (end 99.06 59.69) (width 0.5) (layer F.Cu) (net 8))
-  (via (at 99.06 59.69) (size 0.6) (drill 0.4) (layers F.Cu B.Cu) (net 8))
-  (segment (start 90.198965 53.51) (end 90.211015 53.49795) (width 0.5) (layer F.Cu) (net 8))
-  (segment (start 84.77 53.51) (end 90.198965 53.51) (width 0.5) (layer F.Cu) (net 8))
-  (via (at 90.211015 53.49795) (size 0.6) (drill 0.4) (layers F.Cu B.Cu) (net 8))
-  (segment (start 158.75 58.42) (end 154.381826 58.42) (width 0.5) (layer F.Cu) (net 9))
+  (via (at 99.06 59.69) (size 1) (drill 0.8) (layers F.Cu B.Cu) (net 8))
+  (segment (start 158.75 58.42) (end 160.655 56.515) (width 0.5) (layer B.Cu) (net 9))
+  (segment (start 154.25 58.42) (end 151.075 55.245) (width 0.5) (layer F.Cu) (net 9))
+  (segment (start 158.75 58.42) (end 154.25 58.42) (width 0.5) (layer F.Cu) (net 9))
+  (segment (start 151.075 55.245) (end 149.7 55.245) (width 0.5) (layer F.Cu) (net 9))
+  (segment (start 111.814097 62.649097) (end 106.68 57.515) (width 0.5) (layer F.Cu) (net 9))
   (segment (start 150.152729 62.649097) (end 111.814097 62.649097) (width 0.5) (layer F.Cu) (net 9))
   (segment (start 154.381826 58.42) (end 150.152729 62.649097) (width 0.5) (layer F.Cu) (net 9))
-  (segment (start 111.814097 62.649097) (end 106.68 57.515) (width 0.5) (layer F.Cu) (net 9))
-  (segment (start 158.75 58.42) (end 154.25 58.42) (width 0.5) (layer F.Cu) (net 9))
-  (segment (start 154.25 58.42) (end 151.075 55.245) (width 0.5) (layer F.Cu) (net 9))
-  (segment (start 151.075 55.245) (end 149.7 55.245) (width 0.5) (layer F.Cu) (net 9))
-  (segment (start 158.75 58.42) (end 160.655 56.515) (width 0.5) (layer B.Cu) (net 9))
-  (via (at 158.75 58.42) (size 0.6) (drill 0.4) (layers F.Cu B.Cu) (net 9))
-  (segment (start 157.48 56.515) (end 155.375 56.515) (width 0.6) (layer B.Cu) (net 10))
-  (segment (start 155.1 56.515) (end 157.48 56.515) (width 0.6) (layer F.Cu) (net 10))
-  (via (at 157.48 56.515) (size 0.6) (drill 0.4) (layers F.Cu B.Cu) (net 10))
+  (segment (start 158.75 58.42) (end 154.381826 58.42) (width 0.5) (layer F.Cu) (net 9))
+  (via (at 158.75 58.42) (size 1) (drill 0.8) (layers F.Cu B.Cu) (net 9))
+  (segment (start 157.635538 56.515) (end 157.945139 56.824601) (width 0.6) (layer F.Cu) (net 10))
+  (segment (start 155.1 56.515) (end 157.635538 56.515) (width 0.6) (layer F.Cu) (net 10))
+  (segment (start 157.635538 56.515) (end 157.945139 56.824601) (width 0.6) (layer B.Cu) (net 10))
+  (segment (start 155.375 56.515) (end 157.635538 56.515) (width 0.6) (layer B.Cu) (net 10))
+  (via (at 157.945139 56.824601) (size 1) (drill 0.8) (layers F.Cu B.Cu) (net 10))
   (segment (start 93.98 60.96) (end 129.746733 60.96) (width 0.4) (layer B.Cu) (net 11))
   (segment (start 129.746733 60.96) (end 130.964502 59.742231) (width 0.4) (layer B.Cu) (net 11))

Commit message: test
Parts:
- removed P1, P7, P8: CONN_XT60, KiCad-Dev:XT60
- P3, P4: footprint Pin_Headers:Pin_Header_Straight_2x03 -> KiCad-Dev:Pin_Header_Straight_2x03_box
- moved P6 35.6 mm to (139.7, 59.7)
- moved Q2 23.7 mm to (128.9, 54.6)
- moved U7 22.9 mm to (129.5, 54.6)
- moved P5 21.6 mm to (106.7, 59.7)
- moved F6 20.3 mm to (99.1, 54.6)
- moved C3 17.2 mm to (127.6, 59.8)
- moved P4 16.6 mm to (116.8, 59.7)
- moved C1 12.7 mm to (72.4, 59.3)
- moved C2 12.7 mm to (69.8, 59.3)
- moved R2 12.7 mm to (67.5, 59.3)
- moved R1 12.7 mm to (71.1, 54.6)
- moved U1 12.7 mm to (71.1, 54.6)
- moved P2 11.4 mm to (61.0, 59.7)
- moved U2 10.2 mm to (90.2, 61.0)
- moved U3 10.2 mm to (94.0, 61.0)
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Routing:
- net /channel/kill_sw/in+: track 44.2 -> 27.4 mm, vias 1 -> 2
- net /channel/out+: track 69.0 -> 56.7 mm
- net /channel/kill_sw/enable: track 43.2 -> 34.2 mm
- net /channel/kill_sw/enabled2_3.3v: track 36.2 -> 41.9 mm, vias 0 -> 1
- net /channel/fuse/in+: track 12.3 -> 15.5 mm
- net Net-(P4-Pad2): track 5.61 -> 8.15 mm
- net /channel/fuse/enabled1_3.3v: track 14.1 -> 16.4 mm, vias 0 -> 1
- net /channel/current_sensor/sense: track 18.2 -> 19.9 mm
- net Net-(Q2-Pad4): track 5.67 -> 4.34 mm
- net /channel/fuse/enabled2_3.3v: track 24.9 -> 24.1 mm, vias 0 -> 1
- net Net-(P5-Pad2): track 26.6 -> 26.1 mm, vias 0 -> 1
- net /channel/GND: track 39.9 -> 40.0 mm, vias 2 -> 3
Other:
- board size 142.2 x 17.8 mm -> 97.8 x 17.8 mm
- net class Default: via_dia 1 -> 1.4; via_drill 0.8 -> 1.2
- board text added: "CAO"
- board text added: "Fuse"
- board text added: "VC1"
- board text added: "VC2"
- board text added: "VC3"
- board text removed: "Battery Output"
- board text removed: "Curr sens"
- board text removed: "P3 Enb"
- board text removed: "P4 Enb"
- board text removed: "PWR 1"
- board text removed: "PWR 2"
- board text removed: "PWR 3"
- board text removed: "VCC1 PWR"
- board text removed: "VCC2 PWR"
- board text removed: "VCC3 PWR"

Commit message: test
Other:
- board text added: "+ Rail"
- board text added: "Battery Out"
- board text added: "Fused"
- board text added: "GND Rail"
Changed lines of the file:
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@@
     (area 51.719999 50.449999 150.210001 68.930001)
     (thickness 1.6)
-    (drawings 71)
+    (drawings 78)
     (tracks 154)
     (zones 0)
@@
     (pad 6 thru_hole oval (at 1.27 2.54 90) (size 1.1 2) (drill 1.016) (layers *.Cu *.Mask))
   )
+  (gr_text Fused (at 132.715 51.435) (layer F.SilkS)
+    (effects (font (size 0.6 0.6) (thickness 0.15)))
+  )
+  (gr_text "Current Sense" (at 95.25 51.435) (layer F.SilkS)
+    (effects (font (size 0.6 0.6) (thickness 0.15)))
+  )
+  (gr_line (start 57.15 50.8) (end 57.15 68.58) (layer F.SilkS) (width 0.2))
+  (gr_text "+ Rail" (at 54.61 51.435) (layer F.SilkS)
+    (effects (font (size 0.6 0.6) (thickness 0.15)))
+  )
+  (gr_text "GND Rail" (at 147.32 51.435) (layer F.SilkS)
+    (effects (font (size 0.6 0.6) (thickness 0.15)))
+  )
+  (gr_line (start 144.145 68.58) (end 144.145 50.8) (layer F.SilkS) (width 0.2))
+  (gr_text "Battery Out" (at 140.97 51.435) (layer F.SilkS)
+    (effects (font (size 0.6 0.6) (thickness 0.15)))
+  )
   (gr_text Fuse (at 93.98 57.785) (layer F.SilkS)
     (effects (font (size 0.6 0.6) (thickness 0.15)))
@@
   (gr_line (start 118.11 64.135) (end 118.11 65.405) (layer F.SilkS) (width 0.2))
   (gr_line (start 115.57 64.135) (end 115.57 65.405) (layer F.SilkS) (width 0.2))
-  (gr_text VCC3 (at 135.89 51.435) (layer F.SilkS)
+  (gr_text VCC3 (at 136.525 51.435) (layer F.SilkS)
     (effects (font (size 0.6 0.6) (thickness 0.15)))
   )
   (gr_line (start 109.22 57.15) (end 99.695 57.15) (layer F.SilkS) (width 0.2))
   (gr_line (start 99.695 68.58) (end 99.695 57.15) (layer F.SilkS) (width 0.2))
-  (gr_line (start 133.985 50.8) (end 133.985 68.58) (layer F.SilkS) (width 0.2))
+  (gr_line (start 134.62 50.8) (end 134.62 68.58) (layer F.SilkS) (width 0.2))
   (gr_line (start 124.46 68.58) (end 124.46 52.07) (layer F.SilkS) (width 0.2))
   (gr_text VCC1 (at 90.17 67.945) (layer F.SilkS)
@@
     (effects (font (size 0.6 0.6) (thickness 0.15)))
   )
-  (gr_text VCC0 (at 53.975 51.435) (layer F.SilkS)
+  (gr_text VCC0 (at 59.055 51.435) (layer F.SilkS)
     (effects (font (size 0.6 0.6) (thickness 0.15)))
   )
@@
     (effects (font (size 1 1) (thickness 0.2)))
   )
-  (gr_text "FET Driver" (at 128.905 67.31) (layer F.SilkS)
+  (gr_text "FET Driver" (at 129.54 67.31) (layer F.SilkS)
     (effects (font (size 1 1) (thickness 0.2)))
   )

Commit message: test
Parts:
- removed P6: CONN_XT60, KiCad-Dev:XT60
- added P1: CONN_XT60, KiCad-Dev:XT60, F.Cu at (139.7, 59.7)
- added U4: LM3480-3.3, TO_SOT_Packages_SMD:SOT-23, B.Cu at (120.7, 59.7)
- added U5: 74LVC1G08, TO_SOT_Packages_SMD:SOT-353, F.Cu at (120.7, 59.7)
- P4: value CONN_02X03 -> CONN_01X02; footprint KiCad-Dev:Pin_Header_Straight_2x03_box -> Pin_Headers:Pin_Header_Straight_1x02
- P5: value CONN_01X03 -> CONN_01X02; footprint Pin_Headers:Pin_Header_Straight_1x03 -> Pin_Headers:Pin_Header_Straight_1x02
- moved P4 1.27 mm to (115.6, 59.7), turned to 270 degrees
- turned P5 to 90 degrees
Connections:
- P4 pad 1: /channel/GND -> Net-(P4-Pad1)
- P5 pad 1: Net-(P4-Pad2) -> /channel/kill_sw/enable
- P5 pad 2: Net-(P5-Pad2) -> Net-(P4-Pad2)
- U7 pad 2: Net-(P5-Pad2) -> Net-(U5-Pad4)
Routing:
- net Net-(P5-Pad2): track 26.1 -> 0.00 mm, vias 1 -> 0
- net Net-(P4-Pad1): track 0.00 -> 11.5 mm
- net Net-(U5-Pad4): track 0.00 -> 8.55 mm
- net /channel/GND: track 40.0 -> 47.7 mm
- net /channel/kill_sw/enable: track 34.2 -> 41.0 mm
- net Net-(P4-Pad2): track 8.15 -> 12.8 mm
- net /channel/kill_sw/enabled2_3.3v: track 41.9 -> 39.5 mm
- net /channel/kill_sw/in+: track 27.4 -> 28.3 mm

Commit message: test
Parts:
- added R3: R, Resistors_SMD:R_0603, F.Cu at (123.8, 62.9)
- added R4: R, Resistors_SMD:R_0603, F.Cu at (123.8, 60.3)
- moved P2 1.27 mm to (59.7, 59.7)
- moved C3 0.64 mm to (128.3, 59.8)
Routing:
- net /channel/in+: track 31.3 -> 40.7 mm
- net Net-(P4-Pad2): track 12.8 -> 18.9 mm, vias 0 -> 1
- net /channel/kill_sw/enable: track 41.0 -> 46.8 mm, vias 0 -> 1
- net /channel/kill_sw/in+: track 28.3 -> 31.8 mm
- net /channel/out+: track 56.4 -> 54.8 mm
- net Net-(P4-Pad1): track 11.5 -> 13.1 mm, vias 0 -> 1
- net /channel/GND: track 47.7 -> 49.0 mm
- net Net-(Q2-Pad4): track 4.34 -> 5.37 mm
- net /channel/fuse/in+: track 15.5 -> 14.6 mm
- net /channel/fuse/enabled2_3.3v: track 24.5 -> 25.2 mm
Other:
- board size 97.8 x 17.8 mm -> 99.1 x 17.8 mm
- net class Default: via_dia 1.4 -> 2; via_drill 1.2 -> 1.4

Commit message: test
Routing:
- net /channel/current_sensor/sense: track 19.9 -> 22.3 mm
Changed lines of the file:
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@@
-(kicad_pcb (version 4) (host pcbnew 4.0.4-stable)
+(kicad_pcb (version 4) (host pcbnew 4.0.4+e1-6308~48~ubuntu16.04.1-stable)
   (general
     (links 54)
     (no_connects 0)
-    (area 50.449999 50.449999 150.210001 68.930001)
+    (area 50.449999 46.015 150.210001 68.930001)
     (thickness 1.6)
     (drawings 75)
-    (tracks 186)
+    (tracks 187)
     (zones 0)
     (modules 24)
@@
   )
   (setup
-    (last_trace_width 0.5)
+    (last_trace_width 0.25)
     (user_trace_width 0.3)
     (user_trace_width 0.4)
@@
   (segment (start 71.508586 60.0075) (end 71.12 60.0075) (width 0.5) (layer F.Cu) (net 2))
   (via (at 71.12 63.754) (size 2) (drill 1.4) (layers F.Cu B.Cu) (net 2))
-  (segment (start 78.74 58.42) (end 65.883551 58.42) (width 0.5) (layer B.Cu) (net 3))
-  (segment (start 65.883551 58.42) (end 65.815282 58.488269) (width 0.5) (layer B.Cu) (net 3))
-  (segment (start 67.484392 58.501086) (end 65.828099 58.501086) (width 0.4) (layer F.Cu) (net 3))
-  (segment (start 65.828099 58.501086) (end 65.815282 58.488269) (width 0.4) (layer F.Cu) (net 3))
-  (via (at 65.815282 58.488269) (size 2) (drill 1.4) (layers F.Cu B.Cu) (net 3))
+  (segment (start 65.624384 58.501086) (end 64.908756 59.216714) (width 0.4) (layer F.Cu) (net 3))
+  (segment (start 67.484392 58.501086) (end 65.624384 58.501086) (width 0.4) (layer F.Cu) (net 3))
+  (segment (start 65.70547 58.42) (end 64.908756 59.216714) (width 0.5) (layer B.Cu) (net 3))
+  (segment (start 78.74 58.42) (end 65.70547 58.42) (width 0.5) (layer B.Cu) (net 3))
+  (via (at 64.908756 59.216714) (size 2) (drill 1.4) (layers F.Cu B.Cu) (net 3))
   (segment (start 70.17 55.71) (end 70.17 58.181086) (width 0.4) (layer F.Cu) (net 3))
   (segment (start 70.17 58.181086) (end 69.85 58.501086) (width 0.4) (layer F.Cu) (net 3))
@@
   (via (at 113.137105 62.470628) (size 2) (drill 1.4) (layers F.Cu B.Cu) (net 12))
   (segment (start 109.22 59.69) (end 113.03 59.69) (width 0.3) (layer B.Cu) (net 12))
+  (segment (start 115.57 57.226029) (end 116.251041 56.544988) (width 0.4) (layer B.Cu) (net 13))
+  (segment (start 115.57 59.69) (end 115.57 57.226029) (width 0.4) (layer B.Cu) (net 13))
+  (segment (start 119.036735 56.544988) (end 117.665254 56.544988) (width 0.4) (layer F.Cu) (net 13))
+  (segment (start 119.283859 56.792112) (end 119.036735 56.544988) (width 0.4) (layer F.Cu) (net 13))
+  (segment (start 117.665254 56.544988) (end 116.251041 56.544988) (width 0.4) (layer F.Cu) (net 13))
+  (via (at 116.251041 56.544988) (size 2) (drill 1.4) (layers F.Cu B.Cu) (net 13))
   (segment (start 120.015 58.674) (end 120.015 57.523253) (width 0.3) (layer F.Cu) (net 13))
   (segment (start 120.015 57.523253) (end 119.283859 56.792112) (width 0.3) (layer F.Cu) (net 13))
-  (segment (start 119.283859 56.792112) (end 117.408322 56.792112) (width 0.4) (layer F.Cu) (net 13))
-  (segment (start 117.408322 56.792112) (end 115.994109 56.792112) (width 0.4) (layer F.Cu) (net 13))
-  (segment (start 115.57 57.216221) (end 115.994109 56.792112) (width 0.4) (layer B.Cu) (net 13))
-  (segment (start 115.57 59.69) (end 115.57 57.216221) (width 0.4) (layer B.Cu) (net 13))
-  (via (at 115.994109 56.792112) (size 2) (drill 1.4) (layers F.Cu B.Cu) (net 13))
   (segment (start 119.7 58.68924) (end 116.765659 58.68924) (width 0.5) (layer B.Cu) (net 13))
   (segment (start 116.765659 58.68924) (end 115.764899 59.69) (width 0.5) (layer B.Cu) (net 13))
