File: pdb1/_autosave-pdb1.kicad_pcb (KiCad board)
At the start: 2 copper layers, 142.2 x 17.8 mm, 23 parts, among them P1 CONN_XT60, P2 CONN_XT60, P3 CONN_02X03, P4 CONN_02X03, P5 CONN_01X03, P6 CONN_XT60, P7 CONN_XT60, P8 CONN_XT60, Q2 BUK9Y4R8-60E, U1 INA169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

Commit message: test
Other:
- board text added: "Controll C"
Changed lines of the file:
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@@
   )
   (gr_line (start 63.5 68.58) (end 205.74 68.58) (layer F.SilkS) (width 0.2))
-  (gr_text "Controll B" (at 135.89 67.31) (layer F.SilkS)
+  (gr_text "Controll C" (at 135.89 67.31) (layer F.SilkS)
     (effects (font (size 1 1) (thickness 0.2)))
   )
