File: pdb1/channel.sch (KiCad schematic (older format))
At the start: 5 parts

Commit message: test
Parts:
- added D3: 3.3v, Discret:D3, symbol ZENER
- added F1, F2, F3, F4, F5: FUSE, Fuse_Holders_and_Fuses:Fuse_SMD1206_HandSoldering, symbol FUSE
- added P1, P2: CONN_XT60, KiCad-Dev:XT60, symbol CONN_XT60
- D1, D2, D4, D5: renamed from D?; footprint (none) -> Discret:D3
- P3: renamed from P?; footprint (none) -> Pin_Headers:Pin_Header_Straight_2x03
Connections:
- wire segments 54 -> 48

Commit message: test
Parts:
- D1, D2, D3, D4, D5: footprint Discret:D3 -> Diodes_SMD:SOD-123
Changed lines of the file:
@@
 F 0 "D4" H 7900 2000 50  0000 C CNN
 F 1 "3.3v" H 7900 1800 50  0000 C CNN
-F 2 "Discret:D3" H 7900 1900 50  0001 C CNN
+F 2 "Diodes_SMD:SOD-123" H 7900 1900 50  0001 C CNN
 F 3 "" H 7900 1900 50  0000 C CNN
 	1    7900 1900
@@
 F 0 "D5" H 8200 2000 50  0000 C CNN
 F 1 "3.3v" H 8200 1800 50  0000 C CNN
-F 2 "Discret:D3" H 8200 1900 50  0001 C CNN
+F 2 "Diodes_SMD:SOD-123" H 8200 1900 50  0001 C CNN
 F 3 "" H 8200 1900 50  0000 C CNN
 	1    8200 1900
@@
 F 0 "D1" H 4350 1950 50  0000 C CNN
 F 1 "15v" H 4350 1750 50  0000 C CNN
-F 2 "Discret:D3" H 4350 1850 50  0001 C CNN
+F 2 "Diodes_SMD:SOD-123" H 4350 1850 50  0001 C CNN
 F 3 "" H 4350 1850 50  0000 C CNN
 	1    4350 1850
@@
 F 0 "D2" H 5450 2000 50  0000 C CNN
 F 1 "3.3v" H 5450 1800 50  0000 C CNN
-F 2 "Discret:D3" H 5450 1900 50  0001 C CNN
+F 2 "Diodes_SMD:SOD-123" H 5450 1900 50  0001 C CNN
 F 3 "" H 5450 1900 50  0000 C CNN
 	1    5450 1900
@@
 F 0 "D3" H 6450 2000 50  0000 C CNN
 F 1 "3.3v" H 6450 1800 50  0000 C CNN
-F 2 "Discret:D3" H 6450 1900 50  0001 C CNN
+F 2 "Diodes_SMD:SOD-123" H 6450 1900 50  0001 C CNN
 F 3 "" H 6450 1900 50  0000 C CNN
 	1    6450 1900

Commit message: test
Parts:
- removed D1: 15v, Diodes_SMD:SOD-123, symbol ZENER
- removed D2, D3, D4, D5: 3.3v, Diodes_SMD:SOD-123, symbol ZENER
- removed F1, F2, F3, F4, F5: FUSE, Fuse_Holders_and_Fuses:Fuse_SMD1206_HandSoldering, symbol FUSE
Connections:
- wire segments 48 -> 34
Changed lines of the file:
@@
 	1    0    0    -1
 $EndComp
-$Sheet
-S 6300 3300 1300 1200
-U 581FE98D
-F0 "kill_sw" 60
-F1 "kill_sw.sch" 60
-F2 "in+" I L 6300 3700 60
-F3 "enabled2_3.3v" O R 7600 3350 60
-F4 "enabled1_3.3v" O R 7600 3450 60
-F5 "enable" I L 6300 3350 60
-F6 "GND" I L 6300 4450 60
-F7 "out+" O R 7600 3700 60
-$EndSheet
 Wire Wire Line
 	3050 4450 3050 4800
@@
 Wire Wire Line
 	2550 4800 8100 4800
-Wire Wire Line
-	5750 2250 5800 2250
 Connection ~ 3050 4800
 Wire Wire Line
 	4350 3350 3950 3350
-Wire Wire Line
-	5450 2450 5800 2450
 Text HLabel 2800 3700 0    60   Input ~ 0
 in+
@@
 Text HLabel 2550 4800 0    60   Input ~ 0
 GND
-$Comp
-L ZENER D4
-U 1 1 582002DA
-P 7900 1900
-F 0 "D4" H 7900 2000 50  0000 C CNN
-F 1 "3.3v" H 7900 1800 50  0000 C CNN
-F 2 "Diodes_SMD:SOD-123" H 7900 1900 50  0001 C CNN
-F 3 "" H 7900 1900 50  0000 C CNN
-	1    7900 1900
-	0    -1   -1   0
-$EndComp
-$Comp
-L ZENER D5
-U 1 1 58200500
-P 8200 1900
-F 0 "D5" H 8200 2000 50  0000 C CNN
-F 1 "3.3v" H 8200 1800 50  0000 C CNN
-F 2 "Diodes_SMD:SOD-123" H 8200 1900 50  0001 C CNN
-F 3 "" H 8200 1900 50  0000 C CNN
-	1    8200 1900
-	0    -1   -1   0
-$EndComp
-$Comp
-L ZENER D1
-U 1 1 5820057B
-P 4350 1850
-F 0 "D1" H 4350 1950 50  0000 C CNN
-F 1 "15v" H 4350 1750 50  0000 C CNN
-F 2 "Diodes_SMD:SOD-123" H 4350 1850 50  0001 C CNN
-F 3 "" H 4350 1850 50  0000 C CNN
-	1    4350 1850
-	0    -1   -1   0
-$EndComp
-$Comp
-L ZENER D2
-U 1 1 582005F9
-P 5450 1900
-F 0 "D2" H 5450 2000 50  0000 C CNN
-F 1 "3.3v" H 5450 1800 50  0000 C CNN
-F 2 "Diodes_SMD:SOD-123" H 5450 1900 50  0001 C CNN
-F 3 "" H 5450 1900 50  0000 C CNN
-	1    5450 1900
-	0    -1   -1   0
-$EndComp
-Text HLabel 3950 1500 0    60   Input ~ 0
-GND
 Wire Wire Line
-	3950 1500 8200 1500
+	6450 3150 6200 3150
 Wire Wire Line
-	4350 1500 7900 1500
+	4350 1950 4350 3350
 Wire Wire Line
-	7900 1500 7900 1700
+	5600 3150 5850 3150
 Wire Wire Line
-	8200 1500 8200 1700
-Connection ~ 7900 1500
+	5600 2450 5600 3150
 Wire Wire Line
-	4350 1500 4350 1650
-Connection ~ 4350 1500
-Wire Wire Line
-	7900 2100 7900 2550
-Connection ~ 7900 2350
-Wire Wire Line
-	8200 2100 8200 2550
-Wire Wire Line
-	5450 1700 5450 1500
-Connection ~ 5450 1500
-Connection ~ 4350 2350
-Connection ~ 5450 2450
-Wire Wire Line
-	5750 2250 5750 1500
-Connection ~ 5750 1500
-Wire Wire Line
-	6200 3150 6450 3150
-Wire Wire Line
-	6450 2100 6450 2550
-$Comp
-L FUSE F1
-U 1 1 58203F80
-P 4350 2750
-F 0 "F1" H 4450 2800 50  0000 C CNN
-F 1 "FUSE" H 4250 2700 50  0000 C CNN
-F 2 "Fuse_Holders_and_Fuses:Fuse_SMD1206_HandSoldering" H 4350 2750 50  0001 C CNN
-F 3 "" H 4350 2750 50  0000 C CNN
-	1    4350 2750
-	0    1    1    0
-$EndComp
-Wire Wire Line
-	4350 3000 4350 3350
-Wire Wire Line
-	4350 2050 4350 2500
-Wire Wire Line
-	4350 2350 5800 2350
-$Comp
-L FUSE F2
-U 1 1 582046F6
-P 5450 2800
-F 0 "F2" H 5550 2850 50  0000 C CNN
-F 1 "FUSE" H 5350 2750 50  0000 C CNN
-F 2 "Fuse_Holders_and_Fuses:Fuse_SMD1206_HandSoldering" H 5450 2800 50  0001 C CNN
-F 3 "" H 5450 2800 50  0000 C CNN
-	1    5450 2800
-	0    1    1    0
-$EndComp
-Wire Wire Line
-	5450 2100 5450 2550
-Wire Wire Line
-	5850 3150 5450 3150
-Wire Wire Line
-	5450 3150 5450 3050
-$Comp
-L FUSE F3
-U 1 1 58204DFD
-P 6450 2800
-F 0 "F3" H 6550 2850 50  0000 C CNN
-F 1 "FUSE" H 6350 2750 50  0000 C CNN
-F 2 "Fuse_Holders_and_Fuses:Fuse_SMD1206_HandSoldering" H 6450 2800 50  0001 C CNN
-F 3 "" H 6450 2800 50  0000 C CNN
-	1    6450 2800
-	0    1    1    0
-$EndComp
-$Comp
-L ZENER D3
-U 1 1 58204EC7
-P 6450 1900
-F 0 "D3" H 6450 2000 50  0000 C CNN
-F 1 "3.3v" H 6450 1800 50  0000 C CNN
-F 2 "Diodes_SMD:SOD-123" H 6450 1900 50  0001 C CNN
-F 3 "" H 6450 1900 50  0000 C CNN
-	1    6450 1900
-	0    -1   -1   0
-$EndComp
-Wire Wire Line
-	6450 1500 6450 1700
-Connection ~ 6450 1500
-Wire Wire Line
-	6450 3150 6450 3050
-$Comp
-L FUSE F4
-U 1 1 58206065
-P 7900 2800
-F 0 "F4" H 8000 2850 50  0000 C CNN
-F 1 "FUSE" H 7800 2750 50  0000 C CNN
-F 2 "Fuse_Holders_and_Fuses:Fuse_SMD1206_HandSoldering" H 7900 2800 50  0001 C CNN
-F 3 "" H 7900 2800 50  0000 C CNN
-	1    7900 2800
-	0    1    1    0
-$EndComp
-$Comp
-L FUSE F5
-U 1 1 58206220
-P 8200 2800
-F 0 "F5" H 8300 2850 50  0000 C CNN
-F 1 "FUSE" H 8100 2750 50  0000 C CNN
-F 2 "Fuse_Holders_and_Fuses:Fuse_SMD1206_HandSoldering" H 8200 2800 50  0001 C CNN
-F 3 "" H 8200 2800 50  0000 C CNN
-	1    8200 2800
-	0    1    1    0
-$EndComp
+	6450 2450 6450 3150
 Wire Wire Line
 	5750 3350 5850 3350
@@
 	6200 3350 6200 3150
 Wire Wire Line
-	7900 3050 7900 3350
+	7900 2350 7900 3350
 Wire Wire Line
 	7900 3350 7600 3350
-Wire Wire Line
-	8200 3050 8200 3450
-Wire Wire Line
-	8200 3450 7600 3450
-Connection ~ 8200 2250
-Connection ~ 6450 2450
-Wire Wire Line
-	6300 2450 6450 2450
-Wire Wire Line
-	7900 2350 6300 2350
-Wire Wire Line
-	8200 2250 6300 2250
 $Comp
 L CONN_XT60 P1
@@
 Wire Wire Line
 	2150 1600 1850 1600
+Text HLabel 5550 2250 0    60   Input ~ 0
+GND
+Wire Wire Line
+	5550 2250 5800 2250
+Wire Wire Line
+	5600 2450 5800 2450
+Wire Wire Line
+	6450 2450 6300 2450
+Wire Wire Line
+	7900 2350 6300 2350
+Wire Wire Line
+	4350 1950 6600 1950
+Wire Wire Line
+	6600 1950 6600 2250
+Wire Wire Line
+	6600 2250 6300 2250
+$Sheet
+S 6300 3300 1300 1200
+U 581FE98D
+F0 "kill_sw" 60
+F1 "kill_sw.sch" 60
+F2 "in+" I L 6300 3700 60
+F3 "enabled2_3.3v" O R 7600 3350 60
+F4 "enable" I L 6300 3350 60
+F5 "GND" I L 6300 4450 60
+F6 "out+" O R 7600 3700 60
+$EndSheet
 $EndSCHEMATC

Commit message: test
Parts:
- added P? (x3): CONN_XT60, KiCad-Dev:XT60, symbol CONN_XT60
Connections:
- net GND: now also P?.1 (-), P?.1 (-), P?.1 (-)
- net fuse/enabled1_3.3v: now also P3.4 (P4)
- net fuse/enabled2_3.3v: now also P3.6 (P6); no longer P3.5 (P5)
- net kill_sw/enable: now also P3.5 (P5); no longer P3.6 (P6)
- net kill_sw/enabled2_3.3v: now also P3.3 (P3); no longer P3.4 (P4)
- net out+: now also P?.2 (+), P?.2 (+), P?.2 (+)
Other:
- moved on the sheet: P1, P2
Changed lines of the file:
@@
 F6 "out+" O R 5750 3700 60
 $EndSheet
-Wire Wire Line
-	3950 3700 4650 3700
-Wire Wire Line
-	5750 3700 6300 3700
 $Comp
 L CONN_02X03 P3
@@
 	1    0    0    -1
 $EndComp
-Wire Wire Line
-	3050 4450 3050 4800
-Wire Wire Line
-	4650 4450 4450 4450
-Wire Wire Line
-	4450 4450 4450 4800
-Connection ~ 4450 4800
-Connection ~ 6000 4800
-Wire Wire Line
-	2550 4800 8100 4800
-Connection ~ 3050 4800
-Wire Wire Line
-	4350 3350 3950 3350
 Text HLabel 2800 3700 0    60   Input ~ 0
 in+
 Text HLabel 8550 3700 2    60   Output ~ 0
 out+
-Wire Wire Line
-	8550 3700 7600 3700
-Wire Wire Line
-	3300 3700 2800 3700
 Text HLabel 2550 4800 0    60   Input ~ 0
 GND
-Wire Wire Line
-	6450 3150 6200 3150
-Wire Wire Line
-	4350 1950 4350 3350
-Wire Wire Line
-	5600 3150 5850 3150
-Wire Wire Line
-	5600 2450 5600 3150
-Wire Wire Line
-	6450 2450 6450 3150
-Wire Wire Line
-	5750 3350 5850 3350
-Wire Wire Line
-	5850 3350 5850 3150
-Wire Wire Line
-	3050 4450 3300 4450
-Wire Wire Line
-	6300 4450 6000 4450
-Wire Wire Line
-	6000 4450 6000 4800
-Wire Wire Line
-	6300 3350 6200 3350
-Wire Wire Line
-	6200 3350 6200 3150
-Wire Wire Line
-	7900 2350 7900 3350
-Wire Wire Line
-	7900 3350 7600 3350
 $Comp
 L CONN_XT60 P1
 U 1 1 5820B578
-P 1550 1550
-F 0 "P1" H 1550 1700 60  0000 C CNN
-F 1 "CONN_XT60" H 1550 1400 60  0000 C CNN
-F 2 "KiCad-Dev:XT60" H 1450 1700 60  0001 C CNN
-F 3 "" H 1450 1700 60  0001 C CNN
-	1    1550 1550
+P 1350 2850
+F 0 "P1" H 1350 3000 60  0000 C CNN
+F 1 "CONN_XT60" H 1350 2700 60  0000 C CNN
+F 2 "KiCad-Dev:XT60" H 1250 3000 60  0001 C CNN
+F 3 "" H 1250 3000 60  0001 C CNN
+	1    1350 2850
 	1    0    0    -1
 $EndComp
@@
 L CONN_XT60 P2
 U 1 1 5820B780
-P 1550 2000
-F 0 "P2" H 1550 2150 60  0000 C CNN
-F 1 "CONN_XT60" H 1550 1850 60  0000 C CNN
-F 2 "KiCad-Dev:XT60" H 1450 2150 60  0001 C CNN
-F 3 "" H 1450 2150 60  0001 C CNN
-	1    1550 2000
-	1    0    0    -1
-$EndComp
-Wire Wire Line
-	1850 1950 2150 1950
-Wire Wire Line
-	1850 1500 2150 1500
-Text HLabel 2150 1950 2    60   Input ~ 0
-GND
-Text HLabel 2150 1500 2    60   Input ~ 0
-GND
-Text HLabel 2150 2050 2    60   Input ~ 0
+P 1350 3300
+F 0 "P2" H 1350 3450 60  0000 C CNN
+F 1 "CONN_XT60" H 1350 3150 60  0000 C CNN
+F 2 "KiCad-Dev:XT60" H 1250 3450 60  0001 C CNN
+F 3 "" H 1250 3450 60  0001 C CNN
+	1    1350 3300
+	1    0    0    -1
+$EndComp
+Text HLabel 1950 3250 2    60   Input ~ 0
+GND
+Text HLabel 1950 2800 2    60   Input ~ 0
+GND
+Text HLabel 1950 3350 2    60   Input ~ 0
 in+
-Wire Wire Line
-	2150 2050 1850 2050
-Text HLabel 2150 1600 2    60   Output ~ 0
-out+
-Wire Wire Line
-	2150 1600 1850 1600
+Text HLabel 1950 2900 2    60   Output ~ 0
+out+
 Text HLabel 5550 2250 0    60   Input ~ 0
 GND
-Wire Wire Line
-	5550 2250 5800 2250
-Wire Wire Line
-	5600 2450 5800 2450
-Wire Wire Line
-	6450 2450 6300 2450
-Wire Wire Line
-	7900 2350 6300 2350
-Wire Wire Line
-	4350 1950 6600 1950
-Wire Wire Line
-	6600 1950 6600 2250
-Wire Wire Line
-	6600 2250 6300 2250
 $Sheet
 S 6300 3300 1300 1200
@@
 F6 "out+" O R 7600 3700 60
 $EndSheet
+Wire Wire Line
+	3950 3700 4650 3700
+Wire Wire Line
+	5750 3700 6300 3700
+Wire Wire Line
+	3050 4450 3050 4800
+Wire Wire Line
+	4650 4450 4450 4450
+Wire Wire Line
+	4450 4450 4450 4800
+Connection ~ 4450 4800
+Connection ~ 6000 4800
+Wire Wire Line
+	2550 4800 8100 4800
+Connection ~ 3050 4800
+Wire Wire Line
+	4350 3350 3950 3350
+Wire Wire Line
+	8550 3700 7600 3700
+Wire Wire Line
+	3300 3700 2800 3700
+Wire Wire Line
+	4350 1950 4350 3350
+Wire Wire Line
+	5850 3350 5750 3350
+Wire Wire Line
+	5850 2800 5850 3350
+Wire Wire Line
+	3050 4450 3300 4450
+Wire Wire Line
+	6300 4450 6000 4450
+Wire Wire Line
+	6000 4450 6000 4800
+Wire Wire Line
+	6200 3350 6300 3350
+Wire Wire Line
+	6200 2900 6200 3350
+Wire Wire Line
+	7900 2600 7900 3350
+Wire Wire Line
+	7900 3350 7600 3350
+Wire Wire Line
+	1650 3250 1950 3250
+Wire Wire Line
+	1650 2800 1950 2800
+Wire Wire Line
+	1950 3350 1650 3350
+Wire Wire Line
+	1950 2900 1650 2900
+Wire Wire Line
+	5550 2250 5800 2250
+Wire Wire Line
+	4350 1950 6600 1950
+Wire Wire Line
+	6600 1950 6600 2250
+Wire Wire Line
+	6600 2250 6300 2250
+Wire Wire Line
+	5750 3450 5950 3450
+Wire Wire Line
+	5950 3450 5950 3050
+Wire Wire Line
+	5850 2800 6400 2800
+Wire Wire Line
+	6400 2800 6400 2450
+Wire Wire Line
+	6400 2450 6300 2450
+Wire Wire Line
+	6200 2900 5600 2900
+Wire Wire Line
+	5600 2900 5600 2450
+Wire Wire Line
+	5600 2450 5800 2450
+Wire Wire Line
+	5950 3050 6550 3050
+Wire Wire Line
+	6550 3050 6550 2350
+Wire Wire Line
+	6550 2350 6300 2350
+Wire Wire Line
+	7900 2600 5700 2600
+Wire Wire Line
+	5700 2600 5700 2350
+Wire Wire Line
+	5700 2350 5800 2350
+$Comp
+L CONN_XT60 P?
+U 1 1 5827545B
+P 1350 2300
+F 0 "P?" H 1350 2450 60  0000 C CNN
+F 1 "CONN_XT60" H 1350 2150 60  0000 C CNN
+F 2 "KiCad-Dev:XT60" H 1250 2450 60  0001 C CNN
+F 3 "" H 1250 2450 60  0001 C CNN
+	1    1350 2300
+	1    0    0    -1
+$EndComp
+Text HLabel 1950 2250 2    60   Input ~ 0
+GND
+Text HLabel 1950 2350 2    60   Output ~ 0
+out+
+Wire Wire Line
+	1650 2250 1950 2250
+Wire Wire Line
+	1950 2350 1650 2350
+$Comp
+L CONN_XT60 P?
+U 1 1 58275597
+P 1350 1750
+F 0 "P?" H 1350 1900 60  0000 C CNN
+F 1 "CONN_XT60" H 1350 1600 60  0000 C CNN
+F 2 "KiCad-Dev:XT60" H 1250 1900 60  0001 C CNN
+F 3 "" H 1250 1900 60  0001 C CNN
+	1    1350 1750
+	1    0    0    -1
+$EndComp
+Text HLabel 1950 1700 2    60   Input ~ 0
+GND
+Text HLabel 1950 1800 2    60   Output ~ 0
+out+
+Wire Wire Line
+	1650 1700 1950 1700
+Wire Wire Line
+	1950 1800 1650 1800
+$Comp
+L CONN_XT60 P?
+U 1 1 582755A1
+P 1350 1200
+F 0 "P?" H 1350 1350 60  0000 C CNN
+F 1 "CONN_XT60" H 1350 1050 60  0000 C CNN
+F 2 "KiCad-Dev:XT60" H 1250 1350 60  0001 C CNN
+F 3 "" H 1250 1350 60  0001 C CNN
+	1    1350 1200
+	1    0    0    -1
+$EndComp
+Text HLabel 1950 1150 2    60   Input ~ 0
+GND
+Text HLabel 1950 1250 2    60   Output ~ 0
+out+
+Wire Wire Line
+	1650 1150 1950 1150
+Wire Wire Line
+	1950 1250 1650 1250
 $EndSCHEMATC

Commit message: test
Parts:
- gave numbers to parts that had none: 3
Changed lines of the file:
@@
 	5700 2350 5800 2350
 $Comp
-L CONN_XT60 P?
+L CONN_XT60 P8
 U 1 1 5827545B
 P 1350 2300
-F 0 "P?" H 1350 2450 60  0000 C CNN
+F 0 "P8" H 1350 2450 60  0000 C CNN
 F 1 "CONN_XT60" H 1350 2150 60  0000 C CNN
 F 2 "KiCad-Dev:XT60" H 1250 2450 60  0001 C CNN
@@
 	1950 2350 1650 2350
 $Comp
-L CONN_XT60 P?
+L CONN_XT60 P7
 U 1 1 58275597
 P 1350 1750
-F 0 "P?" H 1350 1900 60  0000 C CNN
+F 0 "P7" H 1350 1900 60  0000 C CNN
 F 1 "CONN_XT60" H 1350 1600 60  0000 C CNN
 F 2 "KiCad-Dev:XT60" H 1250 1900 60  0001 C CNN
@@
 	1950 1800 1650 1800
 $Comp
-L CONN_XT60 P?
+L CONN_XT60 P6
 U 1 1 582755A1
 P 1350 1200
-F 0 "P?" H 1350 1350 60  0000 C CNN
+F 0 "P6" H 1350 1350 60  0000 C CNN
 F 1 "CONN_XT60" H 1350 1050 60  0000 C CNN
 F 2 "KiCad-Dev:XT60" H 1250 1350 60  0001 C CNN

Commit message: test
Connections:
- net fuse/enabled1_3.3v: now also P3.6 (P6); no longer P3.4 (P4)
- net fuse/enabled2_3.3v: now also P3.4 (P4); no longer P3.6 (P6)
Changed lines of the file:
@@
 	5950 3450 5950 3050
 Wire Wire Line
-	5850 2800 6400 2800
+	6400 2800 5850 2800
 Wire Wire Line
-	6400 2800 6400 2450
-Wire Wire Line
-	6400 2450 6300 2450
+	6400 2350 6400 2800
 Wire Wire Line
 	6200 2900 5600 2900
@@
 	5950 3050 6550 3050
 Wire Wire Line
-	6550 3050 6550 2350
-Wire Wire Line
-	6550 2350 6300 2350
+	6550 3050 6550 2450
 Wire Wire Line
 	7900 2600 5700 2600
@@
 Wire Wire Line
 	1950 1250 1650 1250
+Wire Wire Line
+	6400 2350 6300 2350
+Wire Wire Line
+	6550 2450 6300 2450
 $EndSCHEMATC

Commit message: test
Parts:
- removed P6, P7, P8: CONN_XT60, KiCad-Dev:XT60, symbol CONN_XT60
- P3: footprint Pin_Headers:Pin_Header_Straight_2x03 -> KiCad-Dev:Pin_Header_Straight_2x03_box
Changed lines of the file:
@@
 F 0 "P3" H 6050 2550 50  0000 C CNN
 F 1 "CONN_02X03" H 6050 2150 50  0000 C CNN
-F 2 "Pin_Headers:Pin_Header_Straight_2x03" H 6050 1150 50  0001 C CNN
+F 2 "KiCad-Dev:Pin_Header_Straight_2x03_box" H 6050 1150 50  0001 C CNN
 F 3 "" H 6050 1150 50  0000 C CNN
 	1    6050 2350
@@
 Wire Wire Line
 	5700 2350 5800 2350
-$Comp
-L CONN_XT60 P8
-U 1 1 5827545B
-P 1350 2300
-F 0 "P8" H 1350 2450 60  0000 C CNN
-F 1 "CONN_XT60" H 1350 2150 60  0000 C CNN
-F 2 "KiCad-Dev:XT60" H 1250 2450 60  0001 C CNN
-F 3 "" H 1250 2450 60  0001 C CNN
-	1    1350 2300
-	1    0    0    -1
-$EndComp
-Text HLabel 1950 2250 2    60   Input ~ 0
-GND
-Text HLabel 1950 2350 2    60   Output ~ 0
-out+
-Wire Wire Line
-	1650 2250 1950 2250
-Wire Wire Line
-	1950 2350 1650 2350
-$Comp
-L CONN_XT60 P7
-U 1 1 58275597
-P 1350 1750
-F 0 "P7" H 1350 1900 60  0000 C CNN
-F 1 "CONN_XT60" H 1350 1600 60  0000 C CNN
-F 2 "KiCad-Dev:XT60" H 1250 1900 60  0001 C CNN
-F 3 "" H 1250 1900 60  0001 C CNN
-	1    1350 1750
-	1    0    0    -1
-$EndComp
-Text HLabel 1950 1700 2    60   Input ~ 0
-GND
-Text HLabel 1950 1800 2    60   Output ~ 0
-out+
-Wire Wire Line
-	1650 1700 1950 1700
-Wire Wire Line
-	1950 1800 1650 1800
-$Comp
-L CONN_XT60 P6
-U 1 1 582755A1
-P 1350 1200
-F 0 "P6" H 1350 1350 60  0000 C CNN
-F 1 "CONN_XT60" H 1350 1050 60  0000 C CNN
-F 2 "KiCad-Dev:XT60" H 1250 1350 60  0001 C CNN
-F 3 "" H 1250 1350 60  0001 C CNN
-	1    1350 1200
-	1    0    0    -1
-$EndComp
-Text HLabel 1950 1150 2    60   Input ~ 0
-GND
-Text HLabel 1950 1250 2    60   Output ~ 0
-out+
-Wire Wire Line
-	1650 1150 1950 1150
-Wire Wire Line
-	1950 1250 1650 1250
 Wire Wire Line
 	6400 2350 6300 2350
