File: pdb1/kill_sw.sch (KiCad schematic (older format))
At the start: 10 parts, among them P4 CONN_02X03, P5 CONN_01X03, Q2 BUK9Y4R8-60E, U4 74LVC1G08, U7 MIC5014, U8 NSI45020AT1G

Commit message: test
Parts:
- removed R3, R4: R, Resistors_SMD:R_0603, symbol R
- removed U4: 74LVC1G08, TO_SOT_Packages_SMD:SOT-353, symbol 74LVC1G08
Connections:
- net enable: now also P4.4 (P4)
- net at P4.2 (P2): now also P5.1 (P1)
Other:
- moved on the sheet: D9, P4, Q2, U8
Changed lines of the file:
@@
 	1    0    0    -1
 $EndComp
-Text HLabel 1650 2650 0    60   Input ~ 0
+Text HLabel 1650 2050 0    60   Input ~ 0
 in+
 Text HLabel 1650 4750 0    60   Input ~ 0
 GND
-Text HLabel 6950 2650 2    60   Output ~ 0
+Text HLabel 6950 2050 2    60   Output ~ 0
 out+
 $Comp
 L NSI45020AT1G U?
 U 1 1 581F58D3
-P 6500 3050
+P 6500 2450
 AR Path="/581F28FF/581F58D3" Ref="U?"  Part="1"
 AR Path="/581FE101/581FE98D/581F58D3" Ref="U8"  Part="1"
-F 0 "U8" H 6500 2900 60  0000 C CNN
-F 1 "NSI45020AT1G" H 6500 3200 60  0000 C CNN
-F 2 "Diodes_SMD:SOD-123" H 5750 3200 60  0001 C CNN
-F 3 "" H 5750 3200 60  0001 C CNN
-	1    6500 3050
+F 0 "U8" H 6500 2300 60  0000 C CNN
+F 1 "NSI45020AT1G" H 6500 2600 60  0000 C CNN
+F 2 "Diodes_SMD:SOD-123" H 5750 2600 60  0001 C CNN
+F 3 "" H 5750 2600 60  0001 C CNN
+	1    6500 2450
 	0    1    1    0
 $EndComp
@@
 L LED D?
 U 1 1 581F591A
-P 6500 4400
+P 6500 4150
 AR Path="/581F28FF/581F591A" Ref="D?"  Part="1"
 AR Path="/581FE101/581FE98D/581F591A" Ref="D9"  Part="1"
-F 0 "D9" H 6500 4500 50  0000 C CNN
-F 1 "LED" H 6500 4300 50  0000 C CNN
-F 2 "LEDs:LED_0805" H 6500 4400 50  0001 C CNN
-F 3 "" H 6500 4400 50  0000 C CNN
-	1    6500 4400
+F 0 "D9" H 6500 4250 50  0000 C CNN
+F 1 "LED" H 6500 4050 50  0000 C CNN
+F 2 "LEDs:LED_0805" H 6500 4150 50  0001 C CNN
+F 3 "" H 6500 4150 50  0000 C CNN
+	1    6500 4150
 	0    -1   -1   0
 $EndComp
@@
 L BUK9Y4R8-60E Q2
 U 1 1 58248FB0
-P 5800 2750
-F 0 "Q2" H 6150 2850 50  0000 L CNN
-F 1 "BUK9Y4R8-60E" H 6150 2750 50  0000 L CNN
-F 2 "TO_SOT_Packages_SMD:SOT-669_LFPAK" H 6150 2675 50  0001 L CIN
-F 3 "http://www.farnell.com/datasheets/2053583.pdf?_ga=1.217785489.606791601.1474638083" H 4050 2200 50  0001 L CNN
-	1    5800 2750
+P 5800 2150
+F 0 "Q2" H 6150 2250 50  0000 L CNN
+F 1 "BUK9Y4R8-60E" H 6150 2150 50  0000 L CNN
+F 2 "TO_SOT_Packages_SMD:SOT-669_LFPAK" H 6150 2075 50  0001 L CIN
+F 3 "http://www.farnell.com/datasheets/2053583.pdf?_ga=1.217785489.606791601.1474638083" H 4050 1600 50  0001 L CNN
+	1    5800 2150
 	0    -1   -1   0
 $EndComp
@@
 L CONN_02X03 P4
 U 1 1 5825EF78
-P 2550 3400
-F 0 "P4" H 2550 3600 50  0000 C CNN
-F 1 "CONN_02X03" H 2550 3200 50  0000 C CNN
-F 2 "Pin_Headers:Pin_Header_Straight_2x03" H 2550 2200 50  0001 C CNN
-F 3 "" H 2550 2200 50  0000 C CNN
-	1    2550 3400
+P 2950 3950
+F 0 "P4" H 2950 4150 50  0000 C CNN
+F 1 "CONN_02X03" H 2950 3750 50  0000 C CNN
+F 2 "Pin_Headers:Pin_Header_Straight_2x03" H 2950 2750 50  0001 C CNN
+F 3 "" H 2950 2750 50  0000 C CNN
+	1    2950 3950
 	1    0    0    -1
 $EndComp
-$Comp
-L R R3
-U 1 1 582707A5
-P 3000 4400
-F 0 "R3" V 3080 4400 50  0000 C CNN
-F 1 "R" V 3000 4400 50  0000 C CNN
-F 2 "Resistors_SMD:R_0603" V 2930 4400 50  0001 C CNN
-F 3 "" H 3000 4400 50  0000 C CNN
-	1    3000 4400
-	1    0    0    -1
-$EndComp
-$Comp
-L 74LVC1G08 U4
-U 1 1 582725D8
-P 3500 4050
-F 0 "U4" H 3600 3800 60  0000 C CNN
-F 1 "74LVC1G08" H 3800 4300 60  0000 C CNN
-F 2 "TO_SOT_Packages_SMD:SOT-353" H 3450 4100 60  0001 C CNN
-F 3 "http://www.nxp.com/documents/data_sheet/74LVC1G08.pdf?" H 4000 3600 60  0001 C CNN
-	1    3500 4050
-	1    0    0    -1
-$EndComp
-Wire Wire Line
-	4450 3950 4800 3950
-Wire Wire Line
-	4700 2650 4700 3950
-Wire Wire Line
-	1650 2650 5600 2650
-Connection ~ 4700 2650
-Wire Wire Line
-	5850 2950 5850 4250
-Wire Wire Line
-	5850 4250 5700 4250
-Wire Wire Line
-	4600 4750 4600 4250
-Wire Wire Line
-	4600 4250 4800 4250
-Connection ~ 4600 4750
-Wire Wire Line
-	6000 2650 6950 2650
-Wire Wire Line
-	4800 4150 4700 4150
-Wire Wire Line
-	6050 4650 4700 4650
-Connection ~ 6050 2650
-Connection ~ 4700 3500
-Wire Wire Line
-	6500 2750 6500 2650
-Connection ~ 6500 2650
-Wire Wire Line
-	6500 4750 6500 4600
-Wire Wire Line
-	6500 3350 6500 4200
-Wire Wire Line
-	4700 3500 5000 3500
-Wire Wire Line
-	5300 3500 5500 3500
-Wire Wire Line
-	6700 3600 6500 3600
-Connection ~ 6500 3600
-Wire Wire Line
-	1650 4750 6500 4750
-Wire Wire Line
-	6000 2500 6050 2500
-Connection ~ 6050 2500
-Wire Wire Line
-	6000 2350 6050 2350
-Connection ~ 6050 2350
-Wire Wire Line
-	6050 2350 6050 4650
-Wire Wire Line
-	3500 3500 3500 3650
-Wire Wire Line
-	3500 4450 3500 4750
-Connection ~ 3500 4750
-Wire Wire Line
-	3000 4250 3000 4100
-Wire Wire Line
-	2150 4100 3150 4100
-Wire Wire Line
-	3000 4550 3000 4750
-Connection ~ 3000 4750
-Wire Wire Line
-	2000 3300 2000 4750
-Connection ~ 2000 4750
-Wire Wire Line
-	1750 4000 3150 4000
-Wire Wire Line
-	4700 4650 4700 4150
-$Comp
-L R R4
-U 1 1 58273070
-P 2800 4400
-F 0 "R4" V 2880 4400 50  0000 C CNN
-F 1 "R" V 2800 4400 50  0000 C CNN
-F 2 "Resistors_SMD:R_0603" V 2730 4400 50  0001 C CNN
-F 3 "" H 2800 4400 50  0000 C CNN
-	1    2800 4400
-	1    0    0    -1
-$EndComp
-Wire Wire Line
-	2800 4000 2800 4250
-Connection ~ 2800 4000
-Wire Wire Line
-	2800 4550 2800 4750
-Connection ~ 2800 4750
-Text HLabel 1750 4000 0    60   Input ~ 0
+Text HLabel 3350 3950 2    60   Input ~ 0
 enable
-Wire Wire Line
-	2000 3300 2300 3300
 $Comp
 L CONN_01X03 P5
@@
 $EndComp
 Wire Wire Line
+	4450 3950 4700 3950
+Wire Wire Line
+	4700 3950 4800 3950
+Wire Wire Line
+	4700 2050 4700 3500
+Wire Wire Line
+	4700 3500 4700 3950
+Wire Wire Line
+	1650 2050 4700 2050
+Wire Wire Line
+	4700 2050 5600 2050
+Connection ~ 4700 2050
+Wire Wire Line
+	5850 2350 5850 4250
+Wire Wire Line
+	5850 4250 5700 4250
+Wire Wire Line
+	4600 4750 4600 4250
+Wire Wire Line
+	4600 4250 4800 4250
+Connection ~ 4600 4750
+Wire Wire Line
+	6000 2050 6050 2050
+Wire Wire Line
+	6050 2050 6500 2050
+Wire Wire Line
+	6500 2050 6950 2050
+Wire Wire Line
+	4800 4150 4700 4150
+Wire Wire Line
+	6050 4650 4700 4650
+Connection ~ 6050 2050
+Connection ~ 4700 3500
+Wire Wire Line
+	6500 2150 6500 2050
+Connection ~ 6500 2050
+Wire Wire Line
+	6500 4750 6500 4350
+Wire Wire Line
+	6500 2750 6500 3600
+Wire Wire Line
+	6500 3600 6500 3950
+Wire Wire Line
+	4700 3500 5000 3500
+Wire Wire Line
+	5300 3500 5500 3500
+Wire Wire Line
+	6700 3600 6500 3600
+Connection ~ 6500 3600
+Wire Wire Line
+	1650 4750 1850 4750
+Wire Wire Line
+	1850 4750 4600 4750
+Wire Wire Line
+	4600 4750 6500 4750
+Wire Wire Line
+	6000 1900 6050 1900
+Connection ~ 6050 1900
+Wire Wire Line
+	6000 1750 6050 1750
+Connection ~ 6050 1750
+Wire Wire Line
+	6050 1750 6050 1900
+Wire Wire Line
+	6050 1900 6050 2050
+Wire Wire Line
+	6050 2050 6050 4650
+Wire Wire Line
+	4700 4650 4700 4150
+Wire Wire Line
 	4800 4050 4350 4050
-Wire Wire Line
-	4350 4050 4350 3950
-Wire Wire Line
-	3950 4050 4250 4050
 Wire Wire Line
 	4250 4050 4250 3950
 Connection ~ 4700 3950
 Wire Wire Line
-	2800 3500 3500 3500
-Connection ~ 3000 4100
+	2700 3850 1850 3850
 Wire Wire Line
-	2150 4100 2150 3500
+	1850 3850 1850 4750
+Connection ~ 1850 4750
 Wire Wire Line
-	2150 3500 2300 3500
+	3200 3850 3850 3850
+Wire Wire Line
+	3850 3850 3850 4050
+Wire Wire Line
+	3850 4050 4250 4050
+Wire Wire Line
+	3350 3950 3200 3950
+Wire Wire Line
+	4350 4050 4350 3950
 $EndSCHEMATC

Commit message: test
Changed lines of the file:
@@
 $EndComp
 Wire Wire Line
-	4450 3950 4700 3950
+	4450 3950 4800 3950
 Wire Wire Line
-	4700 3950 4800 3950
+	4700 2050 4700 3950
 Wire Wire Line
-	4700 2050 4700 3500
-Wire Wire Line
-	4700 3500 4700 3950
-Wire Wire Line
-	1650 2050 4700 2050
-Wire Wire Line
-	4700 2050 5600 2050
+	1650 2050 5600 2050
 Connection ~ 4700 2050
 Wire Wire Line
@@
 Connection ~ 4600 4750
 Wire Wire Line
-	6000 2050 6050 2050
-Wire Wire Line
-	6050 2050 6500 2050
-Wire Wire Line
-	6500 2050 6950 2050
+	6000 2050 6950 2050
 Wire Wire Line
 	4800 4150 4700 4150
@@
 	6500 4750 6500 4350
 Wire Wire Line
-	6500 2750 6500 3600
-Wire Wire Line
-	6500 3600 6500 3950
+	6500 2750 6500 3950
 Wire Wire Line
 	4700 3500 5000 3500
@@
 Connection ~ 6500 3600
 Wire Wire Line
-	1650 4750 1850 4750
-Wire Wire Line
-	1850 4750 4600 4750
-Wire Wire Line
-	4600 4750 6500 4750
+	1650 4750 6500 4750
 Wire Wire Line
 	6000 1900 6050 1900
@@
 Connection ~ 6050 1750
 Wire Wire Line
-	6050 1750 6050 1900
-Wire Wire Line
-	6050 1900 6050 2050
-Wire Wire Line
-	6050 2050 6050 4650
+	6050 1750 6050 4650
 Wire Wire Line
 	4700 4650 4700 4150

Commit message: test
Parts:
- removed P4: CONN_02X03, Pin_Headers:Pin_Header_Straight_2x03, symbol CONN_02X03
- removed P5: CONN_01X03, Pin_Headers:Pin_Header_Straight_1x03, symbol CONN_01X03
- added P4, P5: CONN_01X02, Pin_Headers:Pin_Header_Straight_1x02, symbol CONN_01X02
- added U4: LM3480-3.3, TO_SOT_Packages_SMD:SOT-23, symbol LM3480-3.3
- added U5: 74LVC1G08, TO_SOT_Packages_SMD:SOT-353, symbol 74LVC1G08
Connections:
- net GND: now also U4.3 (GND), U5.3 (GND)
- net enable: now also P5.1 (P1), U5.2 (B)
- net in+: now also U4.2 (VIN)
- net at U7.2 (Input): now also U5.4 (Y)
- new net: P4.2 (P2), P5.2 (P2), U5.1 (A)
- new net: P4.1 (P1), U4.1 (VOUT), U5.5 (VCC)
Changed lines of the file:
@@
 	0    -1   -1   0
 $EndComp
+Text HLabel 1250 4100 0    60   Input ~ 0
+enable
 $Comp
-L CONN_02X03 P4
-U 1 1 5825EF78
-P 2950 3950
-F 0 "P4" H 2950 4150 50  0000 C CNN
-F 1 "CONN_02X03" H 2950 3750 50  0000 C CNN
-F 2 "Pin_Headers:Pin_Header_Straight_2x03" H 2950 2750 50  0001 C CNN
-F 3 "" H 2950 2750 50  0000 C CNN
-	1    2950 3950
+L 74LVC1G08 U5
+U 1 1 582ACE25
+P 2600 4050
+F 0 "U5" H 2700 3800 60  0000 C CNN
+F 1 "74LVC1G08" H 2900 4300 60  0000 C CNN
+F 2 "TO_SOT_Packages_SMD:SOT-353" H 2550 4100 60  0001 C CNN
+F 3 "http://www.nxp.com/documents/data_sheet/74LVC1G08.pdf?" H 3100 3600 60  0001 C CNN
+	1    2600 4050
 	1    0    0    -1
 $EndComp
-Text HLabel 3350 3950 2    60   Input ~ 0
-enable
 $Comp
-L CONN_01X03 P5
-U 1 1 5827405B
-P 4350 3750
-F 0 "P5" H 4350 3950 50  0000 C CNN
-F 1 "CONN_01X03" V 4450 3750 50  0000 C CNN
-F 2 "Pin_Headers:Pin_Header_Straight_1x03" H 4350 3750 50  0001 C CNN
-F 3 "" H 4350 3750 50  0000 C CNN
-	1    4350 3750
+L CONN_01X02 P4
+U 1 1 582AD5E4
+P 2050 3300
+F 0 "P4" H 2050 3450 50  0000 C CNN
+F 1 "CONN_01X02" V 2150 3300 50  0000 C CNN
+F 2 "Pin_Headers:Pin_Header_Straight_1x02" H 2050 3300 50  0001 C CNN
+F 3 "" H 2050 3300 50  0000 C CNN
+	1    2050 3300
+	0    1    -1   0
+$EndComp
+Text HLabel 2000 2650 0    60   Input ~ 0
+GND
+$Comp
+L CONN_01X02 P5
+U 1 1 582ADB70
+P 1650 3500
+F 0 "P5" H 1650 3650 50  0000 C CNN
+F 1 "CONN_01X02" V 1750 3500 50  0000 C CNN
+F 2 "Pin_Headers:Pin_Header_Straight_1x02" H 1650 3500 50  0001 C CNN
+F 3 "" H 1650 3500 50  0000 C CNN
+	1    1650 3500
 	0    -1   -1   0
 $EndComp
-Wire Wire Line
-	4450 3950 4800 3950
 Wire Wire Line
 	4700 2050 4700 3950
@@
 	4700 4650 4700 4150
 Wire Wire Line
-	4800 4050 4350 4050
+	3050 4050 4800 4050
 Wire Wire Line
-	4250 4050 4250 3950
-Connection ~ 4700 3950
+	2600 2150 2600 2050
+Connection ~ 2600 2050
 Wire Wire Line
-	2700 3850 1850 3850
+	2600 3150 2600 3650
 Wire Wire Line
-	1850 3850 1850 4750
-Connection ~ 1850 4750
+	2600 4450 2600 4750
+Connection ~ 2600 4750
 Wire Wire Line
-	3200 3850 3850 3850
+	4700 3950 4800 3950
 Wire Wire Line
-	3850 3850 3850 4050
+	2100 3500 2100 3550
 Wire Wire Line
-	3850 4050 4250 4050
+	2100 3550 2600 3550
+Connection ~ 2600 3550
 Wire Wire Line
-	3350 3950 3200 3950
+	2000 3500 2000 4000
 Wire Wire Line
-	4350 4050 4350 3950
+	2000 2650 2300 2650
+Wire Wire Line
+	1700 3700 1700 4000
+Connection ~ 2000 4000
+Wire Wire Line
+	1600 3700 1600 4100
+Connection ~ 1600 4100
+Wire Wire Line
+	1700 4000 2250 4000
+Wire Wire Line
+	1250 4100 2250 4100
+$Comp
+L LM3480-3.3 U4
+U 1 1 582AF2F2
+P 2600 2650
+F 0 "U4" H 2300 2800 50  0000 L CNN
+F 1 "LM3480-3.3" H 2900 2800 50  0000 R CNN
+F 2 "TO_SOT_Packages_SMD:SOT-23" H 2600 2250 50  0001 C CIN
+F 3 "" H 2600 2650 50  0000 C CNN
+	1    2600 2650
+	0    1    1    0
+$EndComp
 $EndSCHEMATC

Commit message: test
Parts:
- added R3, R4: R, Resistors_SMD:R_0603, symbol R
Connections:
- net GND: now also R3.2, R4.2
- net enable: now also R3.1
- net at P4.2 (P2), P5.2 (P2), U5.1 (A): now also R4.1
Changed lines of the file:
@@
 	0    1    1    0
 $EndComp
+$Comp
+L R R3
+U 1 1 582B6025
+P 1900 4400
+F 0 "R3" V 1980 4400 50  0000 C CNN
+F 1 "R" V 1900 4400 50  0000 C CNN
+F 2 "Resistors_SMD:R_0603" V 1830 4400 50  0001 C CNN
+F 3 "" H 1900 4400 50  0000 C CNN
+	1    1900 4400
+	1    0    0    -1
+$EndComp
+$Comp
+L R R4
+U 1 1 582B608A
+P 2150 4400
+F 0 "R4" V 2230 4400 50  0000 C CNN
+F 1 "R" V 2150 4400 50  0000 C CNN
+F 2 "Resistors_SMD:R_0603" V 2080 4400 50  0001 C CNN
+F 3 "" H 2150 4400 50  0000 C CNN
+	1    2150 4400
+	1    0    0    -1
+$EndComp
+Wire Wire Line
+	2150 4250 2150 4000
+Connection ~ 2150 4000
+Wire Wire Line
+	1900 4250 1900 4100
+Connection ~ 1900 4100
+Wire Wire Line
+	1900 4550 1900 4750
+Connection ~ 1900 4750
+Wire Wire Line
+	2150 4550 2150 4750
+Connection ~ 2150 4750
 $EndSCHEMATC
