File: pdb3/_saved_main.sch (KiCad schematic (older format))
At the start: 6 parts, among them P1 CONN_XT60_Male, P2 CONN_XT60_Male, P3 CONN_01X02, U1 ARDUINO_MICRO_SHIELD, U2 WPMDH1100501S

Commit message: test
Parts:
- P10: renamed from P?; footprint (none) -> Pin_Headers:Pin_Header_Straight_1x02
Changed lines of the file:
@@
 Reed
 $Comp
-L CONN_01X02 P?
+L CONN_01X02 P10
 U 1 1 58311BEB
 P 7000 4300
-F 0 "P?" H 7000 4450 50  0000 C CNN
+F 0 "P10" H 7000 4450 50  0000 C CNN
 F 1 "CONN_01X02_Reed" V 7100 4300 50  0000 C CNN
-F 2 "" H 7000 4300 50  0000 C CNN
+F 2 "Pin_Headers:Pin_Header_Straight_1x02" H 7000 4300 50  0001 C CNN
 F 3 "" H 7000 4300 50  0000 C CNN
 	1    7000 4300
