File: pdb3/main.kicad_pcb (KiCad board)
At the start: 2 copper layers, 12 parts, among them P1 CONN_01X02, P2 CONN_01X02, Q1 BC849, U1 74LVC1G08, U2 LM3480-3.3, U3 AUIPS7111S

Commit message: test
Parts:
- U3: moved to F.Cu
- moved U3 3.41 mm to (175.3, 92.7), turned to 90 degrees
Routing:
- net /KSW/VCC: track 24.3 -> 0.00 mm, vias 1 -> 0
- net GND: track 19.7 -> 10.1 mm, vias 0 -> 1
- net Net-(R4-Pad1): track 19.5 -> 16.5 mm, vias 1 -> 0
- net Net-(D2-Pad1): track 20.1 -> 17.3 mm, vias 1 -> 0
- added copper zone on F.Cu, net /KSW/VCC
- added copper zone on B.Cu, net GND
Changed lines of the file:
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@@
-(kicad_pcb (version 4) (host pcbnew 4.0.4-stable)
+(kicad_pcb (version 4) (host pcbnew 4.0.4+e1-6308~48~ubuntu16.04.1-stable)
   (general
     (links 23)
-    (no_connects 5)
-    (area 169.185 90.214649 184.935 121.873333)
+    (no_connects 1)
+    (area 168.91 66.04 184.935 121.873333)
     (thickness 1.6)
     (drawings 0)
-    (tracks 73)
+    (tracks 52)
     (zones 0)
     (modules 12)
@@
   )
   (setup
-    (last_trace_width 0.6)
+    (last_trace_width 0.4)
     (user_trace_width 0.3)
     (user_trace_width 0.4)
@@
     (user_trace_width 0.6)
     (trace_clearance 0.2)
-    (zone_clearance 0.508)
+    (zone_clearance 1)
     (zone_45_only no)
     (trace_min 0.2)
@@
     (pad_to_mask_clearance 0.2)
     (aux_axis_origin 0 0)
-    (visible_elements FFFFEF7F)
+    (visible_elements FFFFFF7F)
     (pcbplotparams
       (layerselection 0x00030_80000001)
@@
     )
   )
-  (module TO_SOT_Packages_SMD:TO-263-5Lead (layer B.Cu)
-    (at 177.8 94.99 270)
+  (module TO_SOT_Packages_SMD:TO-263-5Lead (layer F.Cu)
+    (at 175.26 92.71 90)
     (descr "D2PAK / TO-263 3-lead smd package")
     (tags "D2PAK D2PAK-3 TO-263AB TO-263")
     (attr smd)
-    (fp_text reference U3 (at 3.5 0 540) (layer B.SilkS)
-      (effects (font (size 1 1) (thickness 0.15)) (justify mirror))
-    )
-    (fp_text value AUIPS7111S (at 15.25 0.25 540) (layer B.Fab)
-      (effects (font (size 1 1) (thickness 0.15)) (justify mirror))
-    )
-    (fp_line (start 14.1 -5.65) (end -2.55 -5.65) (layer B.CrtYd) (width 0.05))
-    (fp_line (start 14.1 5.65) (end 14.1 -5.65) (layer B.CrtYd) (width 0.05))
-    (fp_line (start 14.1 5.65) (end -2.55 5.65) (layer B.CrtYd) (width 0.05))
-    (fp_line (start -2.55 5.65) (end -2.55 -5.65) (layer B.CrtYd) (width 0.05))
-    (fp_line (start 2.5 -5) (end 2.5 -3.75) (layer B.SilkS) (width 0.15))
-    (fp_line (start 2.5 -5) (end 4 -5) (layer B.SilkS) (width 0.15))
-    (fp_line (start 2.5 5) (end 4 5) (layer B.SilkS) (width 0.15))
-    (fp_line (start 2.5 5) (end 2.5 3.75) (layer B.SilkS) (width 0.15))
-    (pad 5 smd rect (at 0 -3.4 270) (size 4.6 1.1) (layers B.Cu B.Paste B.Mask)
+    (fp_text reference U3 (at 3.5 0 180) (layer F.SilkS)
+      (effects (font (size 1 1) (thickness 0.15)))
+    )
+    (fp_text value AUIPS7111S (at 15.25 -0.25 180) (layer F.Fab)
+      (effects (font (size 1 1) (thickness 0.15)))
+    )
+    (fp_line (start 14.1 5.65) (end -2.55 5.65) (layer F.CrtYd) (width 0.05))
+    (fp_line (start 14.1 -5.65) (end 14.1 5.65) (layer F.CrtYd) (width 0.05))
+    (fp_line (start 14.1 -5.65) (end -2.55 -5.65) (layer F.CrtYd) (width 0.05))
+    (fp_line (start -2.55 -5.65) (end -2.55 5.65) (layer F.CrtYd) (width 0.05))
+    (fp_line (start 2.5 5) (end 2.5 3.75) (layer F.SilkS) (width 0.15))
+    (fp_line (start 2.5 5) (end 4 5) (layer F.SilkS) (width 0.15))
+    (fp_line (start 2.5 -5) (end 4 -5) (layer F.SilkS) (width 0.15))
+    (fp_line (start 2.5 -5) (end 2.5 -3.75) (layer F.SilkS) (width 0.15))
+    (pad 5 smd rect (at 0 3.4 90) (size 4.6 1.1) (layers F.Cu F.Paste F.Mask)
       (net 8 /KSW/Out))
-    (pad 4 smd rect (at 0 -1.7 270) (size 4.6 1.1) (layers B.Cu B.Paste B.Mask)
+    (pad 4 smd rect (at 0 1.7 90) (size 4.6 1.1) (layers F.Cu F.Paste F.Mask)
       (net 8 /KSW/Out))
-    (pad 2 smd rect (at 0 1.7 270) (size 4.6 1.1) (layers B.Cu B.Paste B.Mask)
+    (pad 2 smd rect (at 0 -1.7 90) (size 4.6 1.1) (layers F.Cu F.Paste F.Mask)
       (net 6 "Net-(R4-Pad1)"))
-    (pad 3 smd rect (at 9.15 0 270) (size 9.4 10.8) (layers B.Cu B.Paste B.Mask)
+    (pad 3 smd rect (at 9.15 0 90) (size 9.4 10.8) (layers F.Cu F.Paste F.Mask)
       (net 7 /KSW/VCC))
-    (pad 3 smd rect (at 0 0 270) (size 4.6 1.1) (layers B.Cu B.Paste B.Mask)
+    (pad 3 smd rect (at 0 0 90) (size 4.6 1.1) (layers F.Cu F.Paste F.Mask)
       (net 7 /KSW/VCC))
-    (pad 1 smd rect (at 0 3.4 270) (size 4.6 1.1) (layers B.Cu B.Paste B.Mask)
+    (pad 1 smd rect (at 0 -3.4 90) (size 4.6 1.1) (layers F.Cu F.Paste F.Mask)
       (net 9 "Net-(D2-Pad1)"))
     (model TO_SOT_Packages_SMD.3dshapes/TO-263-5Lead.wrl
@@
       (net 1 GND))
   )
-  (segment (start 182.56 100.965) (end 182.56 102.77) (width 0.4) (layer F.Cu) (net 1))
-  (segment (start 182.56 102.77) (end 182.66 102.87) (width 0.4) (layer F.Cu) (net 1))
-  (segment (start 182.56 110.49) (end 182.56 112.98178) (width 0.4) (layer F.Cu) (net 1))
-  (segment (start 182.56 112.98178) (end 182.60822 113.03) (width 0.4) (layer F.Cu) (net 1))
+  (segment (start 182.60822 113.03) (end 182.60822 115.29822) (width 0.4) (layer F.Cu) (net 1))
+  (segment (start 182.60822 115.29822) (end 182.88 115.57) (width 0.4) (layer F.Cu) (net 1))
+  (via (at 182.88 115.57) (size 0.6) (drill 0.4) (layers F.Cu B.Cu) (net 1))
   (segment (start 178.816 107.315) (end 179.331644 107.315) (width 0.25) (layer F.Cu) (net 1))
   (segment (start 179.331644 107.315) (end 179.966644 106.68) (width 0.25) (layer F.Cu) (net 1))
   (segment (start 179.966644 106.68) (end 182.56 106.68) (width 0.4) (layer F.Cu) (net 1))
-  (segment (start 182.56 107.95) (end 182.56 110.49) (width 0.4) (layer F.Cu) (net 1))
-  (segment (start 182.56 106.68) (end 182.56 107.95) (width 0.4) (layer F.Cu) (net 1))
   (segment (start 182.56 104.14) (end 179.07 104.14) (width 0.4) (layer F.Cu) (net 1))
-  (segment (start 182.56 104.14) (end 182.56 102.97) (width 0.4) (layer F.Cu) (net 1))
-  (segment (start 182.56 105.41) (end 182.56 104.14) (width 0.4) (layer F.Cu) (net 1))
-  (segment (start 182.56 102.97) (end 182.66 102.87) (width 0.4) (layer F.Cu) (net 1))
-  (segment (start 182.56 105.41) (end 182.56 106.68) (width 0.4) (layer F.Cu) (net 1))
   (segment (start 178.005839 107.95) (end 177.8 108.155839) (width 0.4) (layer F.Cu) (net 2))
   (segment (start 177.8 109.36089) (end 177.395693 109.765197) (width 0.4) (layer F.Cu) (net 2))
@@
   (segment (start 177.17 104.14) (end 177.17 105.41) (width 0.4) (layer F.Cu) (net 5))
   (segment (start 180.66 105.41) (end 177.17 105.41) (width 0.4) (layer F.Cu) (net 5))
-  (segment (start 180.66 100.965) (end 177.689386 100.965) (width 0.4) (layer F.Cu) (net 6))
-  (segment (start 177.689386 100.965) (end 176.112817 99.388431) (width 0.4) (layer F.Cu) (net 6))
-  (segment (start 176.112817 99.388431) (end 176.112817 91.027825) (width 0.4) (layer F.Cu) (net 6))
-  (segment (start 176.112817 91.027825) (end 176.099642 91.01465) (width 0.4) (layer F.Cu) (net 6))
-  (segment (start 176.099642 91.01465) (end 176.099642 94.989642) (width 0.4) (layer B.Cu) (net 6))
-  (segment (start 176.099642 94.989642) (end 176.1 94.99) (width 0.4) (layer B.Cu) (net 6))
-  (via (at 176.099642 91.01465) (size 0.6) (drill 0.4) (layers F.Cu B.Cu) (net 6))
+  (segment (start 180.66 100.965) (end 174.808292 100.965) (width 0.4) (layer F.Cu) (net 6))
+  (segment (start 174.808292 100.965) (end 173.56 99.716708) (width 0.4) (layer F.Cu) (net 6))
+  (segment (start 173.56 99.716708) (end 173.56 92.71) (width 0.4) (layer F.Cu) (net 6))
   (segment (start 180.66 99.06) (end 180.66 100.965) (width 0.4) (layer F.Cu) (net 6))
-  (segment (start 180.594 116.078) (end 180.594 106.934) (width 0.6) (layer B.Cu) (net 7))
-  (segment (start 180.594 106.934) (end 177.8 104.14) (width 0.6) (layer B.Cu) (net 7))
-  (segment (start 180.60924 113.98) (end 180.60924 116.06276) (width 0.6) (layer F.Cu) (net 7))
-  (segment (start 180.60924 116.06276) (end 180.594 116.078) (width 0.6) (layer F.Cu) (net 7))
-  (via (at 180.594 116.078) (size 0.6) (drill 0.4) (layers F.Cu B.Cu) (net 7))
-  (segment (start 177.8 94.99) (end 177.8 104.14) (width 0.6) (layer B.Cu) (net 7))
+  (segment (start 178.12 102.14102) (end 173.819387 102.14102) (width 0.4) (layer F.Cu) (net 9))
+  (segment (start 173.819387 102.14102) (end 171.86 100.181633) (width 0.4) (layer F.Cu) (net 9))
+  (segment (start 171.86 100.181633) (end 171.86 92.71) (width 0.4) (layer F.Cu) (net 9))
   (segment (start 178.12 102.14102) (end 179.255952 102.14102) (width 0.4) (layer F.Cu) (net 9))
   (segment (start 179.255952 102.14102) (end 179.984932 102.87) (width 0.4) (layer F.Cu) (net 9))
   (segment (start 179.984932 102.87) (end 180.56 102.87) (width 0.4) (layer F.Cu) (net 9))
-  (segment (start 178.12 102.14102) (end 176.573784 102.14102) (width 0.4) (layer F.Cu) (net 9))
-  (segment (start 174.343846 91.185954) (end 174.31822 91.160328) (width 0.4) (layer F.Cu) (net 9))
-  (segment (start 176.573784 102.14102) (end 174.343846 99.911082) (width 0.4) (layer F.Cu) (net 9))
-  (segment (start 174.343846 99.911082) (end 174.343846 91.185954) (width 0.4) (layer F.Cu) (net 9))
-  (segment (start 174.31822 91.160328) (end 174.31822 94.90822) (width 0.4) (layer B.Cu) (net 9))
-  (segment (start 174.31822 94.90822) (end 174.4 94.99) (width 0.4) (layer B.Cu) (net 9))
-  (via (at 174.31822 91.160328) (size 0.6) (drill 0.4) (layers F.Cu B.Cu) (net 9))
+  (zone (net 1) (net_name GND) (layer B.Cu) (hatch edge 0.508)
+    (connect_pads (clearance 1))
+    (min_thickness 0.254)
+    (fill yes (arc_segments 16) (thermal_gap 0.508) (thermal_bridge_width 0.508))
+    (polygon
+      (pts
+        (xy 168.91 66.04) (xy 168.91 120.65) (xy 184.15 120.65) (xy 184.15 66.04)
+      )
+    )
+  )
+  (zone (net 7) (net_name /KSW/VCC) (layer F.Cu) (hatch edge 0.508)
+    (connect_pads (clearance 0.508))
+    (min_thickness 0.254)
+    (fill yes (arc_segments 16) (thermal_gap 0.508) (thermal_bridge_width 0.508))
+    (polygon
+      (pts
+        (xy 184.15 120.65) (xy 184.15 66.04) (xy 168.91 66.04) (xy 168.91 120.65)
+      )
+    )
+  )
 )

Commit message: test
Parts:
- removed Q1: BC849, TO_SOT_Packages_SMD:SOT-23
- removed R3: 5k, Resistors_SMD:R_0805
- removed R4: 10k, Resistors_SMD:R_0805
- removed Rfib1: R, Resistors_SMD:R_0805
- removed U2: LM3480-3.3, TO_SOT_Packages_SMD:SOT-23
- added D1: D_Small, Diodes_SMD:D_0805, F.Cu at (210.1, 69.9)
- added P10: CONN_01X02_Reed, Pin_Headers:Pin_Header_Straight_1x02, F.Cu at (221.0, 55.9)
- added P4: CONN_01X03, Pin_Headers:Pin_Header_Straight_1x03, F.Cu at (205.7, 86.4)
- added P5: CONN_01X03, Pin_Headers:Pin_Header_Straight_1x03, F.Cu at (195.6, 86.4)
- added P6: CONN_XT60_Female, KiCad-Dev:XT60, F.Cu at (217.2, 76.2)
- added P7: CONN_01X03, Pin_Headers:Pin_Header_Straight_1x03, F.Cu at (205.7, 104.1)
- added P8: CONN_01X03, Pin_Headers:Pin_Header_Straight_1x03, F.Cu at (195.6, 104.1)
- added P9: CONN_XT60_Female, KiCad-Dev:XT60, F.Cu at (217.2, 94.0)
- added Q_NPN1: BC849, TO_SOT_Packages_SMD:SOT-23, F.Cu at (210.1, 73.7)
- added Q_NPN2: BC849, TO_SOT_Packages_SMD:SOT-23, F.Cu at (209.6, 92.6)
- added R_fib1: R, Resistors_SMD:R_0805, F.Cu at (187.6, 74.9)
- added R_fib2: R, Resistors_SMD:R_0805, F.Cu at (190.5, 94.0)
- added R_pulldown1: 5k, Resistors_SMD:R_0805, F.Cu at (210.1, 80.1)
- added R_pulldown2: 5k, Resistors_SMD:R_0805, F.Cu at (210.1, 82.6)
- added R_pulldown3: 5k, Resistors_SMD:R_0805, F.Cu at (210.1, 76.9)
- added R_pulldown4: 5k, Resistors_SMD:R_0805, F.Cu at (209.6, 99.1)
- added R_pulldown5: 5k, Resistors_SMD:R_0805, F.Cu at (209.6, 101.6)
- added R_pulldown6: 5k, Resistors_SMD:R_0805, F.Cu at (209.6, 95.2)
- added U4: AUIPS7111S, TO_SOT_Packages_SMD:TO-263-5Lead, B.Cu at (209.8, 95.2)
- added U_and_gate1: 74LVC1G08, TO_SOT_Packages_SMD:SOT-353, F.Cu at (205.1, 79.4)
- added U_and_gate2: 74LVC1G08, TO_SOT_Packages_SMD:SOT-353, F.Cu at (205.7, 97.8)
- P1, P2: value CONN_01X02 -> CONN_XT60_Male; footprint Pin_Headers:Pin_Header_Straight_1x02 -> KiCad-Dev:XT60
- R1, R2: value 5k -> 10k
- U1: value 74LVC1G08 -> ARDUINO_MICRO_SHIELD; footprint TO_SOT_Packages_SMD:SOT-353 -> arduino:ARDUINO_MICRO_SHIELD
- U3: moved to B.Cu
- moved U1 71.3 mm to (216.9, 48.3)
- moved P2 54.6 mm to (163.8, 59.7)
- moved U3 37.8 mm to (209.8, 77.5), turned to 180 degrees
- moved R1 36.1 mm to (188.0, 72.4)
- moved D2 30.7 mm to (209.6, 90.2)
- moved P1 25.6 mm to (163.8, 94.0), turned to 90 degrees
- moved R2 21.0 mm to (190.5, 91.4)
Connections:
- net /KSW/Out renamed /KSW1/Out
- D2 pad 1: Net-(D2-Pad1) -> /KSW2/AUIPS7111S_IN
- P1 pad 1: Net-(P1-Pad1) -> VCC_8..50V
- P1 pad 2: /KSW/3.3V -> GND
- P2 pad 1: Net-(P2-Pad1) -> VCC_7..12V
- P2 pad 2: /KSW/3.3V -> GND
- R1 pad 1: Net-(P1-Pad1) -> Net-(R1-Pad1)
- R1 pad 2: GND -> /A0
- R2 pad 1: Net-(P2-Pad1) -> Net-(R2-Pad1)
- R2 pad 2: GND -> /A1
- U1 pad 2: Net-(P1-Pad1) -> (no net)
- U1 pad 3: GND -> (no net)
- U1 pad 4: Net-(Q1-Pad1) -> (no net)
- U1 pad 5: /KSW/3.3V -> /Enable1
- U3 pad 1: Net-(D2-Pad1) -> /KSW1/AUIPS7111S_IN
- U3 pad 2: Net-(R4-Pad1) -> Net-(R1-Pad1)
- U3 pad 3: /KSW/VCC -> VCC_8..50V
Routing:
- net GND: track 10.1 -> 63.7 mm, vias 1 -> 0
- net /KSW/3.3V: track 27.2 -> 0.00 mm
- net /Arduino_3.3V: track 0.00 -> 19.2 mm
- net Net-(D2-Pad1): track 17.3 -> 0.00 mm
- net Net-(R4-Pad1): track 16.5 -> 0.00 mm
- net Net-(P1-Pad1): track 16.0 -> 0.00 mm
- net Net-(P5-Pad2): track 0.00 -> 15.4 mm
- net Net-(P2-Pad1): track 10.6 -> 0.00 mm
- net Net-(Q_NPN1-Pad1): track 0.00 -> 9.64 mm
- net Net-(P4-Pad2): track 0.00 -> 9.22 mm
- net /KSW1/AUIPS7111S_IN: track 0.00 -> 7.54 mm, vias 0 -> 1
- net Net-(Q1-Pad1): track 7.05 -> 0.00 mm
- net /KSW2/AUIPS7111S_IN: track 0.00 -> 4.99 mm, vias 0 -> 1
- added copper zone on B.Cu, net /KSW1/Out
- added copper zone on B.Cu, net /KSW2/Out
- added copper zone on Ground.Cu, net GND
- added copper zone on B.Cu, net VCC_8..50V
- removed copper zone on F.Cu, net /KSW/VCC
- removed copper zone on B.Cu, net GND
Other:
- copper layers 2 -> 4

Commit message: test
Parts:
- added P3: CONN_01X02, Pin_Headers:Pin_Header_Straight_1x02, F.Cu at (7.62, 3.81)
- added R3: 5k, Resistors_SMD:R_0805, F.Cu at (205.7, 74.9)
- added R4: 5k, Resistors_SMD:R_0805, F.Cu at (205.7, 92.7)
- added U2: WPMDH1100501S, we:WPMDH1100xx1S, F.Cu at (19.1, 3.81)
- P4, P5, P7, P8: footprint Pin_Headers:Pin_Header_Straight_1x03 -> Pin_Headers:Pin_Header_Angled_1x03
- R1, R2, R_fib1, R_fib2: moved to B.Cu
- moved P10 62.1 mm to (189.2, 109.2), turned to 90 degrees
- moved R_fib1 28.3 mm to (215.9, 73.7), turned to 270 degrees
- moved R_fib2 25.5 mm to (215.9, 91.4), turned to 270 degrees
- moved R1 25.4 mm to (213.4, 73.7), turned to 90 degrees
- moved R2 22.9 mm to (213.4, 91.4), turned to 90 degrees
- moved P4 10.2 mm to (195.6, 86.4)
- moved P7 10.2 mm to (195.6, 104.1)
- moved P5 8.89 mm to (186.7, 86.4)
- moved P8 8.89 mm to (186.7, 104.1)
- moved P6 3.81 mm to (221.0, 76.2)
- moved P9 3.81 mm to (221.0, 94.0)
- moved D1 2.54 mm to (209.6, 72.4)
- moved Q_NPN1 1.34 mm to (209.6, 74.9)
- moved R_pulldown4 1.27 mm to (209.6, 97.8)
- moved R_pulldown5 1.27 mm to (209.6, 100.3)
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Connections:
- R_pulldown3 pad 1: Net-(Q_NPN1-Pad1) -> Net-(R3-Pad2)
- R_pulldown6 pad 1: Net-(Q_NPN2-Pad1) -> Net-(R4-Pad2)
- U_and_gate1 pad 4: Net-(Q_NPN1-Pad1) -> Net-(R3-Pad2)
- U_and_gate2 pad 4: Net-(Q_NPN2-Pad1) -> Net-(R4-Pad2)
Routing:
- net /Arduino_3.3V: track 19.2 -> 92.4 mm
- net /Enable1: track 0.00 -> 64.1 mm
- net /Enable0: track 0.00 -> 34.7 mm
- net /A1: track 0.00 -> 29.8 mm, vias 0 -> 1
- net Net-(P8-Pad2): track 0.00 -> 22.1 mm
- net GND: track 63.7 -> 85.3 mm
- net VCC_8..50V: track 0.00 -> 18.3 mm
- net Reed: track 0.00 -> 17.8 mm
- net Net-(P7-Pad2): track 0.00 -> 16.7 mm
- net /A0: track 0.00 -> 14.3 mm, vias 0 -> 1
- net Net-(P4-Pad2): track 9.22 -> 18.7 mm
- net Net-(R4-Pad2): track 0.00 -> 8.28 mm
- net Net-(R3-Pad2): track 0.00 -> 8.28 mm
- net Net-(R2-Pad1): track 0.00 -> 8.11 mm
- net Net-(R1-Pad1): track 0.00 -> 8.11 mm
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
Commit message: test
Parts:
- moved P3 173.4 mm to (177.8, 36.8)
- moved U2 173.4 mm to (189.2, 36.8)
Routing:
- net /Enable1: track 64.1 -> 67.2 mm
Changed lines of the file:
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@@
   (general
     (links 68)
-    (no_connects 18)
-    (area 2.586667 -2.265 228.405 116.44381)
+    (no_connects 10)
+    (area 156.505 30.755 228.405 116.44381)
     (thickness 1.6)
     (drawings 0)
-    (tracks 143)
+    (tracks 142)
     (zones 0)
     (modules 32)
@@
   )
   (setup
-    (last_trace_width 0.6)
+    (last_trace_width 0.4)
     (user_trace_width 0.3)
     (user_trace_width 0.4)
@@
     (pad_to_mask_clearance 0.2)
     (aux_axis_origin 0 0)
-    (visible_elements 7FFFFFFF)
+    (visible_elements 7FFFEFFF)
     (pcbplotparams
       (layerselection 0x00030_80000001)
@@
   )
   (module Pin_Headers:Pin_Header_Straight_1x02 (layer F.Cu)
-    (at 7.62 3.81)
+    (at 177.8 36.83)
     (descr "Through hole pin header")
     (tags "pin header")
@@
   )
   (module we:WPMDH1100xx1S (layer F.Cu)
-    (at 19.05 3.81)
+    (at 189.23 36.83)
     (fp_text reference U2 (at 0 -5.08) (layer Dwgs.User)
       (effects (font (size 0.762 0.762) (thickness 0.1524)))
@@
   (segment (start 208.6 86.04) (end 208.6 82.620685) (width 0.3) (layer F.Cu) (net 15) (status 20))
   (segment (start 186.69 104.14) (end 186.69 86.36) (width 0.4) (layer In2.Cu) (net 16))
+  (segment (start 179.07 60.96) (end 190.5 49.53) (width 0.4) (layer In2.Cu) (net 17))
+  (segment (start 179.07 67.31) (end 179.07 60.96) (width 0.4) (layer In2.Cu) (net 17))
+  (segment (start 196.85 85.09) (end 179.07 67.31) (width 0.4) (layer In2.Cu) (net 17))
+  (segment (start 195.58 96.52) (end 196.85 95.25) (width 0.4) (layer In2.Cu) (net 17))
+  (segment (start 196.85 95.25) (end 196.85 85.09) (width 0.4) (layer In2.Cu) (net 17))
   (segment (start 195.58 104.14) (end 195.58 96.52) (width 0.4) (layer In2.Cu) (net 17))
-  (segment (start 195.58 96.52) (end 204.47 87.63) (width 0.4) (layer In2.Cu) (net 17))
-  (segment (start 204.47 87.63) (end 204.47 82.249048) (width 0.4) (layer In2.Cu) (net 17))
-  (segment (start 204.47 82.249048) (end 191.798244 69.577292) (width 0.4) (layer In2.Cu) (net 17))
-  (segment (start 190.5 57.15) (end 190.5 49.53) (width 0.4) (layer In2.Cu) (net 17))
-  (segment (start 191.798244 69.577292) (end 191.798244 58.448244) (width 0.4) (layer In2.Cu) (net 17))
-  (segment (start 191.798244 58.448244) (end 190.5 57.15) (width 0.4) (layer In2.Cu) (net 17))
   (segment (start 198.12 104.14) (end 198.12 104.789527) (width 0.3) (layer F.Cu) (net 18))
   (segment (start 198.12 104.789527) (end 199.345773 106.0153) (width 0.3) (layer F.Cu) (net 18))

Commit message: test
Routing:
- net /Arduino_3.3V: track 92.4 -> 91.7 mm
Changed lines of the file:
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@@
-(kicad_pcb (version 4) (host pcbnew 4.0.4-stable)
+(kicad_pcb (version 4) (host pcbnew 4.0.4+e1-6308~48~ubuntu16.04.1-stable)
   (general
     (links 68)
@@
   )
   (setup
-    (last_trace_width 0.4)
+    (last_trace_width 0.25)
     (user_trace_width 0.3)
     (user_trace_width 0.4)
@@
   (segment (start 207.34 75.88) (end 206.69 75.23) (width 0.3) (layer F.Cu) (net 2) (status 20))
   (segment (start 206.69 75.23) (end 206.69 74.93) (width 0.3) (layer F.Cu) (net 2) (status 30))
+  (segment (start 191.77 86.36) (end 191.77 84.801208) (width 0.3) (layer F.Cu) (net 3))
+  (segment (start 191.77 84.801208) (end 194.656208 81.915) (width 0.3) (layer F.Cu) (net 3))
+  (segment (start 194.656208 81.915) (end 202.565 81.915) (width 0.3) (layer F.Cu) (net 3))
   (segment (start 191.77 86.36) (end 191.77 104.14) (width 0.6) (layer In2.Cu) (net 3))
   (segment (start 175.26 65.022) (end 175.26 67.384251) (width 0.6) (layer In2.Cu) (net 3))
@@
   (segment (start 204.724 81.0974) (end 203.9064 81.915) (width 0.3) (layer F.Cu) (net 3))
   (segment (start 203.9064 81.915) (end 202.565 81.915) (width 0.3) (layer F.Cu) (net 3))
-  (segment (start 191.77 86.36) (end 191.77 83.530057) (width 0.3) (layer F.Cu) (net 3) (status 10))
-  (segment (start 191.77 83.530057) (end 193.385057 81.915) (width 0.3) (layer F.Cu) (net 3))
-  (segment (start 193.385057 81.915) (end 202.565 81.915) (width 0.3) (layer F.Cu) (net 3))
   (segment (start 202.565 81.915) (end 200.66 83.82) (width 0.3) (layer F.Cu) (net 3))
   (segment (start 200.66 83.82) (end 200.66 86.36) (width 0.3) (layer F.Cu) (net 3) (status 20))
@@
     (polygon
       (pts
-        (xy 226.06 44.45) (xy 160.02 44.45) (xy 160.02 106.68) (xy 226.06 106.68)
+        (xy 226.06 48.26) (xy 160.02 48.26) (xy 160.02 106.68) (xy 226.06 106.68)
       )
     )
@@
     (polygon
       (pts
-        (xy 207.645 76.835) (xy 226.06 76.835) (xy 226.06 83.185) (xy 207.645 83.185)
+        (xy 208.28 78.74) (xy 226.06 78.74) (xy 226.06 81.28) (xy 208.28 81.28)
       )
     )
