File: LTC6802-2/main.sch (KiCad schematic (older format))
At the start: 10 parts, among them P1 CONN_01X13, P2 CONN_01X04, P3 CONN_01X04, P4 CONN_01X06, P5 CONN_01X13, U1 LTC6802-2

Commit message: test
Connections:
- net CSBI: no longer P4.5 (P5), R2.1, U1.42 (SDI)
- new net SDI: P4.5 (P5), R2.1, U1.42 (SDI)
Changed lines of the file:
@@
 LIBS:dev_switch
 LIBS:ltc6802
+LIBS:main-cache
 EELAYER 25 0
 EELAYER END
@@
 SDO
 Text Label 5600 2900 0    60   ~ 0
-CSBI
+SDI
 Text Label 5600 3000 0    60   ~ 0
 SCKI
@@
 GPIO1
 Wire Wire Line
-	4700 5300 4700 5950
-Wire Wire Line
-	4700 5050 4700 5300
+	4700 5050 4700 5950
 Connection ~ 4750 5000
 Text Label 4500 5250 1    60   ~ 0

Commit message: test
Parts:
- removed U1: LTC6802-2, KiCad-Dev:SSOP-44, symbol LTC6802-2
- added U?: LTC6802-2, symbol LTC6802-2
Connections:
- wire segments 74 -> 75
Other:
- moved on the sheet: C1, C2, P1, P2, P3, P4, P5, R1, R2
