File: pdb2/channel.sch (KiCad schematic (older format))
At the start: 3 parts, among them P1 CONN_XT60, P2 CONN_XT60, P3 CONN_02X03

Commit message: test
Parts:
- P1: footprint KiCad-Dev:XT60 -> KiCad-Dev:XT60_Horizontal1
- P2: footprint KiCad-Dev:XT60 -> KiCad-Dev:XT60_Horizontal2
Changed lines of the file:
@@
 F 0 "P1" H 1350 3000 60  0000 C CNN
 F 1 "CONN_XT60" H 1350 2700 60  0000 C CNN
-F 2 "KiCad-Dev:XT60" H 1250 3000 60  0001 C CNN
+F 2 "KiCad-Dev:XT60_Horizontal1" H 1250 3000 60  0001 C CNN
 F 3 "" H 1250 3000 60  0001 C CNN
 	1    1350 2850
@@
 F 0 "P2" H 1350 3450 60  0000 C CNN
 F 1 "CONN_XT60" H 1350 3150 60  0000 C CNN
-F 2 "KiCad-Dev:XT60" H 1250 3450 60  0001 C CNN
+F 2 "KiCad-Dev:XT60_Horizontal2" H 1250 3450 60  0001 C CNN
 F 3 "" H 1250 3450 60  0001 C CNN
 	1    1350 3300
