File: pdb2/kill_sw.sch (KiCad schematic (older format))
At the start: 11 parts, among them P4 CONN_01X02, P5 CONN_01X02, Q2 BUK9Y4R8-60E, U4 LM3480-3.3, U5 74LVC1G08, U7 MIC5014, U8 NSI45020AT1G

Commit message: test
Parts:
- added R5: R, Resistors_SMD:R_0603, symbol R
- C3: footprint Capacitors_ThroughHole:C_Radial_D5_L6_P2.5 -> Capacitors_ThroughHole:C_Axial_D5_L11_P18
Connections:
- net GND: now also R5.2
- net at U5.4 (Y), U7.2 (Input): now also R5.1
Changed lines of the file:
@@
 F 0 "C3" H 5175 3600 50  0000 L CNN
 F 1 "CP" H 5175 3400 50  0000 L CNN
-F 2 "Capacitors_ThroughHole:C_Radial_D5_L6_P2.5" H 5188 3350 50  0001 C CNN
+F 2 "Capacitors_ThroughHole:C_Axial_D5_L11_P18" H 5188 3350 50  0001 C CNN
 F 3 "" H 5150 3500 50  0000 C CNN
 	1    5150 3500
@@
 	2150 4550 2150 4750
 Connection ~ 2150 4750
+$Comp
+L R R5
+U 1 1 582F017F
+P 3150 4400
+F 0 "R5" V 3230 4400 50  0000 C CNN
+F 1 "R" V 3150 4400 50  0000 C CNN
+F 2 "Resistors_SMD:R_0603" V 3080 4400 50  0001 C CNN
+F 3 "" H 3150 4400 50  0000 C CNN
+	1    3150 4400
+	1    0    0    -1
+$EndComp
+Wire Wire Line
+	3150 4550 3150 4750
+Connection ~ 3150 4750
+Wire Wire Line
+	3150 4250 3150 4050
+Connection ~ 3150 4050
 $EndSCHEMATC
