File: pdb4/kill_sw.sch (KiCad schematic (older format))
At the start: 12 parts, among them P5 CONN_01X03, P6 CONN_01X03, Q1 BUK9Y4R8-60E, U2 74LVC1G08, U3 MIC5014, U4 NSI45020AT1G

Commit message: test
Parts:
- C1: footprint Capacitors_SMD:c_elec_8x10 -> Capacitors_SMD:c_elec_4x4.5
Changed lines of the file:
@@
 F 0 "C1" H 7125 3650 50  0000 L CNN
 F 1 "CP" H 7125 3450 50  0000 L CNN
-F 2 "Capacitors_SMD:c_elec_8x10" H 7138 3400 50  0001 C CNN
+F 2 "Capacitors_SMD:c_elec_4x4.5" H 7138 3400 50  0001 C CNN
 F 3 "" H 7100 3550 50  0000 C CNN
 	1    7100 3550
