File: pdb4/pdb1.kicad_pcb (KiCad board)
At the start: 4 copper layers, 47 parts, among them P1 CONN_XT60_Male, P2 CONN_02X06, P3 CONN_02X06, P4 CONN_XT60_Female, P5 CONN_01X03, P6 CONN_01X03, P7 CONN_XT60_Female, P8 CONN_01X03, P9 CONN_01X03, Q1 BUK9Y4R8-60E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

Commit message: test
Parts:
- added P10: CONN_02X06, Pin_Headers:Pin_Header_Straight_2x06, F.Cu at (166.4, 63.5)
- added P11: CONN_02X06, Pin_Headers:Pin_Header_Straight_2x06, F.Cu at (219.7, 63.5)
- C1, C4: footprint Capacitors_SMD:c_elec_8x10 -> Capacitors_SMD:c_elec_4x4.5
- P1: footprint KiCad-Dev:CONN_XT60_Male_Horizontal -> KiCad-Dev:CONN_XT60_Male1_Horizontal; moved to F.Cu
- moved D2 56.5 mm to (222.2, 92.1)
- moved U4 55.9 mm to (227.3, 92.1), turned to 0 degrees
- moved R5 53.2 mm to (222.2, 90.2)
- moved U6 32.5 mm to (212.1, 82.5), turned to 0 degrees
- moved R8 30.5 mm to (205.7, 81.3), turned to 270 degrees
- moved P2 30.3 mm to (246.4, 63.5), turned to 90 degrees
- moved D3 30.2 mm to (208.3, 81.3), turned to 270 degrees
- moved P1 23.1 mm to (170.2, 80.1), turned to 270 degrees
- moved R6 22.2 mm to (199.4, 97.8)
- moved U5 22.1 mm to (199.4, 97.6)
- moved R13 21.9 mm to (199.4, 80.0)
- moved U10 21.9 mm to (199.4, 80.0)
- moved F1 20.6 mm to (210.8, 104.1)
- moved F2 19.9 mm to (210.8, 86.4)
- moved C2 19.7 mm to (199.1, 102.7)
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Connections:
- C3 pad 1: /channel0/Current_Feedback -> /Current_Feedback0
- C6 pad 1: /channel1/Current_Feedback -> /Current_Feedback1
- P2 pad 3: /channel0/Current_Feedback -> /Enabled_SW0
- P2 pad 5: /channel1/Current_Feedback -> /Enabled_SW1
- P3 pad 3: /channel0/Enable_MCU -> /Enabled_Fuse0
- P3 pad 5: /channel1/Enable_MCU -> /Enabled_Fuse1
- P5 pad 3: (no net) -> /channel0/Enable_Reed
- P6 pad 3: /channel0/Enable_MCU -> /Enable_MCU0
- P8 pad 3: (no net) -> /channel0/Enable_Reed
- P9 pad 3: /channel1/Enable_MCU -> /Enable_MCU1
- R1 pad 1: (no net) -> /Enabled_Fuse0
- R12 pad 1: (no net) -> /Enabled_SW1
- R14 pad 1: /channel1/Current_Feedback -> /Current_Feedback1
- R5 pad 1: (no net) -> /Enabled_SW0
- R7 pad 1: /channel0/Current_Feedback -> /Current_Feedback0
- R8 pad 1: (no net) -> /Enabled_Fuse1
- U10 pad 1: /channel1/Current_Feedback -> /Current_Feedback1
- U5 pad 1: /channel0/Current_Feedback -> /Current_Feedback0
Routing:
- net GND: track 64.4 -> 0.00 mm
- net /channel1/3.3V: track 17.5 -> 0.00 mm
- net /channel0/3.3V: track 17.4 -> 0.00 mm
- net Net-(P8-Pad2): track 17.0 -> 0.00 mm
- net Net-(P5-Pad2): track 16.8 -> 0.00 mm
- net Net-(P9-Pad2): track 12.2 -> 0.00 mm
- net Net-(P6-Pad2): track 10.7 -> 0.00 mm
- net /channel1/fuse/in+: track 8.37 -> 0.00 mm
- net /channel0/fuse/in+: track 8.37 -> 0.00 mm
- net Net-(R4-Pad1): track 6.80 -> 0.00 mm
- net Net-(R11-Pad1): track 6.55 -> 0.00 mm
