File: pdb4/pdb1.sch (KiCad schematic (older format))
At the start: 3 parts, among them P1 CONN_XT60_Male, P2 CONN_02X06, P3 CONN_02X06

Commit message: test
Parts:
- added P10, P11: CONN_02X06, Pin_Headers:Pin_Header_Straight_2x06, symbol CONN_02X06
Connections:
- net GND: now also P10.1 (P1), P11.1 (P1)
- net channel0/Current_Feedback renamed Enabled_SW0
- net channel0/Enable_MCU renamed Enabled_Fuse0
- net channel1/Current_Feedback renamed Enabled_SW1
- net channel1/Enable_MCU renamed Enabled_Fuse1
- new net Current_Feedback0: P10.3 (P3)
- new net Current_Feedback1: P10.5 (P5)
- new net Enable_MCU0: P11.3 (P3)
- new net Enable_MCU1: P11.5 (P5)
Other:
- moved on the sheet: P1, P2, P3
