File: PCA9698/PCA9698.kicad_pcb (KiCad board)
At the start: 4 copper layers, 8 parts, among them U1 WPMDH1100501S, U2 PCA9698, U3 ADS7828, U4 LTC6802-2, U5 SC18IS602B, U6 LTC6802-2, U7 LTC6802-2, U8 LTC6802-2

Commit message: test
Parts:
- U1: value WPMDH1100501S -> LTC6802-2; footprint we:WPMDH1100xx1S -> KiCad-Dev:SSOP-44
- U8: value LTC6802-2 -> WPMDH1100331S; footprint KiCad-Dev:SSOP-44 -> we:WPMDH1100xx1S
- moved U5 46.6 mm to (203.8, 81.3)
- moved U1 38.2 mm to (222.9, 94.0)
- moved U8 36.4 mm to (198.1, 61.0)
- moved U6 33.0 mm to (213.4, 94.0)
- moved U4 23.5 mm to (203.8, 94.0)
- moved U3 18.5 mm to (194.3, 81.9)
- moved U7 14.0 mm to (194.3, 94.0)
Connections:
- U1 pad 1: (no net) -> +3V3
- U6 pad 1: (no net) -> +3V3
- U8 pad 2: (no net) -> GND
- U8 pad 3: (no net) -> +3V3

Commit message: test
Parts:
- removed U1, U4, U6, U7: LTC6802-2, KiCad-Dev:SSOP-44
- removed U3: ADS7828, Housings_SSOP:TSSOP-16_4.4x5mm_Pitch0.65mm
- removed U5: SC18IS602B, Housings_SSOP:TSSOP-16_4.4x5mm_Pitch0.65mm
- removed U8: WPMDH1100331S, we:WPMDH1100xx1S
- added D1: LED, LEDs:LED_0805, F.Cu at (176.5, 62.2)
- added P1: Power connector, Pin_Headers:Pin_Header_Straight_1x10, B.Cu at (167.6, 43.2)
- added P10: CONN_01X03, Pin_Headers:Pin_Header_Straight_1x03, F.Cu at (161.3, 53.3)
- added P2: CONN_01X03, Pin_Headers:Pin_Header_Straight_1x03, F.Cu at (171.4, 88.9)
- added P3: I2C connector, Pin_Headers:Pin_Header_Straight_1x05, B.Cu at (161.3, 43.2)
- added P4: CONN_01X03, Pin_Headers:Pin_Header_Straight_1x03, B.Cu at (167.6, 88.9)
- added P5: GPIO 0, Pin_Headers:Pin_Header_Straight_1x08, B.Cu at (137.2, 48.3)
- added P6: GPIO 1, Pin_Headers:Pin_Header_Straight_1x08, B.Cu at (137.2, 71.1)
- added P7: GPIO 2, Pin_Headers:Pin_Header_Straight_1x08, B.Cu at (144.8, 99.1)
- added P8: GPIO 3, Pin_Headers:Pin_Header_Straight_1x08, B.Cu at (200.7, 88.9)
- added P9: GPIO 4, Pin_Headers:Pin_Header_Straight_1x08, B.Cu at (200.7, 66.0)
- added R1: R, Resistors_SMD:R_0805, F.Cu at (176.5, 58.4)
- moved U2 3.59 mm to (170.2, 73.7)
Connections:
- U2 pad 1: (no net) -> /SDA
- U2 pad 10: (no net) -> Net-(P5-Pad7)
- U2 pad 12: (no net) -> Net-(P5-Pad8)
- U2 pad 13: (no net) -> Net-(P6-Pad1)
- U2 pad 14: (no net) -> Net-(P6-Pad2)
- U2 pad 15: (no net) -> Net-(P6-Pad3)
- U2 pad 16: (no net) -> Net-(P6-Pad4)
- U2 pad 17: (no net) -> Net-(P6-Pad5)
- U2 pad 19: (no net) -> Net-(P6-Pad6)
- U2 pad 2: (no net) -> /SCL
- U2 pad 20: (no net) -> Net-(P6-Pad7)
- U2 pad 21: (no net) -> Net-(P6-Pad8)
- U2 pad 22: (no net) -> Net-(P7-Pad1)
- U2 pad 24: (no net) -> Net-(P7-Pad2)
- U2 pad 25: (no net) -> Net-(P7-Pad3)
- U2 pad 26: (no net) -> Net-(P7-Pad4)
- U2 pad 27: (no net) -> Net-(P4-Pad3)
- U2 pad 28: (no net) -> Net-(P4-Pad2)
- U2 pad 29: (no net) -> Net-(P4-Pad1)
- U2 pad 3: (no net) -> Net-(P5-Pad1)
- U2 pad 30: (no net) -> /OE
- U2 pad 31: (no net) -> Net-(P7-Pad5)
- U2 pad 32: (no net) -> Net-(P7-Pad6)
- U2 pad 33: (no net) -> Net-(P7-Pad7)
- U2 pad 35: (no net) -> Net-(P7-Pad8)
- U2 pad 36: (no net) -> Net-(P8-Pad1)
- U2 pad 37: (no net) -> Net-(P8-Pad2)
- U2 pad 38: (no net) -> Net-(P8-Pad3)
- U2 pad 4: (no net) -> Net-(P5-Pad2)
- U2 pad 40: (no net) -> Net-(P8-Pad4)
- U2 pad 41: (no net) -> Net-(P8-Pad5)
- U2 pad 42: (no net) -> Net-(P8-Pad6)
- U2 pad 43: (no net) -> Net-(P8-Pad7)
- U2 pad 44: (no net) -> Net-(P8-Pad8)
- U2 pad 45: (no net) -> Net-(P9-Pad1)
- U2 pad 47: (no net) -> Net-(P9-Pad2)
- U2 pad 48: (no net) -> Net-(P9-Pad3)
- U2 pad 49: (no net) -> Net-(P9-Pad4)
- U2 pad 5: (no net) -> Net-(P5-Pad3)
- U2 pad 50: (no net) -> Net-(P9-Pad5)
- U2 pad 52: (no net) -> Net-(P9-Pad6)
- U2 pad 53: (no net) -> Net-(P9-Pad7)
- U2 pad 54: (no net) -> Net-(P9-Pad8)
- U2 pad 55: (no net) -> /INT
- U2 pad 56: (no net) -> /Reset
- U2 pad 7: (no net) -> Net-(P5-Pad4)
- U2 pad 8: (no net) -> Net-(P5-Pad5)
- U2 pad 9: (no net) -> Net-(P5-Pad6)
Routing:
- net +3V3: track 0.00 -> 413.7 mm
- net GND: track 0.00 -> 93.9 mm
- net Net-(P7-Pad5): track 0.00 -> 45.4 mm
- net Net-(P7-Pad6): track 0.00 -> 44.7 mm
- net Net-(P7-Pad7): track 0.00 -> 44.2 mm
- net Net-(P7-Pad8): track 0.00 -> 44.0 mm
- net /SCL: track 0.00 -> 40.4 mm
- net Net-(P5-Pad1): track 0.00 -> 37.4 mm
- net /SDA: track 0.00 -> 37.1 mm
- net Net-(P5-Pad2): track 0.00 -> 36.6 mm
- net Net-(P5-Pad3): track 0.00 -> 35.7 mm
- net Net-(P5-Pad4): track 0.00 -> 35.1 mm
- net Net-(P9-Pad8): track 0.00 -> 34.9 mm
- net Net-(P7-Pad1): track 0.00 -> 34.3 mm
- net Net-(P6-Pad8): track 0.00 -> 34.2 mm
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Other:
- board outline added: 76.2 x 71.1 mm
- board text added: "3.3V"
- board text added: "=KJ="
- board text added: "AD0..2"
- board text added: "GND"
- board text added: "INT"
- board text added: "IO0"
- board text added: "IO1"
- board text added: "IO3"
- board text added: "IO4"
- board text added: "OE"
- board text added: "RST"
- board text added: "SCL"
- board text added: "SDA"
