File: PCA9698/PCA9698.sch (KiCad schematic (older format))
At the start: 8 parts, among them U1 WPMDH1100501S, U2 PCA9698, U3 ADS7828, U4 LTC6802-2, U5 SC18IS602B, U6 LTC6802-2, U7 LTC6802-2, U8 LTC6802-2

Commit message: test
Parts:
- removed U1: WPMDH1100501S, we:WPMDH1100xx1S, symbol WPMDH1100501S
- removed U8: LTC6802-2, KiCad-Dev:SSOP-44, symbol LTC6802-2
- added U1: LTC6802-2, KiCad-Dev:SSOP-44, symbol LTC6802-2
- added U8: WPMDH1100331S, we:WPMDH1100xx1S, symbol WPMDH1100331S
- added U?: AUIPS7111S, symbol AUIPS7111S
Connections:
- net labels added: VCC
- wire segments 18 -> 23
Other:
- moved on the sheet: U2, U3, U5

Commit message: test
Parts:
- removed U1, U4, U6, U7: LTC6802-2, KiCad-Dev:SSOP-44, symbol LTC6802-2
- removed U3: ADS7828, Housings_SSOP:TSSOP-16_4.4x5mm_Pitch0.65mm, symbol ADS7828
- removed U5: SC18IS602B, Housings_SSOP:TSSOP-16_4.4x5mm_Pitch0.65mm, symbol SC18IS602B
- removed U8: WPMDH1100331S, we:WPMDH1100xx1S, symbol WPMDH1100331S
- removed U?: AUIPS7111S, symbol AUIPS7111S
- added D1: LED, LEDs:LED_0805, symbol LED
- added P1: Power connector, Pin_Headers:Pin_Header_Straight_1x10, symbol CONN_01X10
- added P10, P2, P4: CONN_01X03, Pin_Headers:Pin_Header_Straight_1x03, symbol CONN_01X03
- added P3: I2C connector, Pin_Headers:Pin_Header_Straight_1x05, symbol CONN_01X05
- added P5: GPIO 0, Pin_Headers:Pin_Header_Straight_1x08, symbol CONN_01X08
- added P6: GPIO 1, Pin_Headers:Pin_Header_Straight_1x08, symbol CONN_01X08
- added P7: GPIO 2, Pin_Headers:Pin_Header_Straight_1x08, symbol CONN_01X08
- added P8: GPIO 3, Pin_Headers:Pin_Header_Straight_1x08, symbol CONN_01X08
- added P9: GPIO 4, Pin_Headers:Pin_Header_Straight_1x08, symbol CONN_01X08
- added R1: R, Resistors_SMD:R_0805, symbol R
Connections:
- net +3V3: now also P1.10 (P10), P1.6 (P6), P1.7 (P7), P1.8 (P8), P1.9 (P9), P10.3 (P3), P2.3 (P3), R1.2
- net GND: now also P1.1 (P1), P1.2 (P2), P1.3 (P3), P1.4 (P4), P1.5 (P5), P10.1 (P1), P2.1 (P1), P3.1 (P1)
- net SDA: now reaches U2.1 (SDA)
- net SDA: now also P3.2 (P2), P3.3 (P3)
- net at U2.10 (IO_0_6): now also P5.7 (P7)
- net at U2.12 (IO_0_7): now also P5.8 (P8)
- net at U2.13 (IO_1_0): now also P6.1 (P1)
- net at U2.14 (IO_1_1): now also P6.2 (P2)
- net at U2.15 (IO_1_2): now also P6.3 (P3)
- net at U2.16 (IO_1_3): now also P6.4 (P4)
- net at U2.17 (IO_1_4): now also P6.5 (P5)
- net at U2.19 (IO_1_5): now also P6.6 (P6)
- net SCL: now reaches U2.2 (SCL)
- net SCL: now also P3.4 (P4), P3.5 (P5)
- net at U2.20 (IO_1_6): now also P6.7 (P7)
- net at U2.21 (IO_1_7): now also P6.8 (P8)
- net at U2.22 (IO_2_0): now also P7.1 (P1)
- net at U2.24 (IO_2_1): now also P7.2 (P2)
- net at U2.25 (IO_2_2): now also P7.3 (P3)
- net at U2.26 (IO_2_3): now also P7.4 (P4)
- net at U2.27 (AD0): now also P4.3 (P3)
- net at U2.28 (AD1): now also P4.2 (P2)
- net at U2.29 (AD2): now also P4.1 (P1)
- net at U2.3 (IO_0_0): now also P5.1 (P1)
- net OE: now reaches U2.30 (OE)
- net OE: now also P2.2 (P2)
- net at U2.31 (IO_2_4): now also P7.5 (P5)
- net at U2.32 (IO_2_5): now also P7.6 (P6)
- net at U2.33 (IO_2_6): now also P7.7 (P7)
- net at U2.35 (IO_2_7): now also P7.8 (P8)
- net at U2.36 (IO_3_0): now also P8.1 (P1)
- net at U2.37 (IO_3_1): now also P8.2 (P2)
- net at U2.38 (IO_3_2): now also P8.3 (P3)
- net at U2.4 (IO_0_1): now also P5.2 (P2)
- net at U2.40 (IO_3_3): now also P8.4 (P4)
- net at U2.41 (IO_3_4): now also P8.5 (P5)
- net at U2.42 (IO_3_5): now also P8.6 (P6)
- net at U2.43 (IO_3_6): now also P8.7 (P7)
- net at U2.44 (IO_3_7): now also P8.8 (P8)
- net at U2.45 (IO_4_0): now also P9.1 (P1)
- net at U2.47 (IO_4_1): now also P9.2 (P2)
- net at U2.48 (IO_4_2): now also P9.3 (P3)
- net at U2.49 (IO_4_3): now also P9.4 (P4)
- net at U2.5 (IO_0_2): now also P5.3 (P3)
- net at U2.50 (IO_4_4): now also P9.5 (P5)
- net at U2.52 (IO_4_5): now also P9.6 (P6)
- net at U2.53 (IO_4_6): now also P9.7 (P7)
- net at U2.54 (IO_4_7): now also P9.8 (P8)
- net INT: now reaches U2.55 (INT/SMBALERT)
- net INT: now also D1.1 (K)
- net Reset: now reaches U2.56 (RESET)
- net Reset: now also P10.2 (P2)
- net at U2.7 (IO_0_3): now also P5.4 (P4)
- net at U2.8 (IO_0_4): now also P5.5 (P5)
- net at U2.9 (IO_0_5): now also P5.6 (P6)
- new net: D1.2 (A), R1.1
