File: ADS7828/main.sch (KiCad schematic (older format))
At the start: 12 parts, among them P1 CONN_01X10, P2 Address 0, P3 Address 1, P4 I2C Connector, P5 Power Connector, U1 ADS7828

Commit message: test
Parts:
- P1: value CONN_01X10 -> Analog input connector
Connections:
- net SCL: now also P4.2 (P2); no longer P4.3 (P3)
- net SDA: now also P4.3 (P3); no longer P4.2 (P2)
Other:
- moved on the sheet: P2, P3, P4, P5
Changed lines of the file:
@@
 LIBS:dev_conn
 LIBS:dev_bjt
+LIBS:main-cache
 EELAYER 25 0
 EELAYER END
@@
 L CONN_01X03 P4
 U 1 1 5836BE61
-P 9400 2950
-F 0 "P4" H 9400 3150 50  0000 C CNN
-F 1 "I2C Connector" V 9500 2950 50  0000 C CNN
-F 2 "Pin_Headers:Pin_Header_Straight_1x03" H 9400 2950 50  0001 C CNN
-F 3 "" H 9400 2950 50  0000 C CNN
-	1    9400 2950
-	1    0    0    -1
-$EndComp
-Wire Wire Line
-	6750 2950 9200 2950
-Wire Wire Line
-	6750 3050 9200 3050
+P 8650 3050
+F 0 "P4" H 8650 3250 50  0000 C CNN
+F 1 "I2C Connector" V 8750 3050 50  0000 C CNN
+F 2 "Pin_Headers:Pin_Header_Straight_1x03" H 8650 3050 50  0001 C CNN
+F 3 "" H 8650 3050 50  0000 C CNN
+	1    8650 3050
+	1    0    0    1
+$EndComp
+Wire Wire Line
+	6750 2950 8000 2950
+Wire Wire Line
+	8000 2950 8450 2950
+Wire Wire Line
+	6750 3050 8250 3050
+Wire Wire Line
+	8250 3050 8450 3050
 $Comp
 L GND #PWR01
 U 1 1 5836BF45
-P 9050 2850
-F 0 "#PWR01" H 9050 2600 50  0001 C CNN
-F 1 "GND" H 9050 2700 50  0000 C CNN
-F 2 "" H 9050 2850 50  0000 C CNN
-F 3 "" H 9050 2850 50  0000 C CNN
-	1    9050 2850
-	0    1    1    0
-$EndComp
-Wire Wire Line
-	9050 2850 9200 2850
+P 8350 3150
+F 0 "#PWR01" H 8350 2900 50  0001 C CNN
+F 1 "GND" H 8350 3000 50  0000 C CNN
+F 2 "" H 8350 3150 50  0000 C CNN
+F 3 "" H 8350 3150 50  0000 C CNN
+	1    8350 3150
+	1    0    0    -1
+$EndComp
+Wire Wire Line
+	8350 3150 8450 3150
 $Comp
 L GND #PWR02
@@
 	6950 2850 6750 2850
 Wire Wire Line
-	6750 2750 7750 2750
+	6750 2750 7300 2750
+Wire Wire Line
+	7300 2750 7750 2750
 $Comp
 L R R2
@@
 Connection ~ 8000 2950
 Wire Wire Line
-	6850 1800 9700 1800
+	6850 1800 7300 1800
+Wire Wire Line
+	7300 1800 7750 1800
+Wire Wire Line
+	7750 1800 8000 1800
+Wire Wire Line
+	8000 1800 8250 1800
+Wire Wire Line
+	8250 1800 8450 1800
 $Comp
 L VCC #PWR03
@@
 L CONN_01X03 P2
 U 1 1 5836C619
-P 8650 3350
-F 0 "P2" H 8650 3550 50  0000 C CNN
-F 1 "Address 0" V 8750 3350 50  0000 C CNN
-F 2 "Pin_Headers:Pin_Header_Straight_1x03" H 8650 3350 50  0001 C CNN
-F 3 "" H 8650 3350 50  0000 C CNN
-	1    8650 3350
+P 8650 3750
+F 0 "P2" H 8650 3950 50  0000 C CNN
+F 1 "Address 0" V 8750 3750 50  0000 C CNN
+F 2 "Pin_Headers:Pin_Header_Straight_1x03" H 8650 3750 50  0001 C CNN
+F 3 "" H 8650 3750 50  0000 C CNN
+	1    8650 3750
 	1    0    0    -1
 $EndComp
@@
 L VCC #PWR04
 U 1 1 5836C698
-P 8350 3250
-F 0 "#PWR04" H 8350 3100 50  0001 C CNN
-F 1 "VCC" H 8350 3400 50  0000 C CNN
-F 2 "" H 8350 3250 50  0000 C CNN
-F 3 "" H 8350 3250 50  0000 C CNN
-	1    8350 3250
-	0    -1   -1   0
-$EndComp
-Wire Wire Line
-	8350 3250 8450 3250
+P 8350 3650
+F 0 "#PWR04" H 8350 3500 50  0001 C CNN
+F 1 "VCC" H 8350 3800 50  0000 C CNN
+F 2 "" H 8350 3650 50  0000 C CNN
+F 3 "" H 8350 3650 50  0000 C CNN
+	1    8350 3650
+	1    0    0    -1
+$EndComp
+Wire Wire Line
+	8350 3650 8450 3650
 $Comp
 L GND #PWR05
 U 1 1 5836C6DB
-P 8350 3450
-F 0 "#PWR05" H 8350 3200 50  0001 C CNN
-F 1 "GND" H 8350 3300 50  0000 C CNN
-F 2 "" H 8350 3450 50  0000 C CNN
-F 3 "" H 8350 3450 50  0000 C CNN
-	1    8350 3450
-	0    1    1    0
-$EndComp
-Wire Wire Line
-	8350 3450 8450 3450
+P 8350 3850
+F 0 "#PWR05" H 8350 3600 50  0001 C CNN
+F 1 "GND" H 8350 3700 50  0000 C CNN
+F 2 "" H 8350 3850 50  0000 C CNN
+F 3 "" H 8350 3850 50  0000 C CNN
+	1    8350 3850
+	1    0    0    -1
+$EndComp
+Wire Wire Line
+	8350 3850 8450 3850
 $Comp
 L CONN_01X03 P3
 U 1 1 5836C757
-P 8650 3850
-F 0 "P3" H 8650 4050 50  0000 C CNN
-F 1 "Address 1" V 8750 3850 50  0000 C CNN
-F 2 "Pin_Headers:Pin_Header_Straight_1x03" H 8650 3850 50  0001 C CNN
-F 3 "" H 8650 3850 50  0000 C CNN
-	1    8650 3850
+P 8650 4400
+F 0 "P3" H 8650 4600 50  0000 C CNN
+F 1 "Address 1" V 8750 4400 50  0000 C CNN
+F 2 "Pin_Headers:Pin_Header_Straight_1x03" H 8650 4400 50  0001 C CNN
+F 3 "" H 8650 4400 50  0000 C CNN
+	1    8650 4400
 	1    0    0    -1
 $EndComp
@@
 L VCC #PWR06
 U 1 1 5836C75D
-P 8350 3750
-F 0 "#PWR06" H 8350 3600 50  0001 C CNN
-F 1 "VCC" H 8350 3900 50  0000 C CNN
-F 2 "" H 8350 3750 50  0000 C CNN
-F 3 "" H 8350 3750 50  0000 C CNN
-	1    8350 3750
-	0    -1   -1   0
-$EndComp
-Wire Wire Line
-	8350 3750 8450 3750
+P 8350 4300
+F 0 "#PWR06" H 8350 4150 50  0001 C CNN
+F 1 "VCC" H 8350 4450 50  0000 C CNN
+F 2 "" H 8350 4300 50  0000 C CNN
+F 3 "" H 8350 4300 50  0000 C CNN
+	1    8350 4300
+	1    0    0    -1
+$EndComp
+Wire Wire Line
+	8350 4300 8450 4300
 $Comp
 L GND #PWR07
 U 1 1 5836C764
-P 8350 3950
-F 0 "#PWR07" H 8350 3700 50  0001 C CNN
-F 1 "GND" H 8350 3800 50  0000 C CNN
-F 2 "" H 8350 3950 50  0000 C CNN
-F 3 "" H 8350 3950 50  0000 C CNN
-	1    8350 3950
-	0    1    1    0
-$EndComp
-Wire Wire Line
-	8350 3950 8450 3950
+P 8350 4500
+F 0 "#PWR07" H 8350 4250 50  0001 C CNN
+F 1 "GND" H 8350 4350 50  0000 C CNN
+F 2 "" H 8350 4500 50  0000 C CNN
+F 3 "" H 8350 4500 50  0000 C CNN
+	1    8350 4500
+	1    0    0    -1
+$EndComp
+Wire Wire Line
+	8350 4500 8450 4500
 Wire Wire Line
 	6750 3150 7550 3150
 Wire Wire Line
-	7550 3150 7550 3350
-Wire Wire Line
-	7550 3350 8450 3350
+	7550 3150 7550 3750
+Wire Wire Line
+	7550 3750 8450 3750
 Wire Wire Line
 	6750 3250 7400 3250
 Wire Wire Line
-	7400 3250 7400 3850
-Wire Wire Line
-	7400 3850 8450 3850
+	7400 3250 7400 4400
+Wire Wire Line
+	7400 4400 8450 4400
 Wire Wire Line
 	7300 1900 7300 1800
 Connection ~ 7300 1800
-$Comp
-L GND #PWR08
-U 1 1 5836CAA1
-P 7000 2300
-F 0 "#PWR08" H 7000 2050 50  0001 C CNN
-F 1 "GND" H 7000 2150 50  0000 C CNN
-F 2 "" H 7000 2300 50  0000 C CNN
-F 3 "" H 7000 2300 50  0000 C CNN
-	1    7000 2300
-	0    1    1    0
-$EndComp
-Wire Wire Line
-	7000 2300 7300 2300
-Wire Wire Line
-	7300 2200 7300 2400
+Wire Wire Line
+	6950 2300 7300 2300
+Wire Wire Line
+	7300 2200 7300 2300
+Wire Wire Line
+	7300 2300 7300 2400
 Connection ~ 7300 2300
 $Comp
@@
 $EndComp
 Wire Wire Line
-	7200 3950 7200 3750
+	7200 3750 7200 3850
+Wire Wire Line
+	7200 3850 7200 3950
 Wire Wire Line
 	6750 3450 6900 3450
@@
 L CONN_01X02 P5
 U 1 1 5836CF91
-P 9900 1850
-F 0 "P5" H 9900 2000 50  0000 C CNN
-F 1 "Power Connector" V 10000 1850 50  0000 C CNN
-F 2 "Pin_Headers:Pin_Header_Straight_1x02" H 9900 1850 50  0001 C CNN
-F 3 "" H 9900 1850 50  0000 C CNN
-	1    9900 1850
+P 8650 1850
+F 0 "P5" H 8650 2000 50  0000 C CNN
+F 1 "Power Connector" V 8750 1850 50  0000 C CNN
+F 2 "Pin_Headers:Pin_Header_Straight_1x02" H 8650 1850 50  0001 C CNN
+F 3 "" H 8650 1850 50  0000 C CNN
+	1    8650 1850
 	1    0    0    1
 $EndComp
@@
 L GND #PWR010
 U 1 1 5836D001
-P 9350 1900
-F 0 "#PWR010" H 9350 1650 50  0001 C CNN
-F 1 "GND" H 9350 1750 50  0000 C CNN
-F 2 "" H 9350 1900 50  0000 C CNN
-F 3 "" H 9350 1900 50  0000 C CNN
-	1    9350 1900
-	0    1    1    0
-$EndComp
-Wire Wire Line
-	9350 1900 9700 1900
+P 8400 1900
+F 0 "#PWR010" H 8400 1650 50  0001 C CNN
+F 1 "GND" H 8400 1750 50  0000 C CNN
+F 2 "" H 8400 1900 50  0000 C CNN
+F 3 "" H 8400 1900 50  0000 C CNN
+	1    8400 1900
+	1    0    0    -1
+$EndComp
+Wire Wire Line
+	8400 1900 8450 1900
 $Comp
 L CP C2
@@
 Text Label 7450 3050 0    60   ~ 0
 SCL
-Text Label 7700 3350 0    60   ~ 0
+Text Label 6850 3150 0    60   ~ 0
 A0
-Text Label 7700 3850 0    60   ~ 0
+Text Label 6850 3250 0    60   ~ 0
 A1
 $Comp
@@
 P 5550 3200
 F 0 "P1" H 5550 3750 50  0000 C CNN
-F 1 "CONN_01X10" V 5650 3200 50  0000 C CNN
+F 1 "Analog input connector" V 5650 3200 50  0000 C CNN
 F 2 "Pin_Headers:Pin_Header_Straight_1x10" H 5550 3200 50  0001 C CNN
 F 3 "" H 5550 3200 50  0000 C CNN
@@
 L GND #PWR?
 U 1 1 5836DDF8
-P 6000 3650
-F 0 "#PWR?" H 6000 3400 50  0001 C CNN
-F 1 "GND" H 6000 3500 50  0000 C CNN
-F 2 "" H 6000 3650 50  0000 C CNN
-F 3 "" H 6000 3650 50  0000 C CNN
-	1    6000 3650
-	0    -1   -1   0
-$EndComp
-Wire Wire Line
-	6000 3650 5750 3650
+P 5900 3650
+F 0 "#PWR?" H 5900 3400 50  0001 C CNN
+F 1 "GND" H 5900 3500 50  0000 C CNN
+F 2 "" H 5900 3650 50  0000 C CNN
+F 3 "" H 5900 3650 50  0000 C CNN
+	1    5900 3650
+	1    0    0    -1
+$EndComp
+Wire Wire Line
+	5750 3650 5900 3650
 Wire Wire Line
 	5750 3550 5900 3550
@@
 	5900 3550 5900 3650
 Connection ~ 5900 3650
+$Comp
+L GND #PWR08
+U 1 1 5836CAA1
+P 6950 2300
+F 0 "#PWR08" H 6950 2050 50  0001 C CNN
+F 1 "GND" H 6950 2150 50  0000 C CNN
+F 2 "" H 6950 2300 50  0000 C CNN
+F 3 "" H 6950 2300 50  0000 C CNN
+	1    6950 2300
+	1    0    0    -1
+$EndComp
 $EndSCHEMATC

Commit message: test
Parts:
- P2: value Address 0 -> A0 Connector
- P3: value Address 1 -> A1 Connector
Connections:
- net REF: now reaches C1.2, U1.10 (REF)
- net V_IC: now reaches C3.1, U1.16 (VDD)
- net V_IC: now also R1.1; no longer R1.2
- net VCC renamed +3V3
- net +3V3: now also R1.2; no longer R1.1
Other:
- note added: "CRC Filter"
- note added: "Datasheet \nrecomendation of C1"
- note added: "I2C pullup"
- note added: "I2C slave address option"
- moved on the sheet: C1, C2, C3, P2, P3, P4, P5, R1, R2, R3
