File: ESC_Soldering/main.kicad_pcb (KiCad board)
At the start: 2 copper layers, 172 x 77 mm, 27 parts, among them P1 CONN_02X03, P2 CONN_01X03, P3 CONN_01X03, P4 CONN_01X02, P5 CONN_02X05, Q1 BC847CE6327HTSA1, Q2 BC847CE6327HTSA1, U1 PCA9698, U2 ADS7828, U3 AUIPS7111S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

Commit message: test
Connections:
- P5 pad 3: /PWM1 -> (no net)
- P5 pad 5: (no net) -> /PWM1
Changed lines of the file:
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@@
   )
   (setup
-    (last_trace_width 0.3)
+    (last_trace_width 0.25)
     (user_trace_width 0.3)
     (user_trace_width 0.4)
@@
     (pad 1 thru_hole rect (at 0 0) (size 1.7272 1.7272) (drill 1.016) (layers *.Cu *.Mask))
     (pad 2 thru_hole oval (at 2.54 0) (size 1.7272 1.7272) (drill 1.016) (layers *.Cu *.Mask))
-    (pad 3 thru_hole oval (at 0 2.54) (size 1.7272 1.7272) (drill 1.016) (layers *.Cu *.Mask)
+    (pad 3 thru_hole oval (at 0 2.54) (size 1.7272 1.7272) (drill 1.016) (layers *.Cu *.Mask))
+    (pad 4 thru_hole oval (at 2.54 2.54) (size 1.7272 1.7272) (drill 1.016) (layers *.Cu *.Mask))
+    (pad 5 thru_hole oval (at 0 5.08) (size 1.7272 1.7272) (drill 1.016) (layers *.Cu *.Mask)
       (net 25 /PWM1))
-    (pad 4 thru_hole oval (at 2.54 2.54) (size 1.7272 1.7272) (drill 1.016) (layers *.Cu *.Mask))
-    (pad 5 thru_hole oval (at 0 5.08) (size 1.7272 1.7272) (drill 1.016) (layers *.Cu *.Mask))
     (pad 6 thru_hole oval (at 2.54 5.08) (size 1.7272 1.7272) (drill 1.016) (layers *.Cu *.Mask))
     (pad 7 thru_hole oval (at 0 7.62) (size 1.7272 1.7272) (drill 1.016) (layers *.Cu *.Mask))

Commit message: test
Parts:
- added U7: Littlebee, KiCad-Dev:Littlebee, F.Cu at (224.0, 125.0)
- added U8: Littlebee, Littlebee, F.Cu at (224.0, 98.0)
- moved P4 12.1 mm to (189.0, 124.0), turned to 0 degrees
Connections:
- net /pwr_mod_1/Power_Out renamed /pwr_mod_1/Pwr_Out
- net /pwr_mod_2/Power_Out renamed /pwr_mod_2/Pwr_Out
- P5 pad 3: (no net) -> /PWM1
- P5 pad 5: /PWM1 -> (no net)
Routing:
- net /pwr_mod_1/Power_Enanle_B: track 0.00 -> 8.64 mm, vias 0 -> 2
- net GND: track 31.3 -> 36.1 mm
- net +3V3: track 0.00 -> 4.68 mm, vias 0 -> 2
- net /pwr_mod_2/Current_Feedback: track 0.00 -> 1.75 mm, vias 0 -> 1
- net /pwr_mod_1/Current_Feedback: track 0.00 -> 1.75 mm, vias 0 -> 1
Other:
- net class Default: via_dia 0.6 -> 1.6; via_drill 0.4 -> 1.2

Commit message: test
Parts:
- removed C1, C2: CP, SMD_Packages:SMD-1206_Pol
- removed C3: C, Capacitors_SMD:C_0805
- removed P1: CONN_02X03, Pin_Headers:Pin_Header_Straight_2x03
- removed P2, P3: CONN_01X03, Pin_Headers:Pin_Header_Straight_1x03
- removed P4: CONN_01X02, Pin_Headers:Pin_Header_Straight_1x02
- removed R1: R, Resistors_SMD:R_0603
- removed U1: PCA9698, Housings_SSOP:TSSOP-56_6.1x14mm_Pitch0.5mm
- removed U2: ADS7828, Housings_SSOP:TSSOP-16_4.4x5mm_Pitch0.65mm
- added P6: CONN_01X10, Pin_Headers:Pin_Header_Straight_1x10, B.Cu at (244.9, 160.0)
- added P7: CONN_01X10, Pin_Headers:Pin_Header_Straight_1x10, B.Cu at (189.8, 160.0)
- P5: value CONN_02X05 -> CONN_01X10; footprint Pin_Headers:Pin_Header_Straight_2x05 -> Pin_Headers:Pin_Header_Straight_1x10; moved to B.Cu
- U8: footprint Littlebee -> KiCad-Dev:Littlebee
- moved P5 111.4 mm to (217.5, 160.0), turned to 270 degrees
- moved R3 21.5 mm to (214.0, 133.5)
- moved R2 21.5 mm to (210.5, 133.5)
- moved U3 21.5 mm to (214.2, 142.5)
- moved U5 21.4 mm to (206.5, 134.0)
- moved D1 21.0 mm to (217.0, 136.0)
- moved Q1 21.0 mm to (214.0, 136.0)
- moved R4 21.0 mm to (221.0, 136.0)
- moved R5 21.0 mm to (219.0, 136.0)
- moved U7 21.0 mm to (225.0, 146.0)
- moved Q2 18.5 mm to (214.0, 106.5)
- moved D2 18.5 mm to (216.5, 106.5)
- moved R6 18.5 mm to (209.5, 103.5)
- moved R7 18.5 mm to (212.5, 103.5)
- moved R8 18.5 mm to (220.5, 106.5)
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Connections:
- net /pwr_mod_1/Pwr_Out renamed /pwr_mod_1/Power_Out
- net /pwr_mod_2/Pwr_Out renamed /pwr_mod_2/Power_Out
- P5 pad 1: (no net) -> /Enable_1
- P5 pad 2: (no net) -> /Enable_2
- P5 pad 3: /PWM1 -> (no net)
- R4 pad 2: /pwr_mod_1/Current_Feedback -> /CH1
- R8 pad 2: /pwr_mod_2/Current_Feedback -> /CH2
- U5 pad 1: /pwr_mod_1/Power_Enable_A -> /Enable_1
- U6 pad 1: /pwr_mod_2/Power_Enable_A -> /Enable_2
- U7 pad 4: /pwr_mod_1/Power_Enable_A -> /PWM1
- U8 pad 4: /pwr_mod_2/Power_Enable_A -> /PWM2
Routing:
- net GND: track 36.1 -> 0.01 mm
- net Net-(R4-Pad1): track 12.7 -> 0.00 mm
- net /pwr_mod_1/Power_Enanle_B: track 8.64 -> 0.00 mm, vias 2 -> 0
- net Net-(D1-Pad1): track 6.19 -> 0.00 mm
- net Net-(D2-Pad1): track 6.12 -> 0.00 mm
- net +3V3: track 4.68 -> 0.00 mm, vias 2 -> 0
- net Net-(Q2-Pad1): track 3.56 -> 0.03 mm
- net Net-(Q1-Pad1): track 3.52 -> 0.00 mm
- net Net-(R8-Pad1): track 12.9 -> 11.0 mm
- net /pwr_mod_2/Current_Feedback: track 1.75 -> 0.00 mm, vias 1 -> 0
- net /pwr_mod_1/Current_Feedback: track 1.75 -> 0.00 mm, vias 1 -> 0
- net Net-(R6-Pad2): track 1.30 -> 0.00 mm
- net Net-(R2-Pad2): track 1.30 -> 0.00 mm
- added copper zone on B.Cu, net (none)
- added copper zone on F.Cu, net (none)
Other:
- board size 172 x 77 mm -> 85 x 80 mm
- net class Default: via_dia 1.6 -> 1.3; via_drill 1.2 -> 1

Commit message: test
Parts:
- added C1: CP, SMD_Packages:SMD-1206_Pol, F.Cu at (156.3, 99.0)
- added C2: CP, SMD_Packages:SMD-1206_Pol, F.Cu at (158.5, 111.1)
- added C3: C, Capacitors_SMD:C_0805, F.Cu at (160.0, 101.0)
- added P1: CONN_02X03, Pin_Headers:Pin_Header_Straight_2x03, F.Cu at (249.0, 175.1)
- added P2: CONN_01X03, Pin_Headers:Pin_Header_Straight_1x03, F.Cu at (172.0, 102.5)
- added P3: CONN_01X03, Pin_Headers:Pin_Header_Straight_1x03, F.Cu at (170.0, 112.0)
- added P4: CONN_01X02, Pin_Headers:Pin_Header_Straight_1x02, F.Cu at (169.0, 97.0)
- added R1: R, Resistors_SMD:R_0603, F.Cu at (163.2, 105.0)
- added U1: PCA9698, Housings_SSOP:TSSOP-56_6.1x14mm_Pitch0.5mm, F.Cu at (193.0, 125.0)
- added U2: ADS7828, Housings_SSOP:TSSOP-16_4.4x5mm_Pitch0.65mm, F.Cu at (208.0, 124.0)
