File: ESC_Soldering/main.sch (KiCad schematic (older format))
At the start: 11 parts, among them P1 CONN_02X03, P2 CONN_01X03, P3 CONN_01X03, P4 CONN_01X02, P5 CONN_02X05, U1 PCA9698, U2 ADS7828

Commit message: test
Connections:
- net PWM1: now also P5.5 (P5); no longer P5.3 (P3)
- new net PW2: P5.3 (P3)
Changed lines of the file:
@@
 Text Label 9200 5450 2    60   ~ 0
 PWM3
-Text Label 9200 5250 2    60   ~ 0
+Text Label 9200 5350 2    60   ~ 0
 PWM1
 Wire Wire Line
@@
 Wire Wire Line
 	9250 5350 9200 5350
+Text Label 9200 5250 2    60   ~ 0
+PW2
 $EndSCHEMATC

Commit message: test
Connections:
- net PW2 is gone; now on net PWM1: P5.3 (P3)
- net PWM1: no longer P5.5 (P5)
- new net PWM2: P5.5 (P5)
Other:
- moved on the sheet: P5
Changed lines of the file:
@@
 L CONN_02X05 P5
 U 1 1 584FCE49
-P 9500 5350
-F 0 "P5" H 9500 5650 50  0000 C CNN
-F 1 "CONN_02X05" H 9500 5050 50  0000 C CNN
-F 2 "Pin_Headers:Pin_Header_Straight_2x05" H 9500 4150 50  0001 C CNN
-F 3 "" H 9500 4150 50  0000 C CNN
-	1    9500 5350
+P 9250 5350
+F 0 "P5" H 9250 5650 50  0000 C CNN
+F 1 "CONN_02X05" H 9250 5050 50  0000 C CNN
+F 2 "Pin_Headers:Pin_Header_Straight_2x05" H 9250 4150 50  0001 C CNN
+F 3 "" H 9250 4150 50  0000 C CNN
+	1    9250 5350
 	1    0    0    -1
 $EndComp
-Text Label 9800 5550 0    60   ~ 0
+Text Label 9850 5550 0    60   ~ 0
 PWM5
-Text Label 9800 5450 0    60   ~ 0
+Text Label 9850 5450 0    60   ~ 0
 PWM6
-Text Label 9800 5350 0    60   ~ 0
+Text Label 9850 5350 0    60   ~ 0
 PWM7
-Text Label 9800 5250 0    60   ~ 0
+Text Label 9850 5250 0    60   ~ 0
 PWM8
-Text Label 9200 5550 2    60   ~ 0
+Text Label 8800 5550 2    60   ~ 0
 PWM4
-Text Label 9200 5450 2    60   ~ 0
+Text Label 8800 5450 2    60   ~ 0
 PWM3
-Text Label 9200 5350 2    60   ~ 0
+Text Label 8800 5250 2    60   ~ 0
 PWM1
 Wire Wire Line
-	9800 5250 9750 5250
+	9850 5250 9500 5250
 Wire Wire Line
-	9750 5350 9800 5350
+	9500 5350 9850 5350
 Wire Wire Line
-	9800 5450 9750 5450
+	9850 5450 9500 5450
 Wire Wire Line
-	9750 5550 9800 5550
+	9500 5550 9850 5550
+Text Label 8800 5350 2    60   ~ 0
+PWM2
 Wire Wire Line
-	9250 5550 9200 5550
+	8800 5550 9000 5550
 Wire Wire Line
-	9200 5450 9250 5450
+	9000 5250 8800 5250
 Wire Wire Line
-	9200 5250 9250 5250
+	8800 5450 9000 5450
 Wire Wire Line
-	9250 5350 9200 5350
-Text Label 9200 5250 2    60   ~ 0
-PW2
+	8800 5350 9000 5350
 $EndSCHEMATC

Commit message: test
Parts:
- removed P5: CONN_02X05, Pin_Headers:Pin_Header_Straight_2x05, symbol CONN_02X05
- added P5, P6, P7: CONN_01X10, Pin_Headers:Pin_Header_Straight_1x10, symbol CONN_01X10
- added U7, U8: Littlebee, KiCad-Dev:Littlebee, symbol Littlebee
Connections:
- net GND: now also U7.2 (-), U7.3 (GND), U8.2 (-), U8.3 (GND)
- net PWM1: now also P6.1 (P1), U7.4 (In)
- net PWM2: now also P6.2 (P2), U8.4 (In)
- net PWM3: now also P6.3 (P3)
- net PWM4: now also P6.4 (P4)
- net PWM5: now also P6.5 (P5)
- net PWM6: now also P6.6 (P6)
- net PWM7: now also P6.7 (P7)
- net PWM8: now also P6.8 (P8)
- net pwr_mod_1/Power_Out: now also U7.1 (+)
- net pwr_mod_2/Power_Out: now also U8.1 (+)
- net CH3: now reaches U2.3 (CH2)
- net CH3: now also P7.3 (P3)
- net CH4: now reaches U2.4 (CH3)
- net CH4: now also P7.4 (P4)
- net CH5: now reaches U2.5 (CH4)
- net CH5: now also P7.5 (P5)
- net CH6: now reaches U2.6 (CH5)
- net CH6: now also P7.6 (P6)
- net CH7: now reaches U2.7 (CH6)
- net CH7: now also P7.7 (P7)
- net CH8: now reaches U2.8 (CH7)
- net CH8: now also P7.8 (P8)
- net pwr_mod_1/Current_Feedback renamed CH1
- net CH1: now also P7.1 (P1)
- net pwr_mod_1/Power_Enable_A renamed Enable_1
- net Enable_1: now also P5.1 (P1)
- net pwr_mod_2/Current_Feedback renamed CH2
- net CH2: now also P7.2 (P2)
- net pwr_mod_2/Power_Enable_A renamed Enable_2
- net Enable_2: now also P5.2 (P2)
- new net CH10: P7.10 (P10)
- new net CH9: P7.9 (P9)
- new net Enable_10: P5.10 (P10)
- new net Enable_3: P5.3 (P3)
- new net Enable_4: P5.4 (P4)
- new net Enable_5: P5.5 (P5)
- new net Enable_6: P5.6 (P6)
- new net Enable_7: P5.7 (P7)
- new net Enable_8: P5.8 (P8)
- new net Enable_9: P5.9 (P9)
- new net PWM10: P6.10 (P10)
- new net PWM9: P6.9 (P9)
Other:
- moved on the sheet: P4

Commit message: test
Parts:
- added U? (x4): LTC6802-2, symbol LTC6802-2
- added U?: SC18IS602B, symbol SC18IS602B
Changed lines of the file:
@@
 Text Label 10100 3350 2    60   ~ 0
 Enable_2
+$Comp
+L LTC6802-2 U?
+U 1 1 5854091D
+P 12200 5600
+F 0 "U?" H 12200 6750 60  0000 C CNN
+F 1 "LTC6802-2" H 12200 6850 60  0000 C CNN
+F 2 "" H 11850 5600 60  0000 C CNN
+F 3 "http://cds.linear.com/docs/en/datasheet/68022fa.pdf" H 12200 7200 60  0001 C CNN
+	1    12200 5600
+	1    0    0    -1
+$EndComp
+$Comp
+L SC18IS602B U?
+U 1 1 585409D8
+P 14550 6500
+F 0 "U?" H 14550 7050 60  0000 C CNN
+F 1 "SC18IS602B" H 14550 7150 60  0000 C CNN
+F 2 "" H 14550 6250 60  0001 C CNN
+F 3 "http://www.nxp.com/documents/data_sheet/SC18IS602B.pdf" H 14550 7250 60  0001 C CNN
+	1    14550 6500
+	1    0    0    -1
+$EndComp
+$Comp
+L LTC6802-2 U?
+U 1 1 58540B70
+P 12250 8450
+F 0 "U?" H 12250 9600 60  0000 C CNN
+F 1 "LTC6802-2" H 12250 9700 60  0000 C CNN
+F 2 "" H 11900 8450 60  0000 C CNN
+F 3 "http://cds.linear.com/docs/en/datasheet/68022fa.pdf" H 12250 10050 60  0001 C CNN
+	1    12250 8450
+	1    0    0    -1
+$EndComp
+$Comp
+L LTC6802-2 U?
+U 1 1 58540C42
+P 12300 11350
+F 0 "U?" H 12300 12500 60  0000 C CNN
+F 1 "LTC6802-2" H 12300 12600 60  0000 C CNN
+F 2 "" H 11950 11350 60  0000 C CNN
+F 3 "http://cds.linear.com/docs/en/datasheet/68022fa.pdf" H 12300 12950 60  0001 C CNN
+	1    12300 11350
+	1    0    0    -1
+$EndComp
+$Comp
+L LTC6802-2 U?
+U 1 1 58540D7D
+P 13900 12500
+F 0 "U?" H 13900 13650 60  0000 C CNN
+F 1 "LTC6802-2" H 13900 13750 60  0000 C CNN
+F 2 "" H 13550 12500 60  0000 C CNN
+F 3 "http://cds.linear.com/docs/en/datasheet/68022fa.pdf" H 13900 14100 60  0001 C CNN
+	1    13900 12500
+	1    0    0    -1
+$EndComp
 $EndSCHEMATC
