File: ESC_Soldering/pwr_mod.sch (KiCad schematic (older format))
At the start: 8 parts, among them Q1 BC847CE6327HTSA1, U3 AUIPS7111S, U5 74LVC1G08

Commit message: test
Parts:
- added U7: Littlebee, KiCad-Dev:Littlebee, symbol Littlebee
Connections:
- net GND: now also U7.2 (-), U7.3 (GND)
- net Power_Enable_A: now also U7.4 (In)
- net Power_Out renamed Pwr_Out
- net Pwr_Out: now also U7.1 (+)
Changed lines of the file:
@@
 AR Path="/584F1774/584EF2BD" Ref="U3"  Part="1"
 AR Path="/584F5DF6/584EF2BD" Ref="U4"  Part="1"
-F 0 "U3" H 6950 3100 60  0000 C CNN
+F 0 "U4" H 6950 3100 60  0000 C CNN
 F 1 "AUIPS7111S" H 6950 3200 60  0000 C CNN
 F 2 "TO_SOT_Packages_SMD:TO-263-5Lead" H 6950 2850 60  0001 C CNN
@@
 AR Path="/584F1774/584EF2C4" Ref="R3"  Part="1"
 AR Path="/584F5DF6/584EF2C4" Ref="R7"  Part="1"
-F 0 "R3" V 3680 3200 50  0000 C CNN
+F 0 "R7" V 3680 3200 50  0000 C CNN
 F 1 "R" V 3600 3200 50  0000 C CNN
 F 2 "Resistors_SMD:R_0603" V 3530 3200 50  0001 C CNN
@@
 AR Path="/584F1774/584EF2CB" Ref="R2"  Part="1"
 AR Path="/584F5DF6/584EF2CB" Ref="R6"  Part="1"
-F 0 "R2" V 3430 2950 50  0000 C CNN
+F 0 "R6" V 3430 2950 50  0000 C CNN
 F 1 "R" V 3350 2950 50  0000 C CNN
 F 2 "Resistors_SMD:R_0603" V 3280 2950 50  0001 C CNN
@@
 AR Path="/584F1774/584EF2D2" Ref="R5"  Part="1"
 AR Path="/584F5DF6/584EF2D2" Ref="R9"  Part="1"
-F 0 "R5" V 6530 3000 50  0000 C CNN
+F 0 "R9" V 6530 3000 50  0000 C CNN
 F 1 "R" V 6450 3000 50  0000 C CNN
 F 2 "Resistors_SMD:R_0603" V 6380 3000 50  0001 C CNN
@@
 AR Path="/584F1774/584EF2D9" Ref="Q1"  Part="1"
 AR Path="/584F5DF6/584EF2D9" Ref="Q2"  Part="1"
-F 0 "Q1" H 4100 3025 50  0000 L CNN
+F 0 "Q2" H 4100 3025 50  0000 L CNN
 F 1 "BC847CE6327HTSA1" H 4100 2950 50  0000 L CNN
 F 2 "TO_SOT_Packages_SMD:SOT-23" H 4100 2875 50  0000 L CIN
@@
 AR Path="/584F1774/584EF2E0" Ref="D1"  Part="1"
 AR Path="/584F5DF6/584EF2E0" Ref="D2"  Part="1"
-F 0 "D1" H 5000 3000 50  0000 C CNN
+F 0 "D2" H 5000 3000 50  0000 C CNN
 F 1 "D" H 5000 2800 50  0000 C CNN
 F 2 "Diodes_SMD:D_0603" H 5000 2900 50  0001 C CNN
@@
 AR Path="/584F1774/584EF2E7" Ref="R4"  Part="1"
 AR Path="/584F5DF6/584EF2E7" Ref="R8"  Part="1"
-F 0 "R4" V 6230 2800 50  0000 C CNN
+F 0 "R8" V 6230 2800 50  0000 C CNN
 F 1 "R" V 6150 2800 50  0000 C CNN
 F 2 "Resistors_SMD:R_0603" V 6080 2800 50  0001 C CNN
@@
 	0    1    1    0
 $EndComp
-Wire Wire Line
-	4000 2750 4000 2700
-Wire Wire Line
-	4000 2700 6550 2700
-Wire Wire Line
-	5000 2700 5000 2750
-Wire Wire Line
-	5000 3450 5000 3050
-Wire Wire Line
-	2650 3450 6450 3450
-Wire Wire Line
-	4000 3450 4000 3150
-Connection ~ 5000 2700
-Wire Wire Line
-	6300 2800 6550 2800
-Wire Wire Line
-	6450 2850 6450 2800
-Connection ~ 6450 2800
-Wire Wire Line
-	3600 3050 3600 2950
-Wire Wire Line
-	3500 2950 3700 2950
-Connection ~ 3600 2950
-Wire Wire Line
-	3600 3350 3600 3450
-Connection ~ 4000 3450
-Wire Wire Line
-	6450 3450 6450 3150
-Connection ~ 5000 3450
 $Comp
 L +BATT #PWR012
@@
 P 7500 2700
 AR Path="/584F1774/584EF301" Ref="#PWR012"  Part="1"
-AR Path="/584F5DF6/584EF301" Ref="#PWR015"  Part="1"
-F 0 "#PWR015" H 7500 2550 50  0001 C CNN
+AR Path="/584F5DF6/584EF301" Ref="#PWR017"  Part="1"
+F 0 "#PWR017" H 7500 2550 50  0001 C CNN
 F 1 "+BATT" H 7500 2840 50  0000 C CNN
 F 2 "" H 7500 2700 50  0000 C CNN
@@
 	0    1    1    0
 $EndComp
-Wire Wire Line
-	7500 2700 7300 2700
-Wire Wire Line
-	7300 2800 7400 2800
-Wire Wire Line
-	7400 2800 7400 2900
-Wire Wire Line
-	7300 2900 8200 2900
-Connection ~ 7400 2900
-Text HLabel 8200 2900 2    60   Output ~ 0
-Power_Out
 Text HLabel 5500 3350 2    60   Output ~ 0
 Current_Feedback
-Wire Wire Line
-	6000 2800 5300 2800
-Wire Wire Line
-	5300 2800 5300 3350
-Wire Wire Line
-	5300 3350 5500 3350
 $Comp
 L GND #PWR013
@@
 P 2800 3550
 AR Path="/584F1774/584EF611" Ref="#PWR013"  Part="1"
-AR Path="/584F5DF6/584EF611" Ref="#PWR016"  Part="1"
-F 0 "#PWR016" H 2800 3300 50  0001 C CNN
+AR Path="/584F5DF6/584EF611" Ref="#PWR018"  Part="1"
+F 0 "#PWR018" H 2800 3300 50  0001 C CNN
 F 1 "GND" H 2800 3400 50  0000 C CNN
 F 2 "" H 2800 3550 50  0000 C CNN
@@
 	1    0    0    -1
 $EndComp
-Wire Wire Line
-	2800 3450 2800 3550
-Connection ~ 3600 3450
 Text HLabel 2000 2900 0    60   Input ~ 0
 Power_Enable_A
-Wire Wire Line
-	2000 2900 2300 2900
 $Comp
 L 74LVC1G08 U5
@@
 AR Path="/584F1774/584F6D45" Ref="U5"  Part="1"
 AR Path="/584F5DF6/584F6D45" Ref="U6"  Part="1"
-F 0 "U5" H 2750 2700 60  0000 C CNN
+F 0 "U6" H 2750 2700 60  0000 C CNN
 F 1 "74LVC1G08" H 2950 3200 60  0000 C CNN
 F 2 "TO_SOT_Packages_SMD:SOT-353" H 2600 3000 60  0001 C CNN
@@
 	1    0    0    -1
 $EndComp
-Wire Wire Line
-	3100 2950 3200 2950
-Wire Wire Line
-	2650 3350 2650 3450
-Connection ~ 2800 3450
 $Comp
 L +3.3V #PWR014
@@
 P 2650 2400
 AR Path="/584F1774/584F6E96" Ref="#PWR014"  Part="1"
-AR Path="/584F5DF6/584F6E96" Ref="#PWR017"  Part="1"
-F 0 "#PWR017" H 2650 2250 50  0001 C CNN
+AR Path="/584F5DF6/584F6E96" Ref="#PWR019"  Part="1"
+F 0 "#PWR019" H 2650 2250 50  0001 C CNN
 F 1 "+3.3V" H 2650 2540 50  0000 C CNN
 F 2 "" H 2650 2400 50  0000 C CNN
@@
 	1    0    0    -1
 $EndComp
-Wire Wire Line
-	2650 2400 2650 2550
 Text HLabel 2000 3000 0    60   Input ~ 0
 Power_Enanle_B
+$Comp
+L Littlebee U7
+U 1 1 5850A47D
+P 7450 4100
+AR Path="/584F1774/5850A47D" Ref="U7"  Part="1"
+AR Path="/584F5DF6/5850A47D" Ref="U8"  Part="1"
+F 0 "U8" H 7450 4250 60  0000 C CNN
+F 1 "Littlebee" H 7450 4350 60  0000 C CNN
+F 2 "KiCad-Dev:Littlebee" H 7700 4100 60  0001 C CNN
+F 3 "" H 7700 4100 60  0001 C CNN
+	1    7450 4100
+	1    0    0    -1
+$EndComp
+Text HLabel 7000 4050 0    60   Input ~ 0
+Power_Enable_A
+Wire Wire Line
+	4000 2750 4000 2700
+Wire Wire Line
+	4000 2700 6550 2700
+Wire Wire Line
+	5000 2700 5000 2750
+Wire Wire Line
+	5000 3450 5000 3050
+Wire Wire Line
+	2650 3450 6450 3450
+Wire Wire Line
+	4000 3450 4000 3150
+Connection ~ 5000 2700
+Wire Wire Line
+	6300 2800 6550 2800
+Wire Wire Line
+	6450 2850 6450 2800
+Connection ~ 6450 2800
+Wire Wire Line
+	3600 3050 3600 2950
+Wire Wire Line
+	3500 2950 3700 2950
+Connection ~ 3600 2950
+Wire Wire Line
+	3600 3350 3600 3450
+Connection ~ 4000 3450
+Wire Wire Line
+	6450 3450 6450 3150
+Connection ~ 5000 3450
+Wire Wire Line
+	7500 2700 7300 2700
+Wire Wire Line
+	7300 2800 7400 2800
+Wire Wire Line
+	7400 2800 7400 2900
+Connection ~ 7400 2900
+Wire Wire Line
+	6000 2800 5300 2800
+Wire Wire Line
+	5300 2800 5300 3350
+Wire Wire Line
+	5300 3350 5500 3350
+Wire Wire Line
+	2800 3450 2800 3550
+Connection ~ 3600 3450
+Wire Wire Line
+	2000 2900 2300 2900
+Wire Wire Line
+	3100 2950 3200 2950
+Wire Wire Line
+	2650 3350 2650 3450
+Connection ~ 2800 3450
+Wire Wire Line
+	2650 2400 2650 2550
 Wire Wire Line
 	2000 3000 2300 3000
+Wire Wire Line
+	7900 4050 8050 4050
+Wire Wire Line
+	8050 4050 8050 2900
+Wire Wire Line
+	8050 2900 7300 2900
+$Comp
+L GND #PWR015
+U 1 1 5850AA38
+P 6850 4300
+AR Path="/584F1774/5850AA38" Ref="#PWR015"  Part="1"
+AR Path="/584F5DF6/5850AA38" Ref="#PWR020"  Part="1"
+F 0 "#PWR020" H 6850 4050 50  0001 C CNN
+F 1 "GND" H 6850 4150 50  0000 C CNN
+F 2 "" H 6850 4300 50  0000 C CNN
+F 3 "" H 6850 4300 50  0000 C CNN
+	1    6850 4300
+	1    0    0    -1
+$EndComp
+Wire Wire Line
+	6850 4300 6850 4150
+Wire Wire Line
+	6850 4150 7000 4150
+$Comp
+L GND #PWR016
+U 1 1 5850AB63
+P 8050 4300
+AR Path="/584F1774/5850AB63" Ref="#PWR016"  Part="1"
+AR Path="/584F5DF6/5850AB63" Ref="#PWR021"  Part="1"
+F 0 "#PWR021" H 8050 4050 50  0001 C CNN
+F 1 "GND" H 8050 4150 50  0000 C CNN
+F 2 "" H 8050 4300 50  0000 C CNN
+F 3 "" H 8050 4300 50  0000 C CNN
+	1    8050 4300
+	1    0    0    -1
+$EndComp
+Wire Wire Line
+	8050 4300 8050 4150
+Wire Wire Line
+	8050 4150 7900 4150
+Text Label 7650 2900 0    60   ~ 0
+Pwr_Out
 $EndSCHEMATC

Commit message: test
Parts:
- removed U7: Littlebee, KiCad-Dev:Littlebee, symbol Littlebee
Connections:
- net Pwr_Out renamed Power_Out
Changed lines of the file:
@@
 AR Path="/584F1774/584EF2BD" Ref="U3"  Part="1"
 AR Path="/584F5DF6/584EF2BD" Ref="U4"  Part="1"
-F 0 "U4" H 6950 3100 60  0000 C CNN
+F 0 "U3" H 6950 3100 60  0000 C CNN
 F 1 "AUIPS7111S" H 6950 3200 60  0000 C CNN
 F 2 "TO_SOT_Packages_SMD:TO-263-5Lead" H 6950 2850 60  0001 C CNN
@@
 AR Path="/584F1774/584EF2C4" Ref="R3"  Part="1"
 AR Path="/584F5DF6/584EF2C4" Ref="R7"  Part="1"
-F 0 "R7" V 3680 3200 50  0000 C CNN
+F 0 "R3" V 3680 3200 50  0000 C CNN
 F 1 "R" V 3600 3200 50  0000 C CNN
 F 2 "Resistors_SMD:R_0603" V 3530 3200 50  0001 C CNN
@@
 AR Path="/584F1774/584EF2CB" Ref="R2"  Part="1"
 AR Path="/584F5DF6/584EF2CB" Ref="R6"  Part="1"
-F 0 "R6" V 3430 2950 50  0000 C CNN
+F 0 "R2" V 3430 2950 50  0000 C CNN
 F 1 "R" V 3350 2950 50  0000 C CNN
 F 2 "Resistors_SMD:R_0603" V 3280 2950 50  0001 C CNN
@@
 AR Path="/584F1774/584EF2D2" Ref="R5"  Part="1"
 AR Path="/584F5DF6/584EF2D2" Ref="R9"  Part="1"
-F 0 "R9" V 6530 3000 50  0000 C CNN
+F 0 "R5" V 6530 3000 50  0000 C CNN
 F 1 "R" V 6450 3000 50  0000 C CNN
 F 2 "Resistors_SMD:R_0603" V 6380 3000 50  0001 C CNN
@@
 AR Path="/584F1774/584EF2D9" Ref="Q1"  Part="1"
 AR Path="/584F5DF6/584EF2D9" Ref="Q2"  Part="1"
-F 0 "Q2" H 4100 3025 50  0000 L CNN
+F 0 "Q1" H 4100 3025 50  0000 L CNN
 F 1 "BC847CE6327HTSA1" H 4100 2950 50  0000 L CNN
 F 2 "TO_SOT_Packages_SMD:SOT-23" H 4100 2875 50  0000 L CIN
@@
 AR Path="/584F1774/584EF2E0" Ref="D1"  Part="1"
 AR Path="/584F5DF6/584EF2E0" Ref="D2"  Part="1"
-F 0 "D2" H 5000 3000 50  0000 C CNN
+F 0 "D1" H 5000 3000 50  0000 C CNN
 F 1 "D" H 5000 2800 50  0000 C CNN
 F 2 "Diodes_SMD:D_0603" H 5000 2900 50  0001 C CNN
@@
 AR Path="/584F1774/584EF2E7" Ref="R4"  Part="1"
 AR Path="/584F5DF6/584EF2E7" Ref="R8"  Part="1"
-F 0 "R8" V 6230 2800 50  0000 C CNN
+F 0 "R4" V 6230 2800 50  0000 C CNN
 F 1 "R" V 6150 2800 50  0000 C CNN
 F 2 "Resistors_SMD:R_0603" V 6080 2800 50  0001 C CNN
@@
 $EndComp
 $Comp
-L +BATT #PWR012
+L +BATT #PWR016
 U 1 1 584EF301
 P 7500 2700
-AR Path="/584F1774/584EF301" Ref="#PWR012"  Part="1"
-AR Path="/584F5DF6/584EF301" Ref="#PWR017"  Part="1"
-F 0 "#PWR017" H 7500 2550 50  0001 C CNN
+AR Path="/584F1774/584EF301" Ref="#PWR016"  Part="1"
+AR Path="/584F5DF6/584EF301" Ref="#PWR019"  Part="1"
+F 0 "#PWR019" H 7500 2550 50  0001 C CNN
 F 1 "+BATT" H 7500 2840 50  0000 C CNN
 F 2 "" H 7500 2700 50  0000 C CNN
@@
 Current_Feedback
 $Comp
-L GND #PWR013
+L GND #PWR017
 U 1 1 584EF611
 P 2800 3550
-AR Path="/584F1774/584EF611" Ref="#PWR013"  Part="1"
-AR Path="/584F5DF6/584EF611" Ref="#PWR018"  Part="1"
-F 0 "#PWR018" H 2800 3300 50  0001 C CNN
+AR Path="/584F1774/584EF611" Ref="#PWR017"  Part="1"
+AR Path="/584F5DF6/584EF611" Ref="#PWR020"  Part="1"
+F 0 "#PWR020" H 2800 3300 50  0001 C CNN
 F 1 "GND" H 2800 3400 50  0000 C CNN
 F 2 "" H 2800 3550 50  0000 C CNN
@@
 AR Path="/584F1774/584F6D45" Ref="U5"  Part="1"
 AR Path="/584F5DF6/584F6D45" Ref="U6"  Part="1"
-F 0 "U6" H 2750 2700 60  0000 C CNN
+F 0 "U5" H 2750 2700 60  0000 C CNN
 F 1 "74LVC1G08" H 2950 3200 60  0000 C CNN
 F 2 "TO_SOT_Packages_SMD:SOT-353" H 2600 3000 60  0001 C CNN
@@
 $EndComp
 $Comp
-L +3.3V #PWR014
+L +3.3V #PWR018
 U 1 1 584F6E96
 P 2650 2400
-AR Path="/584F1774/584F6E96" Ref="#PWR014"  Part="1"
-AR Path="/584F5DF6/584F6E96" Ref="#PWR019"  Part="1"
-F 0 "#PWR019" H 2650 2250 50  0001 C CNN
+AR Path="/584F1774/584F6E96" Ref="#PWR018"  Part="1"
+AR Path="/584F5DF6/584F6E96" Ref="#PWR021"  Part="1"
+F 0 "#PWR021" H 2650 2250 50  0001 C CNN
 F 1 "+3.3V" H 2650 2540 50  0000 C CNN
 F 2 "" H 2650 2400 50  0000 C CNN
@@
 Text HLabel 2000 3000 0    60   Input ~ 0
 Power_Enanle_B
-$Comp
-L Littlebee U7
-U 1 1 5850A47D
-P 7450 4100
-AR Path="/584F1774/5850A47D" Ref="U7"  Part="1"
-AR Path="/584F5DF6/5850A47D" Ref="U8"  Part="1"
-F 0 "U8" H 7450 4250 60  0000 C CNN
-F 1 "Littlebee" H 7450 4350 60  0000 C CNN
-F 2 "KiCad-Dev:Littlebee" H 7700 4100 60  0001 C CNN
-F 3 "" H 7700 4100 60  0001 C CNN
-	1    7450 4100
-	1    0    0    -1
-$EndComp
-Text HLabel 7000 4050 0    60   Input ~ 0
-Power_Enable_A
 Wire Wire Line
 	4000 2750 4000 2700
@@
 	2000 3000 2300 3000
 Wire Wire Line
-	7900 4050 8050 4050
-Wire Wire Line
-	8050 4050 8050 2900
-Wire Wire Line
 	8050 2900 7300 2900
-$Comp
-L GND #PWR015
-U 1 1 5850AA38
-P 6850 4300
-AR Path="/584F1774/5850AA38" Ref="#PWR015"  Part="1"
-AR Path="/584F5DF6/5850AA38" Ref="#PWR020"  Part="1"
-F 0 "#PWR020" H 6850 4050 50  0001 C CNN
-F 1 "GND" H 6850 4150 50  0000 C CNN
-F 2 "" H 6850 4300 50  0000 C CNN
-F 3 "" H 6850 4300 50  0000 C CNN
-	1    6850 4300
-	1    0    0    -1
-$EndComp
-Wire Wire Line
-	6850 4300 6850 4150
-Wire Wire Line
-	6850 4150 7000 4150
-$Comp
-L GND #PWR016
-U 1 1 5850AB63
-P 8050 4300
-AR Path="/584F1774/5850AB63" Ref="#PWR016"  Part="1"
-AR Path="/584F5DF6/5850AB63" Ref="#PWR021"  Part="1"
-F 0 "#PWR021" H 8050 4050 50  0001 C CNN
-F 1 "GND" H 8050 4150 50  0000 C CNN
-F 2 "" H 8050 4300 50  0000 C CNN
-F 3 "" H 8050 4300 50  0000 C CNN
-	1    8050 4300
-	1    0    0    -1
-$EndComp
-Wire Wire Line
-	8050 4300 8050 4150
-Wire Wire Line
-	8050 4150 7900 4150
-Text Label 7650 2900 0    60   ~ 0
-Pwr_Out
+Text HLabel 8050 2900 2    60   Input ~ 0
+Power_Out
 $EndSCHEMATC
