File: PDB6_BMS/main.kicad_pcb (KiCad board)
At the start: 2 copper layers, 19 parts, among them P1 CONN_01X13, P2 CONN_01X04, P3 CONN_01X03, P4 CONN_01X03, U1 LTC6802-2

Commit message: test
Parts:
- added P5: CONN_01X20, Pin_Headers:Pin_Header_Straight_1x20_Pitch2.00mm, F.Cu at (168.0, 69.0)
- P2: value CONN_01X04 -> CONN_01X20; footprint Pin_Headers:Pin_Header_Straight_1x04 -> Pin_Headers:Pin_Header_Straight_1x20_Pitch2.00mm
- moved C1 10.6 mm to (193.0, 106.2)
- moved P2 10.5 mm to (204.0, 69.0)
- moved P3 8.19 mm to (213.9, 89.9)
- moved C2 3.25 mm to (192.5, 109.2), turned to 180 degrees
- moved U1 2.88 mm to (195.6, 86.4)
- moved P1 0.20 mm to (178.0, 104.1)
- turned R11 to 180 degrees
- turned R5 to 180 degrees
Routing:
- net Net-(P1-Pad2): track 0.00 -> 29.3 mm
- net Net-(R12-Pad1): track 0.00 -> 25.0 mm
- net Net-(P1-Pad13): track 0.00 -> 21.2 mm
- net Net-(P1-Pad12): track 0.00 -> 18.9 mm
- net Net-(R11-Pad1): track 0.00 -> 18.6 mm
- net Net-(P1-Pad3): track 0.00 -> 17.4 mm
- net Net-(P1-Pad11): track 0.00 -> 17.1 mm
- net Net-(P1-Pad4): track 0.00 -> 16.8 mm
- net Net-(P1-Pad10): track 0.00 -> 16.5 mm
- net Net-(P1-Pad5): track 0.00 -> 16.1 mm
- net Net-(P1-Pad9): track 0.00 -> 15.8 mm
- net Net-(P1-Pad6): track 0.00 -> 15.5 mm
- net Net-(P1-Pad8): track 0.00 -> 15.2 mm
- net Net-(P1-Pad7): track 0.00 -> 14.8 mm
- net Net-(R1-Pad1): track 0.00 -> 13.5 mm
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