File: PDB6_BMS/main.sch (KiCad schematic (older format))
At the start: 19 parts, among them P1 CONN_01X13, P2 CONN_01X04, P3 CONN_01X03, P4 CONN_01X03, U1 LTC6802-2

Commit message: test
Connections:
- net at U1.41 (SCKI): no longer P2.4 (P4)
- net at U1.42 (SDI): no longer P2.3 (P3)
- net at U1.43 (SDO): no longer P2.2 (P2)
- net at U1.44 (CSBI): no longer P2.1 (P1)
Other:
- moved on the sheet: P2
Changed lines of the file:
@@
 	17900 6700 17400 6700
 Wire Wire Line
-	17400 6600 17400 6800
-Wire Wire Line
-	17100 6800 17500 6800
+	17400 6600 17400 6700
+Wire Wire Line
+	17400 6700 17400 6800
+Wire Wire Line
+	17100 6800 17400 6800
+Wire Wire Line
+	17400 6800 17500 6800
 Wire Wire Line
 	17900 6900 17400 6900
@@
 	17400 6900 17400 7000
 Wire Wire Line
-	17200 7000 17500 7000
+	17200 7000 17400 7000
+Wire Wire Line
+	17400 7000 17500 7000
 Wire Wire Line
 	17900 7100 17400 7100
@@
 	17400 7100 17400 7200
 Wire Wire Line
-	17300 7200 17500 7200
+	17300 7200 17400 7200
+Wire Wire Line
+	17400 7200 17500 7200
 Wire Wire Line
 	17900 7300 17400 7300
@@
 	17400 7300 17400 7400
 Wire Wire Line
-	16350 7400 17500 7400
-Wire Wire Line
-	16350 7500 17900 7500
+	16350 7400 17400 7400
+Wire Wire Line
+	17400 7400 17500 7400
+Wire Wire Line
+	16350 7500 17400 7500
+Wire Wire Line
+	17400 7500 17900 7500
 Wire Wire Line
 	17400 7500 17400 7600
@@
 	17400 7600 17500 7600
 Wire Wire Line
-	17300 7700 17900 7700
+	17300 7700 17400 7700
+Wire Wire Line
+	17400 7700 17900 7700
 Wire Wire Line
 	17400 7700 17400 7800
@@
 	17400 7800 17500 7800
 Wire Wire Line
-	17200 7900 17900 7900
+	17200 7900 17400 7900
+Wire Wire Line
+	17400 7900 17900 7900
 Wire Wire Line
 	17400 7900 17400 8000
@@
 	17400 8000 17500 8000
 Wire Wire Line
-	17100 8100 17900 8100
+	17100 8100 17400 8100
+Wire Wire Line
+	17400 8100 17900 8100
 Wire Wire Line
 	17400 8100 17400 8200
@@
 	17400 8200 17500 8200
 Wire Wire Line
-	17000 8300 17900 8300
+	17000 8300 17400 8300
+Wire Wire Line
+	17400 8300 17900 8300
 Wire Wire Line
 	17400 8300 17400 8400
@@
 	17400 8400 17500 8400
 Wire Wire Line
-	16900 8500 17900 8500
+	16900 8500 17400 8500
+Wire Wire Line
+	17400 8500 17900 8500
 Wire Wire Line
 	17400 8500 17400 8600
@@
 	17400 8600 17500 8600
 Wire Wire Line
-	16800 8700 17900 8700
+	16800 8700 17400 8700
+Wire Wire Line
+	17400 8700 17900 8700
 Wire Wire Line
 	17400 8700 17400 8800
@@
 	17400 8800 17500 8800
 Wire Wire Line
-	16700 8900 17900 8900
+	16700 8900 17400 8900
+Wire Wire Line
+	17400 8900 17900 8900
 Wire Wire Line
 	17400 8900 17400 9000
@@
 	17900 9100 17800 9100
 Wire Wire Line
-	17800 9100 17800 9950
-Wire Wire Line
-	19650 6600 19650 9350
+	17800 9100 17800 9700
+Wire Wire Line
+	17800 9700 17800 9950
+Wire Wire Line
+	19650 6600 19650 8450
+Wire Wire Line
+	19650 8450 19650 9350
 Wire Wire Line
 	19100 6600 19650 6600
@@
 	19400 7850 19100 7850
 Wire Wire Line
-	19400 9700 19400 7550
+	19400 9700 19400 8550
+Wire Wire Line
+	19400 8550 19400 7850
+Wire Wire Line
+	19400 7850 19400 7750
+Wire Wire Line
+	19400 7750 19400 7650
+Wire Wire Line
+	19400 7650 19400 7550
 Wire Wire Line
 	19400 7550 19100 7550
@@
 Connection ~ 19400 7850
 Wire Wire Line
-	16400 9700 19650 9700
+	16400 9700 17800 9700
+Wire Wire Line
+	17800 9700 19200 9700
+Wire Wire Line
+	19200 9700 19400 9700
+Wire Wire Line
+	19400 9700 19650 9700
 Connection ~ 19400 8550
 Connection ~ 17800 9700
@@
 L CONN_01X04 P2
 U 1 1 5857469C
-P 19300 7200
-F 0 "P2" H 19300 7450 50  0000 C CNN
-F 1 "CONN_01X04" V 19400 7200 50  0000 C CNN
-F 2 "Pin_Headers:Pin_Header_Straight_1x04" H 19300 7200 50  0001 C CNN
-F 3 "" H 19300 7200 50  0000 C CNN
-	1    19300 7200
+P 20050 7200
+F 0 "P2" H 20050 7450 50  0000 C CNN
+F 1 "CONN_01X04" V 20150 7200 50  0000 C CNN
+F 2 "Pin_Headers:Pin_Header_Straight_1x04" H 20050 7200 50  0001 C CNN
+F 3 "" H 20050 7200 50  0000 C CNN
+	1    20050 7200
 	1    0    0    -1
 $EndComp

Commit message: test
Parts:
- removed P2: CONN_01X04, Pin_Headers:Pin_Header_Straight_1x04, symbol CONN_01X04
- added P2, P5: CONN_01X20, Pin_Headers:Pin_Header_Straight_1x20_Pitch2.00mm, symbol CONN_01X20
Connections:
- net at U1.41 (SCKI): now also P2.4 (P4)
- net at U1.42 (SDI): now also P2.3 (P3)
- net at U1.43 (SDO): now also P2.2 (P2)
- net at U1.44 (CSBI): now also P2.1 (P1)
Other:
- moved on the sheet: P3, P4
Changed lines of the file:
@@
 L CONN_01X03 P4
 U 1 1 58573072
-P 20950 9050
-F 0 "P4" H 20950 9250 50  0000 C CNN
-F 1 "CONN_01X03" V 21050 9050 50  0000 C CNN
-F 2 "Pin_Headers:Pin_Header_Straight_1x03" H 20950 9050 50  0001 C CNN
-F 3 "" H 20950 9050 50  0000 C CNN
-	1    20950 9050
+P 20650 9700
+F 0 "P4" H 20650 9900 50  0000 C CNN
+F 1 "CONN_01X03" V 20750 9700 50  0000 C CNN
+F 2 "Pin_Headers:Pin_Header_Straight_1x03" H 20650 9700 50  0001 C CNN
+F 3 "" H 20650 9700 50  0000 C CNN
+	1    20650 9700
 	1    0    0    1
 $EndComp
@@
 L CONN_01X03 P3
 U 1 1 58573CF0
-P 20950 8500
-F 0 "P3" H 20950 8700 50  0000 C CNN
-F 1 "CONN_01X03" V 21050 8500 50  0000 C CNN
-F 2 "Pin_Headers:Pin_Header_Straight_1x03" H 20950 8500 50  0001 C CNN
-F 3 "" H 20950 8500 50  0000 C CNN
-	1    20950 8500
+P 20650 9150
+F 0 "P3" H 20650 9350 50  0000 C CNN
+F 1 "CONN_01X03" V 20750 9150 50  0000 C CNN
+F 2 "Pin_Headers:Pin_Header_Straight_1x03" H 20650 9150 50  0001 C CNN
+F 3 "" H 20650 9150 50  0000 C CNN
+	1    20650 9150
 	1    0    0    1
 $EndComp
@@
 L GND #PWR02
 U 1 1 58573D72
-P 20700 9200
-F 0 "#PWR02" H 20700 8950 50  0001 C CNN
-F 1 "GND" H 20700 9050 50  0000 C CNN
-F 2 "" H 20700 9200 50  0000 C CNN
-F 3 "" H 20700 9200 50  0000 C CNN
-	1    20700 9200
+P 20400 9850
+F 0 "#PWR02" H 20400 9600 50  0001 C CNN
+F 1 "GND" H 20400 9700 50  0000 C CNN
+F 2 "" H 20400 9850 50  0000 C CNN
+F 3 "" H 20400 9850 50  0000 C CNN
+	1    20400 9850
 	1    0    0    -1
 $EndComp
@@
 L GND #PWR03
 U 1 1 58573E4A
-P 20700 8650
-F 0 "#PWR03" H 20700 8400 50  0001 C CNN
-F 1 "GND" H 20700 8500 50  0000 C CNN
-F 2 "" H 20700 8650 50  0000 C CNN
-F 3 "" H 20700 8650 50  0000 C CNN
-	1    20700 8650
+P 20400 9300
+F 0 "#PWR03" H 20400 9050 50  0001 C CNN
+F 1 "GND" H 20400 9150 50  0000 C CNN
+F 2 "" H 20400 9300 50  0000 C CNN
+F 3 "" H 20400 9300 50  0000 C CNN
+	1    20400 9300
 	1    0    0    -1
 $EndComp
@@
 	17900 6700 17400 6700
 Wire Wire Line
-	17400 6600 17400 6700
-Wire Wire Line
-	17400 6700 17400 6800
-Wire Wire Line
-	17100 6800 17400 6800
-Wire Wire Line
-	17400 6800 17500 6800
+	17400 6600 17400 6800
+Wire Wire Line
+	17100 6800 17500 6800
 Wire Wire Line
 	17900 6900 17400 6900
@@
 	17400 6900 17400 7000
 Wire Wire Line
-	17200 7000 17400 7000
-Wire Wire Line
-	17400 7000 17500 7000
+	17200 7000 17500 7000
 Wire Wire Line
 	17900 7100 17400 7100
@@
 	17400 7100 17400 7200
 Wire Wire Line
-	17300 7200 17400 7200
-Wire Wire Line
-	17400 7200 17500 7200
+	17300 7200 17500 7200
 Wire Wire Line
 	17900 7300 17400 7300
@@
 	17400 7300 17400 7400
 Wire Wire Line
-	16350 7400 17400 7400
-Wire Wire Line
-	17400 7400 17500 7400
-Wire Wire Line
-	16350 7500 17400 7500
-Wire Wire Line
-	17400 7500 17900 7500
+	16350 7400 17500 7400
+Wire Wire Line
+	16350 7500 17900 7500
 Wire Wire Line
 	17400 7500 17400 7600
@@
 	17400 7600 17500 7600
 Wire Wire Line
-	17300 7700 17400 7700
-Wire Wire Line
-	17400 7700 17900 7700
+	17300 7700 17900 7700
 Wire Wire Line
 	17400 7700 17400 7800
@@
 	17400 7800 17500 7800
 Wire Wire Line
-	17200 7900 17400 7900
-Wire Wire Line
-	17400 7900 17900 7900
+	17200 7900 17900 7900
 Wire Wire Line
 	17400 7900 17400 8000
@@
 	17400 8000 17500 8000
 Wire Wire Line
-	17100 8100 17400 8100
-Wire Wire Line
-	17400 8100 17900 8100
+	17100 8100 17900 8100
 Wire Wire Line
 	17400 8100 17400 8200
@@
 	17400 8200 17500 8200
 Wire Wire Line
-	17000 8300 17400 8300
-Wire Wire Line
-	17400 8300 17900 8300
+	17000 8300 17900 8300
 Wire Wire Line
 	17400 8300 17400 8400
@@
 	17400 8400 17500 8400
 Wire Wire Line
-	16900 8500 17400 8500
-Wire Wire Line
-	17400 8500 17900 8500
+	16900 8500 17900 8500
 Wire Wire Line
 	17400 8500 17400 8600
@@
 	17400 8600 17500 8600
 Wire Wire Line
-	16800 8700 17400 8700
-Wire Wire Line
-	17400 8700 17900 8700
+	16800 8700 17900 8700
 Wire Wire Line
 	17400 8700 17400 8800
@@
 	17400 8800 17500 8800
 Wire Wire Line
-	16700 8900 17400 8900
-Wire Wire Line
-	17400 8900 17900 8900
+	16700 8900 17900 8900
 Wire Wire Line
 	17400 8900 17400 9000
@@
 	17900 9100 17800 9100
 Wire Wire Line
-	17800 9100 17800 9700
-Wire Wire Line
-	17800 9700 17800 9950
-Wire Wire Line
-	19650 6600 19650 8450
-Wire Wire Line
-	19650 8450 19650 9350
+	17800 9100 17800 9950
+Wire Wire Line
+	19650 6600 19650 9350
 Wire Wire Line
 	19100 6600 19650 6600
@@
 	19400 7850 19100 7850
 Wire Wire Line
-	19400 9700 19400 8550
-Wire Wire Line
-	19400 8550 19400 7850
-Wire Wire Line
-	19400 7850 19400 7750
-Wire Wire Line
-	19400 7750 19400 7650
-Wire Wire Line
-	19400 7650 19400 7550
+	19400 9700 19400 7550
 Wire Wire Line
 	19400 7550 19100 7550
@@
 Connection ~ 19400 7850
 Wire Wire Line
-	16400 9700 17800 9700
-Wire Wire Line
-	17800 9700 19200 9700
-Wire Wire Line
-	19200 9700 19400 9700
-Wire Wire Line
-	19400 9700 19650 9700
+	16400 9700 19650 9700
 Connection ~ 19400 8550
 Connection ~ 17800 9700
@@
 Connection ~ 19200 9700
 Wire Wire Line
-	20700 9200 20700 9150
-Wire Wire Line
-	20700 9150 20750 9150
-Wire Wire Line
-	20700 8650 20700 8600
-Wire Wire Line
-	20700 8600 20750 8600
+	20400 9850 20400 9800
+Wire Wire Line
+	20400 9800 20450 9800
+Wire Wire Line
+	20400 9300 20400 9250
+Wire Wire Line
+	20400 9250 20450 9250
 Text Label 19100 9000 0    60   ~ 0
 Vtemp1
 Text Label 19100 9100 0    60   ~ 0
 Vtemp2
-Text Label 20750 8950 2    60   ~ 0
+Text Label 20450 9600 2    60   ~ 0
 Vtemp2
-Text Label 20750 8400 2    60   ~ 0
+Text Label 20450 9050 2    60   ~ 0
 Vtemp1
 Text Label 19100 9200 0    60   ~ 0
 Vref
-Text Label 20750 9050 2    60   ~ 0
+Text Label 20450 9700 2    60   ~ 0
 Vref
-Text Label 20750 8500 2    60   ~ 0
+Text Label 20450 9150 2    60   ~ 0
 Vref
 Connection ~ 19650 8450
 $Comp
-L CONN_01X04 P2
-U 1 1 5857469C
-P 20050 7200
-F 0 "P2" H 20050 7450 50  0000 C CNN
-F 1 "CONN_01X04" V 20150 7200 50  0000 C CNN
-F 2 "Pin_Headers:Pin_Header_Straight_1x04" H 20050 7200 50  0001 C CNN
-F 3 "" H 20050 7200 50  0000 C CNN
-	1    20050 7200
-	1    0    0    -1
-$EndComp
+L CONN_01X20 P2
+U 1 1 5857D8A2
+P 21300 8000
+F 0 "P2" H 21300 9050 50  0000 C CNN
+F 1 "CONN_01X20" V 21400 8000 50  0000 C CNN
+F 2 "Pin_Headers:Pin_Header_Straight_1x20_Pitch2.00mm" H 21300 8000 50  0001 C CNN
+F 3 "" H 21300 8000 50  0000 C CNN
+	1    21300 8000
+	1    0    0    -1
+$EndComp
+$Comp
+L CONN_01X20 P5
+U 1 1 5857D917
+P 22350 8050
+F 0 "P5" H 22350 9100 50  0000 C CNN
+F 1 "CONN_01X20" V 22450 8050 50  0000 C CNN
+F 2 "Pin_Headers:Pin_Header_Straight_1x20_Pitch2.00mm" H 22350 8050 50  0001 C CNN
+F 3 "" H 22350 8050 50  0000 C CNN
+	1    22350 8050
+	1    0    0    -1
+$EndComp
+Wire Wire Line
+	19100 7050 21100 7050
+Wire Wire Line
+	19100 7150 21100 7150
+Wire Wire Line
+	19100 7250 21100 7250
+Wire Wire Line
+	21100 7350 19100 7350
 $EndSCHEMATC
