File: PDB5/main.kicad_pcb (KiCad board)
At the start: 2 copper layers, 85 x 80 mm, 31 parts, among them P1 CONN_02X03, P2 CONN_01X03, P3 CONN_01X03, P4 CONN_01X02, P5 CONN_01X10, P6 CONN_01X10, P7 CONN_01X10, Q1 BC847CE6327HTSA1, Q2 BC847CE6327HTSA1, U1 PCA9698, U2 ADS7828, U3 AUIPS7111S, U4 AUIPS7111S, U5 74LVC1G08, U6 74LVC1G08, U7 Littlebee, U8 Littlebee

Commit message: test
Parts:
- added C10: C, Capacitors_SMD:C_0805, F.Cu at (263.8, 19.6)
- added C11: C, Capacitors_SMD:C_0805, F.Cu at (259.0, 29.6)
- added C12: C, Capacitors_SMD:C_0805, F.Cu at (254.9, 29.6)
- added C13: C, Capacitors_SMD:C_0805, F.Cu at (259.8, 23.3)
- added C14: C, Capacitors_SMD:C_0805, F.Cu at (255.7, 23.3)
- added C15: C, Capacitors_SMD:C_0805, F.Cu at (247.4, 32.5)
- added C16: C, Capacitors_SMD:C_0805, F.Cu at (267.9, 25.8)
- added C17: C, Capacitors_SMD:C_0805, F.Cu at (271.9, 19.6)
- added C18: C, Capacitors_SMD:C_0805, F.Cu at (221.6, 141.2)
- added C19: C, Capacitors_SMD:C_0805, F.Cu at (183.7, 163.3)
- added C20: C, Capacitors_SMD:C_0805, F.Cu at (262.9, 76.1)
- added C21: C, Capacitors_SMD:C_0805, F.Cu at (187.3, 119.1)
- added C22: C, Capacitors_SMD:C_0805, F.Cu at (224.3, 119.1)
- added C23: C, Capacitors_SMD:C_0805, F.Cu at (146.7, 163.1)
- added C24: C, Capacitors_SMD:C_0805, F.Cu at (184.6, 141.2)
- added C25: C, Capacitors_SMD:C_0805, F.Cu at (262.9, 54.0)
- added C26: CP, SMD_Packages:SMD-2010_Pol, F.Cu at (133.0, 136.7)
- added C27: CP, SMD_Packages:SMD-2010_Pol, F.Cu at (141.3, 127.6)
- added C28: C, Capacitors_SMD:C_0805, F.Cu at (138.8, 138.8)
- added C29: C, Capacitors_SMD:C_0805, F.Cu at (142.8, 138.8)
- added C30: C, Capacitors_SMD:C_0805, F.Cu at (147.7, 128.8)
- added C31: C, Capacitors_SMD:C_0805, F.Cu at (151.7, 128.8)
- added C32: C, Capacitors_SMD:C_0805, F.Cu at (147.7, 135.0)
- added C33: C, Capacitors_SMD:C_0805, F.Cu at (151.7, 135.0)
- added C34: C, Capacitors_SMD:C_0805, F.Cu at (131.2, 141.7)
- added C35: C, Capacitors_SMD:C_0805, F.Cu at (155.8, 128.8)
- added C36: C, Capacitors_SMD:C_0805, F.Cu at (139.6, 132.5)
- added C37: C, Capacitors_SMD:C_0805, F.Cu at (143.6, 132.5)
- added C38: C, Capacitors_SMD:C_1210, F.Cu at (80.8, 163.3)
- added C39: C, Capacitors_SMD:C_0805, F.Cu at (-15.0, 244.2)
- added C4: C, Capacitors_SMD:C_0805, F.Cu at (220.7, 163.3)
- added C40: C, Capacitors_SMD:C_0805, F.Cu at (-15.0, 200.4)
- added C41: C, Capacitors_SMD:C_0805, F.Cu at (-1.01, 141.9)
- added C5: C, Capacitors_SMD:C_0805, F.Cu at (262.9, 98.2)
- added C6: CP, SMD_Packages:SMD-2010_Pol, F.Cu at (257.5, 18.4)
- added C7: CP, SMD_Packages:SMD-2010_Pol, F.Cu at (249.1, 27.5)
- added C8: C, Capacitors_SMD:C_0805, F.Cu at (263.8, 25.8)
- added C9: C, Capacitors_SMD:C_0805, F.Cu at (267.9, 19.6)
- added D10: 5V, Diodes_SMD:SOD-123, F.Cu at (234.4, 129.3)
- added D11: D, Diodes_SMD:D_0603, F.Cu at (228.7, 141.0)
- added D12: 5V, Diodes_SMD:SOD-123, F.Cu at (196.5, 151.5)
- added D13: D, Diodes_SMD:D_0603, F.Cu at (190.8, 163.1)
- added D14: 5V, Diodes_SMD:SOD-123, F.Cu at (275.7, 64.2)
- added D15: D, Diodes_SMD:D_0603, F.Cu at (270.0, 75.9)
- added D16: 5V, Diodes_SMD:SOD-123, F.Cu at (200.2, 107.2)
- added D17: D, Diodes_SMD:D_0603, F.Cu at (194.4, 118.9)
- added D18: 5V, Diodes_SMD:SOD-123, F.Cu at (237.1, 107.2)
- added D19: D, Diodes_SMD:D_0603, F.Cu at (231.3, 118.9)
- added D20: 5V, Diodes_SMD:SOD-123, F.Cu at (159.6, 151.3)
- added D21: D, Diodes_SMD:D_0603, F.Cu at (153.8, 162.9)
- added D22: 5V, Diodes_SMD:SOD-123, F.Cu at (197.5, 129.3)
- added D23: D, Diodes_SMD:D_0603, F.Cu at (191.7, 141.0)
- added D24: 5V, Diodes_SMD:SOD-123, F.Cu at (275.7, 42.1)
- added D25: D, Diodes_SMD:D_0603, F.Cu at (270.0, 53.8)
- added D26: 3.3V, Diodes_SMD:SOD-123, F.Cu at (147.3, 141.2)
- added D3: LED, LEDs:LED_0603, F.Cu at (155.8, 19.0)
- added D4: 5V, Diodes_SMD:SOD-123, F.Cu at (76.8, 99.5)
- added D5: 5V, Diodes_SMD:SOD-123, F.Cu at (233.5, 151.5)
- added D6: D, Diodes_SMD:D_0603, F.Cu at (227.5, 163.1)
- added D7: 5V, Diodes_SMD:SOD-123, F.Cu at (275.7, 86.3)
- added D8: D, Diodes_SMD:D_0603, F.Cu at (269.7, 98.0)
- added D9: 3.3V, Diodes_SMD:SOD-123, F.Cu at (263.5, 32.0)
- added P10: CONN_01X02, Pin_Headers:Pin_Header_Straight_1x02, F.Cu at (120.1, 47.3)
- added P11: CONN_01X10, Pin_Headers:Pin_Header_Straight_1x10, F.Cu at (69.3, 74.1)
- added P12: CONN_01X02, Pin_Headers:Pin_Header_Straight_1x02, F.Cu at (69.3, 105.1)
- added P13: CONN_01X10, Pin_Headers:Pin_Header_Straight_1x10, F.Cu at (110.0, 22.6)
- added P14: CONN_01X10, Pin_Headers:Pin_Header_Straight_1x10, F.Cu at (59.2, 74.1)
- added P15: CONN_XT60_Female, KiCad-Dev:XT60, F.Cu at (82.8, 75.4)
- added P16: CONN_XT60_Female, KiCad-Dev:XT60, F.Cu at (133.0, 23.8)
- added P17: CONN_01X13, Pin_Headers:Pin_Header_Straight_1x13, F.Cu at (58.4, 182.9)
- added P18: CONN_01X03, Pin_Headers:Pin_Header_Straight_1x03, F.Cu at (94.0, 167.6)
- added P19: CONN_01X03, Pin_Headers:Pin_Header_Straight_1x03, F.Cu at (89.9, 157.5)
- added P20: CONN_01X13, Pin_Headers:Pin_Header_Straight_1x13, F.Cu at (-30.9, 234.1)
- added P21: CONN_01X03, Pin_Headers:Pin_Header_Straight_1x03, F.Cu at (-1.93, 234.1)
- added P22: CONN_01X03, Pin_Headers:Pin_Header_Straight_1x03, F.Cu at (-12.0, 234.1)
- added P23: CONN_01X13, Pin_Headers:Pin_Header_Straight_1x13, F.Cu at (-30.9, 190.2)
- added P24: CONN_01X03, Pin_Headers:Pin_Header_Straight_1x03, F.Cu at (-1.93, 190.2)
- added P25: CONN_01X03, Pin_Headers:Pin_Header_Straight_1x03, F.Cu at (-12.0, 190.2)
- added P26: CONN_01X13, Pin_Headers:Pin_Header_Straight_1x13, F.Cu at (-17.0, 131.8)
- added P27: CONN_01X03, Pin_Headers:Pin_Header_Straight_1x03, F.Cu at (1.99, 131.8)
- added P28: CONN_01X03, Pin_Headers:Pin_Header_Straight_1x03, F.Cu at (12.1, 131.8)
- added P8: CONN_01X02, Pin_Headers:Pin_Header_Straight_1x02, F.Cu at (110.0, 64.1)
- added P9: CONN_01X02, Pin_Headers:Pin_Header_Straight_1x02, F.Cu at (89.4, 85.7)
- added Q10: BC847CE6327HTSA1, TO_SOT_Packages_SMD:SOT-23, F.Cu at (253.1, 54.4)
- added Q3: BC847CE6327HTSA1, TO_SOT_Packages_SMD:SOT-23, F.Cu at (211.8, 141.6)
- added Q4: BC847CE6327HTSA1, TO_SOT_Packages_SMD:SOT-23, F.Cu at (173.9, 163.7)
- added Q5: BC847CE6327HTSA1, TO_SOT_Packages_SMD:SOT-23, F.Cu at (253.1, 76.5)
- added Q6: BC847CE6327HTSA1, TO_SOT_Packages_SMD:SOT-23, F.Cu at (177.5, 119.5)
- added Q7: BC847CE6327HTSA1, TO_SOT_Packages_SMD:SOT-23, F.Cu at (214.5, 119.5)
- added Q8: BC847CE6327HTSA1, TO_SOT_Packages_SMD:SOT-23, F.Cu at (137.0, 163.5)
- added Q9: BC847CE6327HTSA1, TO_SOT_Packages_SMD:SOT-23, F.Cu at (174.9, 141.6)
- added R10: R, Resistors_SMD:R_0603, F.Cu at (272.9, 92.5)
- added R100: R, Resistors_SMD:R_0805, F.Cu at (19.2, 128.6)
- added R101: R, Resistors_SMD:R_0805, F.Cu at (3.14, 147.6)
- added R102: R, Resistors_SMD:R_0805, F.Cu at (-1.31, 148.0)
- added R103: R, Resistors_SMD:R_0805, F.Cu at (-9.81, 159.7)
- added R104: R, Resistors_SMD:R_0805, F.Cu at (7.39, 141.7)
- added R105: R, Resistors_SMD:R_0805, F.Cu at (-9.81, 153.8)
- added R106: R, Resistors_SMD:R_0805, F.Cu at (-5.56, 151.7)
- added R107: R, Resistors_SMD:R_0805, F.Cu at (-5.56, 145.8)
- added R108: R, Resistors_SMD:R_0805, F.Cu at (-9.81, 148.0)
- added R109: R, Resistors_SMD:R_0805, F.Cu at (3.14, 141.7)
- added R11: R, Resistors_SMD:R_0603, F.Cu at (269.6, 92.5)
- added R12: R, Resistors_SMD:R_0603, F.Cu at (275.6, 19.4)
- added R13: R, Resistors_SMD:R_0603, F.Cu at (278.2, 25.2)
- added R14: R, Resistors_SMD:R_0603, F.Cu at (278.2, 31.1)
- added R15: R, Resistors_SMD:R_0603, F.Cu at (251.1, 32.3)
- added R16: R, Resistors_SMD:R_0603, F.Cu at (271.6, 25.6)
- added R17: R, Resistors_SMD:R_0603, F.Cu at (274.9, 25.6)
- added R18: R, Resistors_SMD:R_0603, F.Cu at (267.6, 31.9)
- added R19: R, Resistors_SMD:R_0603, F.Cu at (271.6, 31.5)
- added R20: R, Resistors_SMD:R_0603, F.Cu at (274.9, 31.5)
- added R21: R, Resistors_SMD:R_0603, F.Cu at (225.3, 135.5)
- added R22: R, Resistors_SMD:R_0603, F.Cu at (225.3, 141.4)
- added R23: R, Resistors_SMD:R_0603, F.Cu at (231.9, 135.5)
- added R24: R, Resistors_SMD:R_0603, F.Cu at (228.6, 135.5)
- added R25: R, Resistors_SMD:R_0603, F.Cu at (190.7, 157.7)
- added R26: R, Resistors_SMD:R_0603, F.Cu at (194.0, 157.7)
- added R27: R, Resistors_SMD:R_0603, F.Cu at (187.4, 163.5)
- added R28: R, Resistors_SMD:R_0603, F.Cu at (187.4, 157.7)
- added R29: R, Resistors_SMD:R_0603, F.Cu at (266.6, 70.4)
- added R30: R, Resistors_SMD:R_0603, F.Cu at (269.9, 70.4)
- added R31: R, Resistors_SMD:R_0603, F.Cu at (266.6, 76.3)
- added R32: R, Resistors_SMD:R_0603, F.Cu at (273.2, 70.4)
- added R33: R, Resistors_SMD:R_0603, F.Cu at (191.0, 113.4)
- added R34: R, Resistors_SMD:R_0603, F.Cu at (194.3, 113.4)
- added R35: R, Resistors_SMD:R_0603, F.Cu at (197.6, 113.4)
- added R36: R, Resistors_SMD:R_0603, F.Cu at (191.0, 119.3)
- added R37: R, Resistors_SMD:R_0603, F.Cu at (228.0, 119.3)
- added R38: R, Resistors_SMD:R_0603, F.Cu at (234.6, 113.4)
- added R39: R, Resistors_SMD:R_0603, F.Cu at (231.3, 113.4)
- added R40: R, Resistors_SMD:R_0603, F.Cu at (228.0, 113.4)
- added R41: R, Resistors_SMD:R_0603, F.Cu at (150.4, 157.5)
- added R42: R, Resistors_SMD:R_0603, F.Cu at (150.4, 163.3)
- added R43: R, Resistors_SMD:R_0603, F.Cu at (157.0, 157.5)
- added R44: R, Resistors_SMD:R_0603, F.Cu at (153.7, 157.5)
- added R45: R, Resistors_SMD:R_0603, F.Cu at (188.3, 141.4)
- added R46: R, Resistors_SMD:R_0603, F.Cu at (194.9, 135.5)
- added R47: R, Resistors_SMD:R_0603, F.Cu at (191.6, 135.5)
- added R48: R, Resistors_SMD:R_0603, F.Cu at (188.3, 135.5)
- added R49: R, Resistors_SMD:R_0603, F.Cu at (269.9, 48.3)
- added R50: R, Resistors_SMD:R_0603, F.Cu at (273.2, 48.3)
- added R51: R, Resistors_SMD:R_0603, F.Cu at (266.6, 48.3)
- added R52: R, Resistors_SMD:R_0603, F.Cu at (266.6, 54.2)
- added R53: R, Resistors_SMD:R_0603, F.Cu at (134.9, 141.5)
- added R54: R, Resistors_SMD:R_0603, F.Cu at (159.4, 128.6)
- added R55: R, Resistors_SMD:R_0603, F.Cu at (155.4, 134.8)
- added R56: R, Resistors_SMD:R_0603, F.Cu at (158.7, 134.8)
- added R57: R, Resistors_SMD:R_0603, F.Cu at (151.4, 141.1)
- added R58: R, Resistors_SMD:R_0603, F.Cu at (155.4, 140.7)
- added R59: R, Resistors_SMD:R_0603, F.Cu at (158.7, 140.7)
- added R60: R, Resistors_SMD:R_0603, F.Cu at (162.0, 134.4)
- added R61: R, Resistors_SMD:R_0603, F.Cu at (162.0, 140.3)
- added R62: R, Resistors_SMD:R_0805, F.Cu at (63.5, 152.4)
- added R63: R, Resistors_SMD:R_0805, F.Cu at (63.5, 154.9)
- added R64: R, Resistors_SMD:R_0805, F.Cu at (63.5, 157.5)
- added R65: R, Resistors_SMD:R_0805, F.Cu at (63.5, 160.0)
- added R66: R, Resistors_SMD:R_0805, F.Cu at (63.5, 162.6)
- added R67: R, Resistors_SMD:R_0805, F.Cu at (63.5, 165.1)
- added R68: R, Resistors_SMD:R_0805, F.Cu at (63.5, 167.6)
- added R69: R, Resistors_SMD:R_0805, F.Cu at (63.5, 170.2)
- added R70: R, Resistors_SMD:R_0805, F.Cu at (63.5, 172.7)
- added R71: R, Resistors_SMD:R_0805, F.Cu at (63.5, 175.3)
- added R72: R, Resistors_SMD:R_0805, F.Cu at (63.5, 177.8)
- added R73: R, Resistors_SMD:R_0805, F.Cu at (63.5, 180.3)
- added R74: R, Resistors_SMD:R_0805, F.Cu at (-21.0, 254.0)
- added R75: R, Resistors_SMD:R_0805, F.Cu at (-11.3, 244.0)
- added R76: R, Resistors_SMD:R_0805, F.Cu at (-24.3, 256.1)
- added R77: R, Resistors_SMD:R_0805, F.Cu at (4.75, 230.9)
- added R78: R, Resistors_SMD:R_0805, F.Cu at (-17.7, 256.1)
- added R79: R, Resistors_SMD:R_0805, F.Cu at (-14.4, 250.3)
- added R80: R, Resistors_SMD:R_0805, F.Cu at (-17.7, 250.3)
- added R81: R, Resistors_SMD:R_0805, F.Cu at (-24.3, 262.0)
- added R82: R, Resistors_SMD:R_0805, F.Cu at (-21.0, 259.8)
- added R83: R, Resistors_SMD:R_0805, F.Cu at (-21.0, 248.1)
- added R84: R, Resistors_SMD:R_0805, F.Cu at (-24.3, 250.3)
- added R85: R, Resistors_SMD:R_0805, F.Cu at (-8.02, 244.0)
- added R86: R, Resistors_SMD:R_0805, F.Cu at (-24.3, 206.4)
- added R87: R, Resistors_SMD:R_0805, F.Cu at (-21.0, 204.3)
- added R88: R, Resistors_SMD:R_0805, F.Cu at (-21.0, 210.1)
- added R89: R, Resistors_SMD:R_0805, F.Cu at (-11.3, 200.2)
- added R90: R, Resistors_SMD:R_0805, F.Cu at (-24.3, 212.3)
- added R91: R, Resistors_SMD:R_0805, F.Cu at (-21.0, 216.0)
- added R92: R, Resistors_SMD:R_0805, F.Cu at (4.75, 187.0)
- added R93: R, Resistors_SMD:R_0805, F.Cu at (-17.7, 212.3)
- added R94: R, Resistors_SMD:R_0805, F.Cu at (-14.4, 206.4)
- added R95: R, Resistors_SMD:R_0805, F.Cu at (-17.7, 206.4)
- added R96: R, Resistors_SMD:R_0805, F.Cu at (-24.3, 218.1)
- added R97: R, Resistors_SMD:R_0805, F.Cu at (-8.02, 200.2)
- added R98: R, Resistors_SMD:R_0805, F.Cu at (6.91, 147.6)
- added R99: R, Resistors_SMD:R_0805, F.Cu at (-6.04, 157.5)
- added REF**: Pin_Header_Straight_1x09, Pin_Headers:Pin_Header_Straight_1x09, F.Cu at (106.7, 172.7)
- added REF**: Pin_Header_Straight_1x09, Pin_Headers:Pin_Header_Straight_1x09, F.Cu at (127.0, 172.7)
- added U10: Littlebee, KiCad-Dev:Littlebee, F.Cu at (7.60, 22.7)
- added U11: 74LVC1G08, TO_SOT_Packages_SMD:SOT-353, F.Cu at (226.6, 151.5)
- added U12: AUIPS7111S, TO_SOT_Packages_SMD:TO-263-5Lead, F.Cu at (205.9, 154.4)
- added U13: 74LVC1G08, TO_SOT_Packages_SMD:SOT-353, F.Cu at (268.9, 86.3)
- added U14: AUIPS7111S, TO_SOT_Packages_SMD:TO-263-5Lead, F.Cu at (248.1, 89.2)
- added U15: ADS7828, Housings_SSOP:TSSOP-16_4.4x5mm_Pitch0.65mm, F.Cu at (249.5, 21.0)
- added U16: 74LVC1G08, TO_SOT_Packages_SMD:SOT-353, F.Cu at (227.6, 129.3)
- added U17: AUIPS7111S, TO_SOT_Packages_SMD:TO-263-5Lead, F.Cu at (206.8, 132.2)
- added U18: 74LVC1G08, TO_SOT_Packages_SMD:SOT-353, F.Cu at (189.7, 151.5)
- added U19: AUIPS7111S, TO_SOT_Packages_SMD:TO-263-5Lead, F.Cu at (168.9, 154.4)
- added U20: 74LVC1G08, TO_SOT_Packages_SMD:SOT-353, F.Cu at (268.9, 64.2)
- added U21: AUIPS7111S, TO_SOT_Packages_SMD:TO-263-5Lead, F.Cu at (248.1, 67.1)
- added U22: 74LVC1G08, TO_SOT_Packages_SMD:SOT-353, F.Cu at (193.3, 107.2)
- added U23: AUIPS7111S, TO_SOT_Packages_SMD:TO-263-5Lead, F.Cu at (172.5, 110.1)
- added U24: 74LVC1G08, TO_SOT_Packages_SMD:SOT-353, F.Cu at (230.2, 107.2)
- added U25: AUIPS7111S, TO_SOT_Packages_SMD:TO-263-5Lead, F.Cu at (209.5, 110.1)
- added U26: 74LVC1G08, TO_SOT_Packages_SMD:SOT-353, F.Cu at (152.7, 151.3)
- added U27: AUIPS7111S, TO_SOT_Packages_SMD:TO-263-5Lead, F.Cu at (132.0, 154.2)
- added U28: 74LVC1G08, TO_SOT_Packages_SMD:SOT-353, F.Cu at (190.6, 129.3)
- added U29: AUIPS7111S, TO_SOT_Packages_SMD:TO-263-5Lead, F.Cu at (169.9, 132.2)
- added U30: 74LVC1G08, TO_SOT_Packages_SMD:SOT-353, F.Cu at (268.9, 42.1)
- added U31: AUIPS7111S, TO_SOT_Packages_SMD:TO-263-5Lead, F.Cu at (248.1, 45.0)
- added U32: ADS7828, Housings_SSOP:TSSOP-16_4.4x5mm_Pitch0.65mm, F.Cu at (133.4, 130.2)
- added U33: LTC6802-2, KiCad-Dev:SSOP-44, F.Cu at (74.1, 161.0)
- added U34: LTC6802-2, KiCad-Dev:SSOP-44, F.Cu at (-21.5, 235.4)
- added U35: LTC6802-2, KiCad-Dev:SSOP-44, F.Cu at (-21.5, 191.5)
- added U36: LTC6802-2, KiCad-Dev:SSOP-44, F.Cu at (-7.54, 133.0)
- added U9: Littlebee, KiCad-Dev:Littlebee, F.Cu at (33.0, 22.7)
- C1: value CP -> C; footprint SMD_Packages:SMD-1206_Pol -> Capacitors_SMD:C_0805
- C2: footprint SMD_Packages:SMD-1206_Pol -> SMD_Packages:SMD-2010_Pol
- D1: value D -> ZENER; footprint Diodes_SMD:D_0603 -> Diodes_SMD:SOD-123; moved to F.Cu
- D2: value D -> LED; footprint Diodes_SMD:D_0603 -> LEDs:LED_0603; moved to F.Cu
- P1: value CONN_02X03 -> CONN_01X03; footprint Pin_Headers:Pin_Header_Straight_2x03 -> Pin_Headers:Pin_Header_Straight_1x03
- P2, P3: value CONN_01X03 -> CONN_01X02; footprint Pin_Headers:Pin_Header_Straight_1x03 -> Pin_Headers:Pin_Header_Straight_1x02
- P5, P7: value CONN_01X10 -> CONN_01X02; footprint Pin_Headers:Pin_Header_Straight_1x10 -> Pin_Headers:Pin_Header_Straight_1x02; moved to F.Cu
- P6: value CONN_01X10 -> CONN_02X03; footprint Pin_Headers:Pin_Header_Straight_1x10 -> Pin_Headers:Pin_Header_Straight_2x03; moved to F.Cu
- Q1, Q2, R2, R3, R4, R5, R6, R7, R8, R9: moved to F.Cu
- U1: value PCA9698 -> SC18IS602B; footprint Housings_SSOP:TSSOP-56_6.1x14mm_Pitch0.5mm -> Housings_SSOP:TSSOP-16_4.4x5mm_Pitch0.65mm
- U2: value ADS7828 -> PCA9698; footprint Housings_SSOP:TSSOP-16_4.4x5mm_Pitch0.65mm -> Housings_SSOP:TSSOP-56_6.1x14mm_Pitch0.5mm
- U3, U4: value AUIPS7111S -> Littlebee; footprint TO_SOT_Packages_SMD:TO-263-5Lead -> KiCad-Dev:Littlebee; moved to F.Cu
- U5, U6: value 74LVC1G08 -> Littlebee; footprint TO_SOT_Packages_SMD:SOT-353 -> KiCad-Dev:Littlebee; moved to F.Cu
- moved U5 250.4 mm to (-17.8, 22.7)
- moved U1 240.7 mm to (-43.2, 171.4)
- moved U6 226.3 mm to (-17.8, 74.2)
- moved U4 210.1 mm to (7.60, 74.2), turned to 0 degrees
- moved P1 202.3 mm to (59.2, 105.1)
- moved U3 193.6 mm to (33.0, 74.2), turned to 0 degrees
- moved U8 190.9 mm to (58.4, 22.7), turned to 0 degrees
- moved U7 187.5 mm to (83.8, 22.7), turned to 0 degrees
- moved P6 170.7 mm to (129.5, 34.2), turned to 0 degrees
- moved P5 151.3 mm to (110.0, 53.5), turned to 0 degrees
- moved D1 142.6 mm to (81.0, 93.2), turned to 0 degrees
- moved P7 135.5 mm to (139.6, 34.2), turned to 0 degrees
- moved U2 132.2 mm to (119.8, 25.5)
- moved R2 124.9 mm to (102.5, 70.9), turned to 0 degrees
- moved R3 123.8 mm to (146.2, 30.0)
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Connections:
- C2 pad 1: Net-(C2-Pad1) -> +3V3
- C3 pad 1: Net-(C3-Pad1) -> +3V3
- D1 pad 1: Net-(D1-Pad1) -> GND
- D1 pad 2: GND -> +3V3
- D2 pad 1: Net-(D2-Pad1) -> /GPIO_INT
- D2 pad 2: GND -> Net-(D2-Pad2)
- P1 pad 2: +3V3 -> /GPIO_OE
- P1 pad 3: /SDA -> +3V3
- P2 pad 1: GND -> /SCL
- P3 pad 1: GND -> Net-(P3-Pad1)
- P3 pad 2: Net-(P3-Pad2) -> /SDA
- P4 pad 1: +3V3 -> /SCL
- P4 pad 2: /pwr_mod_1/Power_Enanle_B -> Net-(P4-Pad2)
- P5 pad 1: /Enable_1 -> Net-(P5-Pad1)
- P5 pad 2: /Enable_2 -> /SDA
- P6 pad 1: /PWM1 -> GND
- P6 pad 2: /PWM2 -> +3V3
- P6 pad 3: (no net) -> /SDA
- P6 pad 4: (no net) -> /RST
- P6 pad 5: (no net) -> /SCL
- P7 pad 1: /CH1 -> /SCL
- P7 pad 2: /CH2 -> /ADC_1/SDA
- Q1 pad 3: Net-(D1-Pad1) -> Net-(D6-Pad1)
- Q2 pad 3: Net-(D2-Pad1) -> Net-(D8-Pad1)
- R1 pad 1: Net-(C2-Pad1) -> Net-(D2-Pad2)
- R2 pad 1: Net-(Q1-Pad1) -> Net-(D3-Pad2)
- R2 pad 2: Net-(R2-Pad2) -> +3V3
- R3 pad 1: Net-(Q1-Pad1) -> +3V3
- R3 pad 2: GND -> /RST
- R4 pad 1: Net-(R4-Pad1) -> Net-(Q1-Pad1)
- R4 pad 2: /CH1 -> Net-(R4-Pad2)
- R5 pad 1: GND -> Net-(Q1-Pad1)
- R5 pad 2: Net-(R4-Pad1) -> GND
- R6 pad 1: Net-(Q2-Pad1) -> Net-(R6-Pad1)
- R6 pad 2: Net-(R6-Pad2) -> /CH1
- R7 pad 1: Net-(Q2-Pad1) -> GND
- R7 pad 2: GND -> Net-(R6-Pad1)
- R8 pad 1: Net-(R8-Pad1) -> Net-(Q2-Pad1)
- R8 pad 2: /CH2 -> Net-(R8-Pad2)
- R9 pad 1: GND -> Net-(Q2-Pad1)
- R9 pad 2: Net-(R8-Pad1) -> GND
- U1 pad 1: /SDA -> /SS0
- U1 pad 10: (no net) -> /SS2
- U1 pad 11: GND -> /SCKI
- U1 pad 12: (no net) -> +3V3
- U1 pad 13: (no net) -> /SS3
- U1 pad 14: (no net) -> GND
- U1 pad 15: (no net) -> GND
- U1 pad 16: (no net) -> GND
- U1 pad 2: /SCL -> /SS1
- U1 pad 3: /Enable_1 -> /RST
- U1 pad 4: /Enable_2 -> GND
- U1 pad 5: (no net) -> /SDI
- U1 pad 6: GND -> /SDO
- U1 pad 7: (no net) -> Net-(P3-Pad1)
- U1 pad 8: (no net) -> Net-(P2-Pad2)
- U1 pad 9: (no net) -> Net-(D3-Pad1)
- U2 pad 1: /CH1 -> Net-(P5-Pad1)
- U2 pad 10: Net-(C3-Pad1) -> /Enable_7
- U2 pad 12: Net-(P3-Pad2) -> /Enable_8
- U2 pad 13: Net-(P2-Pad2) -> /Enable_9
- U2 pad 14: /SCL -> /Enable_10
- U2 pad 15: /SDA -> (no net)
- U2 pad 16: Net-(C2-Pad1) -> (no net)
- U2 pad 2: /CH2 -> Net-(P4-Pad2)
- U2 pad 3: /CH3 -> /Enable_1
- U2 pad 4: /CH4 -> /Enable_2
- U2 pad 5: /CH5 -> /Enable_3
- U2 pad 6: /CH6 -> GND
- U2 pad 7: /CH7 -> /Enable_4
- U2 pad 8: /CH8 -> /Enable_5
- U2 pad 9: GND -> /Enable_6
- U3 pad 1: Net-(D1-Pad1) -> /pwr_mod_1/Power_Out
- U3 pad 2: Net-(R4-Pad1) -> GND
- U3 pad 3: +BATT -> GND
- U3 pad 4: /pwr_mod_1/Power_Out -> /PWM1
- U3 pad 5: /pwr_mod_1/Power_Out -> (no net)
- U4 pad 1: Net-(D2-Pad1) -> /pwr_mod_2/Power_Out
- U4 pad 2: Net-(R8-Pad1) -> GND
- U4 pad 3: +BATT -> GND
- U4 pad 4: /pwr_mod_2/Power_Out -> /PWM2
- U4 pad 5: /pwr_mod_2/Power_Out -> (no net)
- U5 pad 1: /Enable_1 -> /pwr_mod_3/Power_Out
- U5 pad 2: /pwr_mod_1/Power_Enanle_B -> GND
- U5 pad 4: Net-(R2-Pad2) -> /PWM3
- U5 pad 5: +3V3 -> (no net)
- U6 pad 1: /Enable_2 -> /pwr_mod_4/Power_Out
- U6 pad 2: /pwr_mod_1/Power_Enanle_B -> GND
- U6 pad 4: Net-(R6-Pad2) -> /PWM4
- U6 pad 5: +3V3 -> (no net)
- U7 pad 1: /pwr_mod_1/Power_Out -> /pwr_mod_5/Power_Out
- U7 pad 4: /PWM1 -> /PWM5
- U8 pad 1: /pwr_mod_2/Power_Out -> /pwr_mod_6/Power_Out
- U8 pad 4: /PWM2 -> /PWM6
Routing:
- net GND: track 0.01 -> 25.1 mm
- net /BMS_1/C5: track 0.00 -> 15.5 mm
- net /BMS_1/C12: track 0.00 -> 15.4 mm
- net /BMS_1/C6: track 0.00 -> 14.4 mm
- net /BMS_1/C11: track 0.00 -> 14.2 mm
- net /BMS_1/C7: track 0.00 -> 13.8 mm
- net /BMS_1/C10: track 0.00 -> 13.3 mm
- net /BMS_1/C8: track 0.00 -> 13.1 mm
- net /BMS_1/C9: track 0.00 -> 12.8 mm
- net Net-(R8-Pad1): track 11.0 -> 0.00 mm
- net Net-(R68-Pad1): track 0.00 -> 8.35 mm
- net Net-(R62-Pad1): track 0.00 -> 7.95 mm
- net Net-(P18-Pad2): track 0.00 -> 7.54 mm
- net Net-(R67-Pad1): track 0.00 -> 7.53 mm
- net Net-(R63-Pad1): track 0.00 -> 7.32 mm
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- removed copper zone on B.Cu, net (none)
- removed copper zone on F.Cu, net (none)
- removed copper zone on F.Cu, net /PWM1
- removed copper zone on B.Cu, net /pwr_mod_1/Power_Out
- removed copper zone on B.Cu, net /pwr_mod_2/Power_Out
- removed copper zone on B.Cu, net GND
Other:
- board outline removed
- net class Default: via_dia 1.3 -> 0.8; via_drill 1 -> 0.4

Commit message: test
Parts:
- moved C39 70.1 mm to (55.0, 241.2)
- moved P20 70.1 mm to (39.1, 231.1)
- moved P21 70.1 mm to (68.1, 231.1)
- moved P22 70.1 mm to (58.0, 231.1)
- moved R74 70.1 mm to (49.0, 251.0)
- moved R75 70.1 mm to (58.7, 241.0)
- moved R76 70.1 mm to (45.7, 253.1)
- moved R77 70.1 mm to (74.8, 227.9)
- moved R78 70.1 mm to (52.3, 253.1)
- moved R79 70.1 mm to (55.6, 247.3)
- moved R80 70.1 mm to (52.3, 247.3)
- moved R81 70.1 mm to (45.7, 259.0)
- moved R82 70.1 mm to (49.0, 256.8)
- moved R83 70.1 mm to (49.0, 245.1)
- moved R84 70.1 mm to (45.7, 247.3)
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Changed lines of the file:
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@@
-(kicad_pcb (version 4) (host pcbnew 4.0.4-stable)
+(kicad_pcb (version 4) (host pcbnew 4.0.4+e1-6308~48~ubuntu16.04.1-stable)
   (general
-    (links 0)
+    (links 649)
     (no_connects 626)
     (area -47.951428 16.5 279.804762 266.570001)
@@
   )
   (module Capacitors_SMD:C_0805 (layer F.Cu)
-    (at -14.994999 244.245)
+    (at 55.005001 241.245)
     (descr "Capacitor SMD 0805, reflow soldering, AVX (see smccp.pdf)")
     (tags "capacitor 0805")
@@
   )
   (module Pin_Headers:Pin_Header_Straight_1x13 (layer F.Cu)
-    (at -30.946667 234.095)
+    (at 39.053333 231.095)
     (descr "Through hole pin header")
     (tags "pin header")
@@
   )
   (module Pin_Headers:Pin_Header_Straight_1x03 (layer F.Cu)
-    (at -1.926667 234.095)
+    (at 68.073333 231.095)
     (descr "Through hole pin header")
     (tags "pin header")
@@
   )
   (module Pin_Headers:Pin_Header_Straight_1x03 (layer F.Cu)
-    (at -11.986667 234.095)
+    (at 58.013333 231.095)
     (descr "Through hole pin header")
     (tags "pin header")
@@
   )
   (module KiCad-Dev:SSOP-44 placed (layer F.Cu)
-    (at -21.519056 235.361459)
+    (at 48.480944 232.361459)
     (solder_mask_margin 0.0508)
     (fp_text reference U34 (at 0.127 8.235542 270) (layer F.SilkS)
@@
   )
   (module Resistors_SMD:R_0805 (layer F.Cu)
-    (at -20.967619 253.995)
+    (at 49.032381 250.995)
     (descr "Resistor SMD 0805, reflow soldering, Vishay (see dcrcw.pdf)")
     (tags "resistor 0805")
@@
   )
   (module Resistors_SMD:R_0805 (layer F.Cu)
-    (at -11.317619 244.045)
+    (at 58.682381 241.045)
     (descr "Resistor SMD 0805, reflow soldering, Vishay (see dcrcw.pdf)")
     (tags "resistor 0805")
@@
   )
   (module Resistors_SMD:R_0805 (layer F.Cu)
-    (at -24.267619 256.145)
+    (at 45.732381 253.145)
     (descr "Resistor SMD 0805, reflow soldering, Vishay (see dcrcw.pdf)")
     (tags "resistor 0805")
@@
   )
   (module Resistors_SMD:R_0805 (layer F.Cu)
-    (at 4.752381 230.895)
+    (at 74.752381 227.895)
     (descr "Resistor SMD 0805, reflow soldering, Vishay (see dcrcw.pdf)")
     (tags "resistor 0805")
@@
   )
   (module Resistors_SMD:R_0805 (layer F.Cu)
-    (at -17.667619 256.145)
+    (at 52.332381 253.145)
     (descr "Resistor SMD 0805, reflow soldering, Vishay (see dcrcw.pdf)")
     (tags "resistor 0805")
@@
   )
   (module Resistors_SMD:R_0805 (layer F.Cu)
-    (at -14.367619 250.295)
+    (at 55.632381 247.295)
     (descr "Resistor SMD 0805, reflow soldering, Vishay (see dcrcw.pdf)")
     (tags "resistor 0805")
@@
   )
   (module Resistors_SMD:R_0805 (layer F.Cu)
-    (at -17.667619 250.295)
+    (at 52.332381 247.295)
     (descr "Resistor SMD 0805, reflow soldering, Vishay (see dcrcw.pdf)")
     (tags "resistor 0805")
@@
   )
   (module Resistors_SMD:R_0805 (layer F.Cu)
-    (at -24.267619 261.995)
+    (at 45.732381 258.995)
     (descr "Resistor SMD 0805, reflow soldering, Vishay (see dcrcw.pdf)")
     (tags "resistor 0805")
@@
   )
   (module Resistors_SMD:R_0805 (layer F.Cu)
-    (at -20.967619 259.845)
+    (at 49.032381 256.845)
     (descr "Resistor SMD 0805, reflow soldering, Vishay (see dcrcw.pdf)")
     (tags "resistor 0805")
@@
   )
   (module Resistors_SMD:R_0805 (layer F.Cu)
-    (at -20.967619 248.145)
+    (at 49.032381 245.145)
     (descr "Resistor SMD 0805, reflow soldering, Vishay (see dcrcw.pdf)")
     (tags "resistor 0805")
@@
   )
   (module Resistors_SMD:R_0805 (layer F.Cu)
-    (at -24.267619 250.295)
+    (at 45.732381 247.295)
     (descr "Resistor SMD 0805, reflow soldering, Vishay (see dcrcw.pdf)")
     (tags "resistor 0805")
@@
   )
   (module Resistors_SMD:R_0805 (layer F.Cu)
-    (at -8.017619 244.045)
+    (at 61.982381 241.045)
     (descr "Resistor SMD 0805, reflow soldering, Vishay (see dcrcw.pdf)")
     (tags "resistor 0805")

Commit message: test
Parts:
- removed D11, D13, D15, D17, D19, D21, D23, D25, D6, D8: D, Diodes_SMD:D_0603
- removed Q1, Q10, Q2, Q3, Q4, Q5, Q6, Q7, Q8, Q9: BC847CE6327HTSA1, TO_SOT_Packages_SMD:SOT-23
- removed R10, R23, R27, R31, R35, R39, R43, R47, R51, R6: R, Resistors_SMD:R_0603
- removed the REF** at (106.7, 172.7)
- removed the REF** at (127.0, 172.7)
- added REF**: MountingHole_4.3mm_M4, Mounting_Holes:MountingHole_4.3mm_M4, F.Cu at (20.0, 41.0)
- added REF**: MountingHole_4.3mm_M4, Mounting_Holes:MountingHole_4.3mm_M4, F.Cu at (82.0, 133.0)
- added REF**: MountingHole_4.3mm_M4, Mounting_Holes:MountingHole_4.3mm_M4, F.Cu at (144.0, 41.0)
- added REF**: MountingHole_4.3mm_M4, Mounting_Holes:MountingHole_4.3mm_M4, F.Cu at (113.0, 41.0)
- added REF**: MountingHole_4.3mm_M4, Mounting_Holes:MountingHole_4.3mm_M4, F.Cu at (82.0, 41.0)
- added REF**: MountingHole_4.3mm_M4, Mounting_Holes:MountingHole_4.3mm_M4, F.Cu at (51.0, 41.0)
- added REF**: MountingHole_4.3mm_M4, Mounting_Holes:MountingHole_4.3mm_M4, F.Cu at (144.0, 133.0)
- added REF**: MountingHole_4.3mm_M4, Mounting_Holes:MountingHole_4.3mm_M4, F.Cu at (113.0, 133.0)
- added REF**: MountingHole_4.3mm_M4, Mounting_Holes:MountingHole_4.3mm_M4, F.Cu at (19.0, 133.0)
- added REF**: MountingHole_4.3mm_M4, Mounting_Holes:MountingHole_4.3mm_M4, F.Cu at (51.0, 133.0)
- C18, C19, C20, C21, C22, C23, C25, C4, C5, D10, D12, D14, D16, D18, D20, D24, D5, D7, R11, R21, R22, R24, R25, R26, R28, R29, R30, R32, R33, R34, R36, R37, R38, R4, R40, R41, R42, R44, R49, R5, R50, R52, R7, R8, R9, U11, U13, U16, U18, U20, U22, U24, U26, U30: moved to B.Cu
- C38: footprint Capacitors_SMD:C_1210 -> Capacitors_SMD:C_0805
- U12, U14, U17, U19, U21, U23, U25, U27, U31: footprint TO_SOT_Packages_SMD:TO-263-5Lead -> KiCad-Dev:TO-263-!3; moved to B.Cu
- U29: footprint TO_SOT_Packages_SMD:TO-263-5Lead -> KiCad-Dev:TO-263-!3
- moved C3 597.3 mm to (662.9, 142.8)
- moved D4 597.3 mm to (673.4, 129.6)
- moved P11 597.3 mm to (665.9, 104.2)
- moved P12 597.3 mm to (665.9, 135.2)
- moved P4 597.3 mm to (692.5, 104.2)
- moved P9 597.3 mm to (686.0, 115.8)
- moved C1 597.3 mm to (672.9, 123.4)
- moved D1 597.3 mm to (677.6, 123.3)
- moved P1 597.3 mm to (655.8, 135.2)
- moved P14 597.3 mm to (655.8, 104.2)
- moved P15 597.3 mm to (679.4, 105.5)
- moved P3 597.3 mm to (675.9, 115.8)
- moved R2 597.3 mm to (699.0, 101.0)
- moved C26 558.6 mm to (691.4, 147.8)
- moved C27 558.6 mm to (699.8, 138.6)
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Connections:
- R11 pad 2: Net-(R10-Pad1) -> /CH2
- R21 pad 1: Net-(Q3-Pad1) -> GND
- R21 pad 2: Net-(R21-Pad2) -> /Enable_3
- R22 pad 1: Net-(Q3-Pad1) -> GND
- R22 pad 2: GND -> /pwr_mod_1/Power_Enanle_B
- R24 pad 2: Net-(R23-Pad1) -> /CH3
- R25 pad 1: Net-(Q4-Pad1) -> GND
- R25 pad 2: Net-(R25-Pad2) -> /Enable_4
- R26 pad 1: Net-(Q4-Pad1) -> GND
- R26 pad 2: GND -> /pwr_mod_1/Power_Enanle_B
- R28 pad 2: Net-(R27-Pad1) -> /CH4
- R29 pad 1: Net-(Q5-Pad1) -> GND
- R29 pad 2: Net-(R29-Pad2) -> /Enable_5
- R30 pad 1: Net-(Q5-Pad1) -> GND
- R30 pad 2: GND -> /pwr_mod_1/Power_Enanle_B
- R32 pad 2: Net-(R31-Pad1) -> /CH5
- R33 pad 1: Net-(Q6-Pad1) -> GND
- R33 pad 2: Net-(R33-Pad2) -> /Enable_6
- R34 pad 1: Net-(Q6-Pad1) -> GND
- R34 pad 2: GND -> /pwr_mod_1/Power_Enanle_B
- R36 pad 2: Net-(R35-Pad1) -> /CH6
- R37 pad 1: Net-(Q7-Pad1) -> GND
- R37 pad 2: Net-(R37-Pad2) -> /Enable_7
- R38 pad 1: Net-(Q7-Pad1) -> GND
- R38 pad 2: GND -> /pwr_mod_1/Power_Enanle_B
- R4 pad 1: Net-(Q1-Pad1) -> GND
- R4 pad 2: Net-(R4-Pad2) -> /Enable_1
- R40 pad 2: Net-(R39-Pad1) -> /CH7
- R41 pad 1: Net-(Q8-Pad1) -> GND
- R41 pad 2: Net-(R41-Pad2) -> /Enable_8
- R42 pad 1: Net-(Q8-Pad1) -> GND
- R42 pad 2: GND -> /pwr_mod_1/Power_Enanle_B
- R44 pad 2: Net-(R43-Pad1) -> /CH8
- R45 pad 1: Net-(Q9-Pad1) -> GND
- R45 pad 2: Net-(R45-Pad2) -> /Enable_9
- R46 pad 1: Net-(Q9-Pad1) -> GND
- R46 pad 2: GND -> /pwr_mod_1/Power_Enanle_B
- R48 pad 2: Net-(R47-Pad1) -> /CH9
- R49 pad 1: Net-(Q10-Pad1) -> GND
- R49 pad 2: Net-(R49-Pad2) -> /Enable_10
- R5 pad 1: Net-(Q1-Pad1) -> GND
- R5 pad 2: GND -> /pwr_mod_1/Power_Enanle_B
- R50 pad 1: Net-(Q10-Pad1) -> GND
- R50 pad 2: GND -> /pwr_mod_1/Power_Enanle_B
- R52 pad 2: Net-(R51-Pad1) -> /CH10
- R7 pad 2: Net-(R6-Pad1) -> /CH1
- R8 pad 1: Net-(Q2-Pad1) -> GND
- R8 pad 2: Net-(R8-Pad2) -> /Enable_2
- R9 pad 1: Net-(Q2-Pad1) -> GND
- R9 pad 2: GND -> /pwr_mod_1/Power_Enanle_B
- U11 pad 4: Net-(R4-Pad2) -> Net-(U11-Pad4)
- U12 pad 1: Net-(D6-Pad1) -> Net-(U11-Pad4)
- U12 pad 2: Net-(R6-Pad1) -> /CH1
- U13 pad 4: Net-(R8-Pad2) -> Net-(U13-Pad4)
- U14 pad 1: Net-(D8-Pad1) -> Net-(U13-Pad4)
- U14 pad 2: Net-(R10-Pad1) -> /CH2
- U16 pad 4: Net-(R21-Pad2) -> Net-(U16-Pad4)
- U17 pad 1: Net-(D11-Pad1) -> Net-(U16-Pad4)
- U17 pad 2: Net-(R23-Pad1) -> /CH3
- U18 pad 4: Net-(R25-Pad2) -> Net-(U18-Pad4)
- U19 pad 1: Net-(D13-Pad1) -> Net-(U18-Pad4)
- U19 pad 2: Net-(R27-Pad1) -> /CH4
- U20 pad 4: Net-(R29-Pad2) -> Net-(U20-Pad4)
- U21 pad 1: Net-(D15-Pad1) -> Net-(U20-Pad4)
- U21 pad 2: Net-(R31-Pad1) -> /CH5
- U22 pad 4: Net-(R33-Pad2) -> Net-(U22-Pad4)
- U23 pad 1: Net-(D17-Pad1) -> Net-(U22-Pad4)
- U23 pad 2: Net-(R35-Pad1) -> /CH6
- U24 pad 4: Net-(R37-Pad2) -> Net-(U24-Pad4)
- U25 pad 1: Net-(D19-Pad1) -> Net-(U24-Pad4)
- U25 pad 2: Net-(R39-Pad1) -> /CH7
- U26 pad 4: Net-(R41-Pad2) -> Net-(U26-Pad4)
- U27 pad 1: Net-(D21-Pad1) -> Net-(U26-Pad4)
- U27 pad 2: Net-(R43-Pad1) -> /CH8
- U28 pad 4: Net-(R45-Pad2) -> Net-(U28-Pad4)
- U29 pad 1: Net-(D23-Pad1) -> Net-(U28-Pad4)
- U29 pad 2: Net-(R47-Pad1) -> /CH9
- U30 pad 4: Net-(R49-Pad2) -> Net-(U30-Pad4)
- U31 pad 1: Net-(D25-Pad1) -> Net-(U30-Pad4)
- U31 pad 2: Net-(R51-Pad1) -> /CH10
Routing:
- net GND: track 25.1 -> 49.3 mm
- net /BMS_1/C5: track 15.5 -> 0.00 mm
- net /BMS_1/C12: track 15.4 -> 0.00 mm
- net /BMS_1/C6: track 14.4 -> 0.00 mm
- net /BMS_1/C11: track 14.2 -> 0.00 mm
- net /BMS_1/C7: track 13.8 -> 0.00 mm
- net /BMS_1/C10: track 13.3 -> 0.00 mm
- net /BMS_1/C8: track 13.1 -> 0.00 mm
- net /BMS_1/C9: track 12.8 -> 0.00 mm
- net /CH4: track 0.00 -> 8.55 mm
- net /CH7: track 0.00 -> 8.41 mm
- net +3V3: track 0.00 -> 8.41 mm
- net Net-(R68-Pad1): track 8.35 -> 0.00 mm
- net Net-(R62-Pad1): track 7.95 -> 0.00 mm
- net Net-(P18-Pad2): track 7.54 -> 0.00 mm
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- added copper zone on B.Cu, net /pwr_mod_4/Power_Out
- added copper zone on B.Cu, net GND
Other:
- board outline added: 140 x 140 mm
