File: PDB5/main.kicad_pcb (KiCad board)
At the start: 2 copper layers, 140 x 140 mm, 230 parts, among them P1 CONN_01X03, P10 CONN_01X02, P11 CONN_01X10, P12 CONN_01X02, P13 CONN_01X10, P14 CONN_01X10, P15 CONN_XT60_Female, P16 CONN_XT60_Female, P17 CONN_01X13, P18 CONN_01X03, P19 CONN_01X03, P2 CONN_01X02, P20 CONN_01X13, P21 CONN_01X03, P22 CONN_01X03, P23 CONN_01X13, P24 CONN_01X03, P25 CONN_01X03, P26 CONN_01X13, P27 CONN_01X03, P28 CONN_01X03, P3 CONN_01X02, P4 CONN_01X02, P5 CONN_01X02, P6 CONN_02X03, P7 CONN_01X02, P8 CONN_01X02, P9 CONN_01X02, U1 SC18IS602B, U10 Littlebee, U11 74LVC1G08, U12 AUIPS7111S, U13 74LVC1G08, U14 AUIPS7111S, U15 ADS7828, U16 74LVC1G08, U17 AUIPS7111S, U18 74LVC1G08, U19 AUIPS7111S, U2 PCA9698, U20 74LVC1G08, U21 AUIPS7111S, U22 74LVC1G08, U23 AUIPS7111S, U24 74LVC1G08, U25 AUIPS7111S, U26 74LVC1G08, U27 AUIPS7111S, U28 74LVC1G08, U29 AUIPS7111S, U3 Littlebee, U30 74LVC1G08, U31 AUIPS7111S, U32 ADS7828, U33 LTC6802-2, U34 LTC6802-2, U35 LTC6802-2, U36 LTC6802-2, U4 Littlebee, U5 Littlebee, U6 Littlebee, U7 Littlebee, U8 Littlebee, U9 Littlebee

Commit message: test
Parts:
- C24, D22, R45, R46, R48, U28, U29: moved to B.Cu
- moved P15 516.2 mm to (164.0, 133.0), turned to 180 degrees
- moved P16 499.8 mm to (164.0, 41.0)
- moved U30 58.2 mm to (161.0, 72.2)
- moved U31 58.2 mm to (167.4, 72.4)
- moved R52 58.2 mm to (162.8, 73.4)
- moved C25 58.2 mm to (159.1, 73.6)
- moved D24 58.2 mm to (163.5, 67.1)
- moved R49 58.2 mm to (159.1, 67.1)
- moved R50 58.2 mm to (161.8, 69.7)
- moved D22 49.6 mm to (169.0, 115.0)
- moved U2 46.3 mm to (97.0, 87.0), turned to 90 degrees
- moved R48 41.5 mm to (171.1, 119.5)
- moved R46 41.5 mm to (177.7, 119.5)
- moved U28 39.2 mm to (161.0, 97.0), turned to 90 degrees
- moved U29 33.7 mm to (155.0, 101.0), turned to 180 degrees
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Routing:
- net GND: vias 0 -> 72
- net +BATT: vias 0 -> 63
- added copper zone on B.Cu, net +BATT
- added copper zone on In2.Cu, net +BATT
- added copper zone on B.Cu, net /pwr_mod_1/Power_Out
- added copper zone on B.Cu, net /pwr_mod_2/Power_Out
- added copper zone on B.Cu, net /pwr_mod_3/Power_Out
- added copper zone on B.Cu, net /pwr_mod_5/Power_Out
- added copper zone on B.Cu, net /pwr_mod_6/Power_Out
- added copper zone on B.Cu, net /pwr_mod_7/Power_Out
- added copper zone on B.Cu, net /pwr_mod_8/Power_Out
- added copper zone on In1.Cu, net GND
Other:
- board size 140 x 140 mm -> 170 x 140 mm
- copper layers 2 -> 4
