File: PDB5/ADC.sch (KiCad schematic (older format))
At the start: 25 parts, among them P8 CONN_01X03, P9 CONN_01X03, U14 ADS7828

Commit message: test
Parts:
- removed P8, P9: CONN_01X03, Pin_Headers:Pin_Header_Straight_1x03, symbol CONN_01X03
- C10: renamed from C7; footprint (none) -> Capacitors_SMD:C_0805
- C11: renamed from C8; footprint (none) -> Capacitors_SMD:C_0805
- C12: renamed from C9; footprint (none) -> Capacitors_SMD:C_0805
- C13: renamed from C10; footprint (none) -> Capacitors_SMD:C_0805
- C14: renamed from C11; footprint (none) -> Capacitors_SMD:C_0805
- C15: renamed from C12; footprint (none) -> Capacitors_SMD:C_0805
- C16: renamed from C13; footprint (none) -> Capacitors_SMD:C_0805
- C17: renamed from C14; footprint (none) -> Capacitors_SMD:C_0805
- C6: renamed from C4; footprint SMD_Packages:SMD-1206_Pol -> SMD_Packages:SMD-2010_Pol
- C7: renamed from C5; footprint SMD_Packages:SMD-1206_Pol -> SMD_Packages:SMD-2010_Pol
- D9: renamed from D?; footprint (none) -> Diodes_SMD:SOD-123
- R13: renamed from R11; footprint (none) -> Resistors_SMD:R_0603
- R14: renamed from R12; footprint (none) -> Resistors_SMD:R_0603
- R15: renamed from R13; footprint (none) -> Resistors_SMD:R_0603
- R16: renamed from R14; footprint (none) -> Resistors_SMD:R_0603
- R17: renamed from R15; footprint (none) -> Resistors_SMD:R_0603
- R18: renamed from R16; footprint (none) -> Resistors_SMD:R_0603
- R19, R20: renamed from R?; footprint (none) -> Resistors_SMD:R_0603
- gave numbers to parts that had none: 1
- renumbered C6 to C9, R10 to R12, U14 to U15
Connections:
- net A0: now reaches U15.12 (A0)
- net A1: now reaches U15.13 (A1)
