File: PDB5/BMS.sch (KiCad schematic (older format))
At the start: 17 parts, among them P17 CONN_01X13, P18 CONN_01X03, P19 CONN_01X03, U33 LTC6802-2

Commit message: test
Changed lines of the file:
@@
 AR Path="/58561F68/58556E47" Ref="U35"  Part="1"
 AR Path="/585624EB/58556E47" Ref="U36"  Part="1"
-F 0 "U33" H 7900 5250 60  0000 C CNN
+F 0 "U36" H 7900 5250 60  0000 C CNN
 F 1 "LTC6802-2" H 7900 5350 60  0000 C CNN
 F 2 "KiCad-Dev:SSOP-44" H 7550 4100 60  0001 C CNN
@@
 AR Path="/58561F68/58556E86" Ref="R86"  Part="1"
 AR Path="/585624EB/58556E86" Ref="R98"  Part="1"
-F 0 "R62" V 7080 3250 50  0000 C CNN
+F 0 "R98" V 7080 3250 50  0000 C CNN
 F 1 "R" V 7000 3250 50  0000 C CNN
 F 2 "Resistors_SMD:R_0805" V 6930 3250 50  0001 C CNN
@@
 AR Path="/58561F68/58556F97" Ref="R87"  Part="1"
 AR Path="/585624EB/58556F97" Ref="R99"  Part="1"
-F 0 "R63" V 7080 3450 50  0000 C CNN
+F 0 "R99" V 7080 3450 50  0000 C CNN
 F 1 "R" V 7000 3450 50  0000 C CNN
 F 2 "Resistors_SMD:R_0805" V 6930 3450 50  0001 C CNN
@@
 AR Path="/58561F68/58557010" Ref="R88"  Part="1"
 AR Path="/585624EB/58557010" Ref="R100"  Part="1"
-F 0 "R64" V 7080 3650 50  0000 C CNN
+F 0 "R100" V 7080 3650 50  0000 C CNN
 F 1 "R" V 7000 3650 50  0000 C CNN
 F 2 "Resistors_SMD:R_0805" V 6930 3650 50  0001 C CNN
@@
 AR Path="/58561F68/5855701B" Ref="R89"  Part="1"
 AR Path="/585624EB/5855701B" Ref="R101"  Part="1"
-F 0 "R65" V 7080 3850 50  0000 C CNN
+F 0 "R101" V 7080 3850 50  0000 C CNN
 F 1 "R" V 7000 3850 50  0000 C CNN
 F 2 "Resistors_SMD:R_0805" V 6930 3850 50  0001 C CNN
@@
 AR Path="/58561F68/585570B5" Ref="R90"  Part="1"
 AR Path="/585624EB/585570B5" Ref="R102"  Part="1"
-F 0 "R66" V 7080 4050 50  0000 C CNN
+F 0 "R102" V 7080 4050 50  0000 C CNN
 F 1 "R" V 7000 4050 50  0000 C CNN
 F 2 "Resistors_SMD:R_0805" V 6930 4050 50  0001 C CNN
@@
 AR Path="/58561F68/585570C0" Ref="R91"  Part="1"
 AR Path="/585624EB/585570C0" Ref="R103"  Part="1"
-F 0 "R67" V 7080 4250 50  0000 C CNN
+F 0 "R103" V 7080 4250 50  0000 C CNN
 F 1 "R" V 7000 4250 50  0000 C CNN
 F 2 "Resistors_SMD:R_0805" V 6930 4250 50  0001 C CNN
@@
 AR Path="/58561F68/5855713B" Ref="R92"  Part="1"
 AR Path="/585624EB/5855713B" Ref="R104"  Part="1"
-F 0 "R68" V 7080 4450 50  0000 C CNN
+F 0 "R104" V 7080 4450 50  0000 C CNN
 F 1 "R" V 7000 4450 50  0000 C CNN
 F 2 "Resistors_SMD:R_0805" V 6930 4450 50  0001 C CNN
@@
 AR Path="/58561F68/58557146" Ref="R93"  Part="1"
 AR Path="/585624EB/58557146" Ref="R105"  Part="1"
-F 0 "R69" V 7080 4650 50  0000 C CNN
+F 0 "R105" V 7080 4650 50  0000 C CNN
 F 1 "R" V 7000 4650 50  0000 C CNN
 F 2 "Resistors_SMD:R_0805" V 6930 4650 50  0001 C CNN
@@
 AR Path="/58561F68/585571AC" Ref="R94"  Part="1"
 AR Path="/585624EB/585571AC" Ref="R106"  Part="1"
-F 0 "R70" V 7080 4850 50  0000 C CNN
+F 0 "R106" V 7080 4850 50  0000 C CNN
 F 1 "R" V 7000 4850 50  0000 C CNN
 F 2 "Resistors_SMD:R_0805" V 6930 4850 50  0001 C CNN
@@
 AR Path="/58561F68/585571B7" Ref="R95"  Part="1"
 AR Path="/585624EB/585571B7" Ref="R107"  Part="1"
-F 0 "R71" V 7080 5050 50  0000 C CNN
+F 0 "R107" V 7080 5050 50  0000 C CNN
 F 1 "R" V 7000 5050 50  0000 C CNN
 F 2 "Resistors_SMD:R_0805" V 6930 5050 50  0001 C CNN
@@
 AR Path="/58561F68/58557233" Ref="R96"  Part="1"
 AR Path="/585624EB/58557233" Ref="R108"  Part="1"
-F 0 "R72" V 7080 5250 50  0000 C CNN
+F 0 "R108" V 7080 5250 50  0000 C CNN
 F 1 "R" V 7000 5250 50  0000 C CNN
 F 2 "Resistors_SMD:R_0805" V 6930 5250 50  0001 C CNN
@@
 AR Path="/58561F68/5855723E" Ref="R97"  Part="1"
 AR Path="/585624EB/5855723E" Ref="R109"  Part="1"
-F 0 "R73" V 7080 5450 50  0000 C CNN
+F 0 "R109" V 7080 5450 50  0000 C CNN
 F 1 "R" V 7000 5450 50  0000 C CNN
 F 2 "Resistors_SMD:R_0805" V 6930 5450 50  0001 C CNN
@@
 AR Path="/58561F68/5855725A" Ref="#PWR098"  Part="1"
 AR Path="/585624EB/5855725A" Ref="#PWR0104"  Part="1"
-F 0 "#PWR086" H 7150 5450 50  0001 C CNN
+F 0 "#PWR0104" H 7150 5450 50  0001 C CNN
 F 1 "GND" H 7150 5550 50  0000 C CNN
 F 2 "" H 7150 5700 50  0000 C CNN
@@
 AR Path="/58561F68/585574CF" Ref="P23"  Part="1"
 AR Path="/585624EB/585574CF" Ref="P26"  Part="1"
-F 0 "P17" H 5350 5550 50  0000 C CNN
+F 0 "P26" H 5350 5550 50  0000 C CNN
 F 1 "CONN_01X13" V 5450 4850 50  0000 C CNN
 F 2 "Pin_Headers:Pin_Header_Straight_1x13" H 5350 4850 50  0001 C CNN
@@
 AR Path="/58561F68/58558154" Ref="#PWR099"  Part="1"
 AR Path="/585624EB/58558154" Ref="#PWR0105"  Part="1"
-F 0 "#PWR087" H 5750 5300 50  0001 C CNN
+F 0 "#PWR0105" H 5750 5300 50  0001 C CNN
 F 1 "GND" H 5750 5400 50  0000 C CNN
 F 2 "" H 5750 5550 50  0000 C CNN
@@
 AR Path="/58561F68/58558771" Ref="C40"  Part="1"
 AR Path="/585624EB/58558771" Ref="C41"  Part="1"
-F 0 "C38" H 9325 3400 50  0000 L CNN
+F 0 "C41" H 9325 3400 50  0000 L CNN
 F 1 "C" H 9325 3200 50  0000 L CNN
 F 2 "Capacitors_SMD:C_0805" H 9338 3150 50  0001 C CNN
@@
 AR Path="/58561F68/58558AFF" Ref="#PWR0100"  Part="1"
 AR Path="/585624EB/58558AFF" Ref="#PWR0106"  Part="1"
-F 0 "#PWR088" H 8550 5650 50  0001 C CNN
+F 0 "#PWR0106" H 8550 5650 50  0001 C CNN
 F 1 "GND" H 8550 5750 50  0000 C CNN
 F 2 "" H 8550 5900 50  0000 C CNN
@@
 AR Path="/58561F68/58558BF4" Ref="P24"  Part="1"
 AR Path="/585624EB/58558BF4" Ref="P27"  Part="1"
-F 0 "P18" H 9750 6300 50  0000 C CNN
+F 0 "P27" H 9750 6300 50  0000 C CNN
 F 1 "CONN_01X03" V 9850 6100 50  0000 C CNN
 F 2 "Pin_Headers:Pin_Header_Straight_1x03" H 9750 6100 50  0001 C CNN
@@
 AR Path="/58561F68/58558C6B" Ref="P25"  Part="1"
 AR Path="/585624EB/58558C6B" Ref="P28"  Part="1"
-F 0 "P19" H 9750 6850 50  0000 C CNN
+F 0 "P28" H 9750 6850 50  0000 C CNN
 F 1 "CONN_01X03" V 9850 6650 50  0000 C CNN
 F 2 "Pin_Headers:Pin_Header_Straight_1x03" H 9750 6650 50  0001 C CNN
@@
 AR Path="/58561F68/58558CAB" Ref="#PWR0101"  Part="1"
 AR Path="/585624EB/58558CAB" Ref="#PWR0107"  Part="1"
-F 0 "#PWR089" H 9500 6550 50  0001 C CNN
+F 0 "#PWR0107" H 9500 6550 50  0001 C CNN
 F 1 "GND" H 9500 6650 50  0000 C CNN
 F 2 "" H 9500 6800 50  0000 C CNN
@@
 AR Path="/58561F68/58558ED2" Ref="#PWR0102"  Part="1"
 AR Path="/585624EB/58558ED2" Ref="#PWR0108"  Part="1"
-F 0 "#PWR090" H 9500 6000 50  0001 C CNN
+F 0 "#PWR0108" H 9500 6000 50  0001 C CNN
 F 1 "GND" H 9500 6100 50  0000 C CNN
 F 2 "" H 9500 6250 50  0000 C CNN
@@
 AR Path="/58561F68/58559799" Ref="#PWR0103"  Part="1"
 AR Path="/585624EB/58559799" Ref="#PWR0109"  Part="1"
-F 0 "#PWR091" H 9300 3300 50  0001 C CNN
+F 0 "#PWR0109" H 9300 3300 50  0001 C CNN
 F 1 "GND" H 9300 3400 50  0000 C CNN
 F 2 "" H 9300 3550 50  0000 C CNN
