File: PDB5/pwr_mod.sch (KiCad schematic (older format))
At the start: 10 parts, among them Q1 BC847CE6327HTSA1, U3 AUIPS7111S, U5 74LVC1G08

Commit message: test
Parts:
- C4: renamed from C?; footprint (none) -> Capacitors_SMD:C_0805
- D5: renamed from D?; footprint (none) -> Diodes_SMD:SOD-123
- renumbered D1 to D6, R2 to R4, R3 to R5, R4 to R6, R5 to R7, U5 to U11, U3 to U12

Commit message: test
Parts:
- removed D6: D, Diodes_SMD:D_0603, symbol D
- removed Q1: BC847CE6327HTSA1, TO_SOT_Packages_SMD:SOT-23, symbol BC847CE6327HTSA1
- removed R5, R6: R, Resistors_SMD:R_0603, symbol R
- added R26: R, Resistors_SMD:R_0603, symbol R
- U12: footprint TO_SOT_Packages_SMD:TO-263-5Lead -> KiCad-Dev:TO-263-!3
Connections:
- net Current_Feedback: now also R7.2, U12.2 (Ifb)
- net GND: now also R4.1, R26.1
- net Power_Enable_A: now also R4.2
- net Power_Enanle_B: now also R26.2
- net at U12.1 (IN): now also U11.4 (Y)
Other:
- moved on the sheet: C19, D12, R28, U18, U19

Commit message: test
Changed lines of the file:
@@
 AR Path="/5855DA87/584EF2BD" Ref="U29"  Part="1"
 AR Path="/5855DD72/584EF2BD" Ref="U31"  Part="1"
-F 0 "U19" H 7000 3450 60  0000 C CNN
+F 0 "U27" H 7000 3450 60  0000 C CNN
 F 1 "AUIPS7111S" H 7000 3550 60  0000 C CNN
 F 2 "KiCad-Dev:TO-263-!3" H 7000 3200 60  0001 C CNN
@@
 AR Path="/5855DA87/584EF2D2" Ref="R48"  Part="1"
 AR Path="/5855DD72/584EF2D2" Ref="R52"  Part="1"
-F 0 "R28" V 6630 3350 50  0000 C CNN
+F 0 "R44" V 6630 3350 50  0000 C CNN
 F 1 "R" V 6550 3350 50  0000 C CNN
 F 2 "Resistors_SMD:R_0603" V 6480 3350 50  0001 C CNN
@@
 AR Path="/5855DA87/584EF301" Ref="#PWR070"  Part="1"
 AR Path="/5855DD72/584EF301" Ref="#PWR073"  Part="1"
-F 0 "#PWR073" H 7550 2900 50  0001 C CNN
+F 0 "#PWR067" H 7550 2900 50  0001 C CNN
 F 1 "+BATT" H 7550 3190 50  0000 C CNN
 F 2 "" H 7550 3050 50  0000 C CNN
@@
 AR Path="/5855DA87/584EF611" Ref="#PWR071"  Part="1"
 AR Path="/5855DD72/584EF611" Ref="#PWR074"  Part="1"
-F 0 "#PWR074" H 3200 3450 50  0001 C CNN
+F 0 "#PWR068" H 3200 3450 50  0001 C CNN
 F 1 "GND" H 3200 3550 50  0000 C CNN
 F 2 "" H 3200 3700 50  0000 C CNN
@@
 AR Path="/5855DA87/584F6E96" Ref="#PWR072"  Part="1"
 AR Path="/5855DD72/584F6E96" Ref="#PWR075"  Part="1"
-F 0 "#PWR075" H 3200 2250 50  0001 C CNN
+F 0 "#PWR069" H 3200 2250 50  0001 C CNN
 F 1 "+3.3V" H 3200 2540 50  0000 C CNN
 F 2 "" H 3200 2400 50  0000 C CNN
@@
 AR Path="/5855DA87/5858505F" Ref="C24"  Part="1"
 AR Path="/5855DD72/5858505F" Ref="C25"  Part="1"
-F 0 "C19" H 3575 3200 50  0000 L CNN
+F 0 "C23" H 3575 3200 50  0000 L CNN
 F 1 "C" H 3575 3000 50  0000 L CNN
 F 2 "Capacitors_SMD:C_0805" H 3588 2950 50  0001 C CNN
@@
 AR Path="/5855DA87/584F6D45" Ref="U28"  Part="1"
 AR Path="/5855DD72/584F6D45" Ref="U30"  Part="1"
-F 0 "U18" H 5350 2800 60  0000 C CNN
+F 0 "U26" H 5350 2800 60  0000 C CNN
 F 1 "74LVC1G08" H 5550 3300 60  0000 C CNN
 F 2 "TO_SOT_Packages_SMD:SOT-353" H 5200 3100 60  0001 C CNN
@@
 AR Path="/5855DA87/585E0291" Ref="D22"  Part="1"
 AR Path="/5855DD72/585E0291" Ref="D24"  Part="1"
-F 0 "D12" H 3200 3200 50  0000 C CNN
+F 0 "D20" H 3200 3200 50  0000 C CNN
 F 1 "5V" H 3200 3000 50  0000 C CNN
 F 2 "Diodes_SMD:SOD-123" H 3200 3100 50  0001 C CNN
@@
 AR Path="/5855DA87/585889A1" Ref="R45"  Part="1"
 AR Path="/5855DD72/585889A1" Ref="R49"  Part="1"
-F 0 "R25" V 4680 3300 50  0000 C CNN
+F 0 "R41" V 4680 3300 50  0000 C CNN
 F 1 "R" V 4600 3300 50  0000 C CNN
 F 2 "Resistors_SMD:R_0603" V 4530 3300 50  0001 C CNN
@@
 AR Path="/5855DA87/58588A50" Ref="R46"  Part="1"
 AR Path="/5855DD72/58588A50" Ref="R50"  Part="1"
-F 0 "R26" V 4880 3300 50  0000 C CNN
+F 0 "R42" V 4880 3300 50  0000 C CNN
 F 1 "R" V 4800 3300 50  0000 C CNN
 F 2 "Resistors_SMD:R_0603" V 4730 3300 50  0001 C CNN

Commit message: test
Parts:
- added C? (x2): CP, symbol CP
- added D? (x3): D_Zener, symbol D_Zener
- added Q?: BC847CE6327HTSA1, SOT-23, symbol BC847CE6327HTSA1
- added Q?: MMBF170, SOT-23, symbol MMBF170
- added R? (x2): R, Resistors_SMD:R_0603, symbol R
- added R? (x2): R, symbol R
- added RV?: Varistor, symbol Varistor
Connections:
- wire segments 22 -> 48
Other:
- moved on the sheet: C4, D5, R4, R5, R7, U11, U12
